File: electrical/kicad/project-button-v2/05_hr30_battery_precharge.kicad_sch (KiCad schematic)
At the start: 11 parts

Commit message: Correct R11 engineering and verification blockers
Parts:
- BAT1: value Professionally assembled 4-series protected battery pack -> Protected battery pack and conversion - SELECTION REQUIRED; Display Professionally assembled 4-series protect... -> Protected battery pack and conversion - S...
Changed lines of the file:
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@@
 				)
 		)
-		(property "Value" "Professionally assembled 4-series protected battery pack"
+		(property "Value" "Protected battery pack and conversion - SELECTION REQUIRED"
 			(at 76.20 55.88 0)
 				(effects
@@
 				)
 		)
-		(property "Description" "Qualified supplier, cells, configuration, protected ports, pack limits, current, capacity, enclosure, and telemetry are unresolved."
+		(property "Description" "Qualified supplier, chemistry, series count, conversion topology, full-charge and loaded end-of-discharge limits, protected ports, fault current, capacity, enclosure, regeneration, and telemetry are unresolved."
 			(at 76.20 55.88 0)
 				(effects
@@
 				)
 		)
-		(property "Display" "Professionally assembled 4-series protect..."
+		(property "Display" "Protected battery pack and conversion - S..."
 			(at 58.42 42.67 0)
 				(effects
