File: electrical/kicad/project-button-v3/11_watchdog_pcb_connectors.kicad_sch (KiCad schematic)
At the start: 3 parts

Commit message: Add native DYNAMIXEL star injection release candidate
Other:
- title: PB HR-V0 Electrical V3 - 11 -> PB HR-V0 V3-P1.2 - 11
- moved on the sheet: JWF1, JWH1, JWP1

Commit message: Document HR-V0 contactor application evidence
Other:
- title: PB HR-V0 V3-P1.2 - 11 -> PB HR-V0 V3-P1.3 - 11
Changed lines of the file:
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@@
   (version 20250114) (generator "eeschema") (generator_version "10.0")
  (paper "A3")
-  (title_block (title "PB HR-V0 V3-P1.2 - 11") (date "2026-08-07") (rev "V3-P1.2")
+  (title_block (title "PB HR-V0 V3-P1.3 - 11") (date "2026-08-07") (rev "V3-P1.3")
     (company "Project Button") (comment 1 "PRELIMINARY - NOT APPROVED FOR FABRICATION OR ENERGIZATION") (comment 2 "CONNECTED DESIGN CANDIDATE - QUALIFIED REVIEW REQUIRED"))
   (text "PRELIMINARY - NOT APPROVED FOR FABRICATION OR ENERGIZATION" (exclude_from_sim no) (at 17.78 10.16 0)

Commit message: Add received-lot control for reset and arm terminals
Other:
- title: PB HR-V0 V3-P1.3 - 11 -> PB HR-V0 V3-P1.4 - 11
Changed lines of the file:
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@@
   (version 20250114) (generator "eeschema") (generator_version "10.0")
  (paper "A3")
-  (title_block (title "PB HR-V0 V3-P1.3 - 11") (date "2026-08-07") (rev "V3-P1.3")
+  (title_block (title "PB HR-V0 V3-P1.4 - 11") (date "2026-08-07") (rev "V3-P1.4")
     (company "Project Button") (comment 1 "PRELIMINARY - NOT APPROVED FOR FABRICATION OR ENERGIZATION") (comment 2 "CONNECTED DESIGN CANDIDATE - QUALIFIED REVIEW REQUIRED"))
   (text "PRELIMINARY - NOT APPROVED FOR FABRICATION OR ENERGIZATION" (exclude_from_sim no) (at 17.78 10.16 0)

Commit message: Reconcile H1 pilot light in electrical V3
Other:
- title: PB HR-V0 V3-P1.4 - 11 -> PB HR-V0 V3-P1.5 - 11
Changed lines of the file:
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@@
   (version 20250114) (generator "eeschema") (generator_version "10.0")
  (paper "A3")
-  (title_block (title "PB HR-V0 V3-P1.4 - 11") (date "2026-08-07") (rev "V3-P1.4")
+  (title_block (title "PB HR-V0 V3-P1.5 - 11") (date "2026-08-07") (rev "V3-P1.5")
     (company "Project Button") (comment 1 "PRELIMINARY - NOT APPROVED FOR FABRICATION OR ENERGIZATION") (comment 2 "CONNECTED DESIGN CANDIDATE - QUALIFIED REVIEW REQUIRED"))
   (text "PRELIMINARY - NOT APPROVED FOR FABRICATION OR ENERGIZATION" (exclude_from_sim no) (at 17.78 10.16 0)

Commit message: Correct control-panel protection fit
Other:
- title: PB HR-V0 V3-P1.5 - 11 -> PB HR-V0 V3-P1.6 - 11
Changed lines of the file:
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@@
   (version 20250114) (generator "eeschema") (generator_version "10.0")
  (paper "A3")
-  (title_block (title "PB HR-V0 V3-P1.5 - 11") (date "2026-08-07") (rev "V3-P1.5")
+  (title_block (title "PB HR-V0 V3-P1.6 - 11") (date "2026-08-07") (rev "V3-P1.6")
     (company "Project Button") (comment 1 "PRELIMINARY - NOT APPROVED FOR FABRICATION OR ENERGIZATION") (comment 2 "CONNECTED DESIGN CANDIDATE - QUALIFIED REVIEW REQUIRED"))
   (text "PRELIMINARY - NOT APPROVED FOR FABRICATION OR ENERGIZATION" (exclude_from_sim no) (at 17.78 10.16 0)

Commit message: Screen service disconnect and freeze fuse end cover
Other:
- title: PB HR-V0 V3-P1.6 - 11 -> PB HR-V0 V3-P1.7 - 11
Changed lines of the file:
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@@
   (version 20250114) (generator "eeschema") (generator_version "10.0")
  (paper "A3")
-  (title_block (title "PB HR-V0 V3-P1.6 - 11") (date "2026-08-07") (rev "V3-P1.6")
+  (title_block (title "PB HR-V0 V3-P1.7 - 11") (date "2026-08-07") (rev "V3-P1.7")
     (company "Project Button") (comment 1 "PRELIMINARY - NOT APPROVED FOR FABRICATION OR ENERGIZATION") (comment 2 "CONNECTED DESIGN CANDIDATE - QUALIFIED REVIEW REQUIRED"))
   (text "PRELIMINARY - NOT APPROVED FOR FABRICATION OR ENERGIZATION" (exclude_from_sim no) (at 17.78 10.16 0)

Commit message: Freeze SD1 candidate and synchronize R64
Other:
- title: PB HR-V0 V3-P1.7 - 11 -> PB HR-V0 V3-P1.8 - 11
Changed lines of the file:
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@@
   (version 20250114) (generator "eeschema") (generator_version "10.0")
  (paper "A3")
-  (title_block (title "PB HR-V0 V3-P1.7 - 11") (date "2026-08-07") (rev "V3-P1.7")
+  (title_block (title "PB HR-V0 V3-P1.8 - 11") (date "2026-08-07") (rev "V3-P1.8")
     (company "Project Button") (comment 1 "PRELIMINARY - NOT APPROVED FOR FABRICATION OR ENERGIZATION") (comment 2 "CONNECTED DESIGN CANDIDATE - QUALIFIED REVIEW REQUIRED"))
   (text "PRELIMINARY - NOT APPROVED FOR FABRICATION OR ENERGIZATION" (exclude_from_sim no) (at 17.78 10.16 0)
