File: electrical/kicad/project-button-v3/04_contactor_edm.kicad_sch (KiCad schematic)
At the start: 4 parts, among them K1 Schneider TeSys D LC1D25BD, 2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, K2 Schneider TeSys D LC1D25BD, 2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

Commit message: Screen service disconnect and freeze fuse end cover
Parts:
- FSR1, FSR2: value Phoenix PT 4-HESI (5X20) item 3211861 holder; fuse link SELECTION REQUIRED -> Phoenix PT 4-HESI (5X20) item 3211861 holder with D-ST 4 item 3030420 end cover; fuse link SELECTION REQUIRED; Display Phoenix PT 4-HESI (5X20) item 3211861 holder; fuse link SEL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 -> Phoenix PT 4-HESI (5X20) item 3211861 holder with D-ST 4 it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; Evidence Phoenix Contact official US product page and generated prod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 -> Phoenix Contact official US product pages for items 3211861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; Status PROPOSED - HOLDER ORDER CODE FROZEN; FUSE LINK AND COORDINA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 -> PROPOSED - HOLDER AND END-COVER ORDER CODES FROZEN; FUSE LI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
Other:
- note added: "NOTE 1: SRA1 outputs are separately protected before K1 and K2 coils. FSR1/FSR2 use proposed"
- note added: "Phoenix PT 4-HESI item 3211861 holders with D-ST 4 item 3030420 end cover; both fuse"
- note added: "links, grouping and coordination remain SELECTION REQUIRED."
- note removed: "NOTE 1: SRA1 outputs are separately protected before K1 and K2 coils. FSR1/FSR2 holder"
- note removed: "candidate is Phoenix PT 4-HESI (5X20) item 3211861; both fuse links, end cover and"
- note removed: "coordination remain SELECTION REQUIRED."
- title: PB HR-V0 V3-P1.6 - 04 -> PB HR-V0 V3-P1.7 - 04
Changed lines of the file:
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@@
   (version 20250114) (generator "eeschema") (generator_version "10.0")
  (paper "A3")
-  (title_block (title "PB HR-V0 V3-P1.6 - 04") (date "2026-08-07") (rev "V3-P1.6")
+  (title_block (title "PB HR-V0 V3-P1.7 - 04") (date "2026-08-07") (rev "V3-P1.7")
     (company "Project Button") (comment 1 "PRELIMINARY - NOT APPROVED FOR FABRICATION OR ENERGIZATION") (comment 2 "CONNECTED DESIGN CANDIDATE - QUALIFIED REVIEW REQUIRED"))
   (text "PRELIMINARY - NOT APPROVED FOR FABRICATION OR ENERGIZATION" (exclude_from_sim no) (at 17.78 10.16 0)
@@
 (text "W4016" (exclude_from_sim no)
               (at 342.90 202.47 0) (effects (font (size 1.27 1.27)) (justify bottom))
-) (text "NOTE 1: SRA1 outputs are separately protected before K1 and K2 coils. FSR1/FSR2 holder" (exclude_from_sim no) (at 17.78 260.00 0)
-      (effects (font (size 1.50 1.50)) (justify left bottom))) (text "        candidate is Phoenix PT 4-HESI (5X20) item 3211861; both fuse links, end cover and" (exclude_from_sim no) (at 17.78 265.50 0)
-      (effects (font (size 1.50 1.50)) (justify left bottom))) (text "        coordination remain SELECTION REQUIRED." (exclude_from_sim no) (at 17.78 271.00 0)
+) (text "NOTE 1: SRA1 outputs are separately protected before K1 and K2 coils. FSR1/FSR2 use proposed" (exclude_from_sim no) (at 17.78 260.00 0)
+      (effects (font (size 1.50 1.50)) (justify left bottom))) (text "        Phoenix PT 4-HESI item 3211861 holders with D-ST 4 item 3030420 end cover; both fuse" (exclude_from_sim no) (at 17.78 265.50 0)
+      (effects (font (size 1.50 1.50)) (justify left bottom))) (text "        links, grouping and coordination remain SELECTION REQUIRED." (exclude_from_sim no) (at 17.78 271.00 0)
       (effects (font (size 1.50 1.50)) (justify left bottom))) (text "NOTE 2: Loaded DC interruption, suppression behavior, mirror-contact use and coordination" (exclude_from_sim no) (at 17.78 276.50 0)
       (effects (font (size 1.50 1.50)) (justify left bottom))) (text "        require qualified review." (exclude_from_sim no) (at 17.78 282.00 0)
@@
       (exclude_from_sim no) (in_bom yes) (on_board yes) (dnp no)
       (property "Reference" "FSR1" (at 59.69 187.77 0) (effects (font (size 1.50 1.50)) (justify left bottom)))
-      (property "Value" "Phoenix PT 4-HESI (5X20) item 3211861 holder; fuse link SELECTION REQUIRED" (at 95.25 204.47 0) (effects (font (size 1.50 1.50)) (hide yes)))
+      (property "Value" "Phoenix PT 4-HESI (5X20) item 3211861 holder with D-ST 4 item 3030420 end cover; fuse link SELECTION REQUIRED" (at 95.25 204.47 0) (effects (font (size 1.50 1.50)) (hide yes)))
       (property "Footprint" "" (at 95.25 204.47 0) (effects (font (size 1.50 1.50)) (hide yes)))
       (property "Datasheet" "https://www.phoenixcontact.com/en-us/products/fuse-terminal-block-pt-4-hesi-5x20-3211861" (at 95.25 204.47 0) (effects (font (size 1.50 1.50)) (hide yes)))
-      (property "Description" "Exact non-LED 5x20 holder candidate only. Fuse link, compatible end cover, fault current, coil pickup/transient, conductor and PNOZ contact-protection coordination remain open; manufacturer maxima are not project selections." (at 95.25 204.47 0) (effects (font (size 1.50 1.50)) (hide yes)))
-      (property "Status" "PROPOSED - HOLDER ORDER CODE FROZEN; FUSE LINK AND COORDINATION SELECTION REQUIRED" (at 95.25 220.17 0) (effects (font (size 1.50 1.50)) (justify bottom)))
-      (property "Evidence" "Phoenix Contact official US product page and generated product PDF dated 2026-07-06; rechecked 2026-08-07." (at 95.25 204.47 0) (effects (font (size 1.50 1.50)) (hide yes)))
-      (property "Display" "Phoenix PT 4-HESI (5X20) item 3211861 holder; fuse link SELECTION REQUIRED" (at 59.69 190.97 0) (effects (font (size 1.50 1.50)) (justify left bottom)))
+      (property "Description" "Exact non-LED 5x20 holder and D-ST 4 item 3030420 end-cover candidates only. Fuse link, fault current, coil pickup/transient, conductor, grouping arrangement and PNOZ contact-protection coordination remain open; manufacturer maxima are not project selections." (at 95.25 204.47 0) (effects (font (size 1.50 1.50)) (hide yes)))
+      (property "Status" "PROPOSED - HOLDER AND END-COVER ORDER CODES FROZEN; FUSE LINK AND COORDINATION SELECTION REQUIRED" (at 95.25 220.17 0) (effects (font (size 1.50 1.50)) (justify bottom)))
+      (property "Evidence" "Phoenix Contact official US product pages for items 3211861 and 3030420; rechecked 2026-08-07." (at 95.25 204.47 0) (effects (font (size 1.50 1.50)) (hide yes)))
+      (property "Display" "Phoenix PT 4-HESI (5X20) item 3211861 holder with D-ST 4 item 3030420 end cover; fuse link SELECTION REQUIRED" (at 59.69 190.97 0) (effects (font (size 1.50 1.50)) (justify left bottom)))
       (pin "1")
       (pin "2")
@@
       (exclude_from_sim no) (in_bom yes) (on_board yes) (dnp no)
       (property "Reference" "FSR2" (at 264.16 187.77 0) (effects (font (size 1.50 1.50)) (justify left bottom)))
-      (property "Value" "Phoenix PT 4-HESI (5X20) item 3211861 holder; fuse link SELECTION REQUIRED" (at 299.72 204.47 0) (effects (font (size 1.50 1.50)) (hide yes)))
+      (property "Value" "Phoenix PT 4-HESI (5X20) item 3211861 holder with D-ST 4 item 3030420 end cover; fuse link SELECTION REQUIRED" (at 299.72 204.47 0) (effects (font (size 1.50 1.50)) (hide yes)))
       (property "Footprint" "" (at 299.72 204.47 0) (effects (font (size 1.50 1.50)) (hide yes)))
       (property "Datasheet" "https://www.phoenixcontact.com/en-us/products/fuse-terminal-block-pt-4-hesi-5x20-3211861" (at 299.72 204.47 0) (effects (font (size 1.50 1.50)) (hide yes)))
-      (property "Description" "Same exact holder candidate and open fuse-link, end-cover, coordination and physical-evidence gate as FSR1." (at 299.72 204.47 0) (effects (font (size 1.50 1.50)) (hide yes)))
-      (property "Status" "PROPOSED - HOLDER ORDER CODE FROZEN; FUSE LINK AND COORDINATION SELECTION REQUIRED" (at 299.72 220.17 0) (effects (font (size 1.50 1.50)) (justify bottom)))
-      (property "Evidence" "Phoenix Contact official US product page and generated product PDF dated 2026-07-06; rechecked 2026-08-07." (at 299.72 204.47 0) (effects (font (size 1.50 1.50)) (hide yes)))
-      (property "Display" "Phoenix PT 4-HESI (5X20) item 3211861 holder; fuse link SELECTION REQUIRED" (at 264.16 190.97 0) (effects (font (size 1.50 1.50)) (justify left bottom)))
+      (property "Description" "Same exact holder/end-cover candidates and open fuse-link, grouping, coordination and physical-evidence gate as FSR1; manufacturer maxima are not project selections." (at 299.72 204.47 0) (effects (font (size 1.50 1.50)) (hide yes)))
+      (property "Status" "PROPOSED - HOLDER AND END-COVER ORDER CODES FROZEN; FUSE LINK AND COORDINATION SELECTION REQUIRED" (at 299.72 220.17 0) (effects (font (size 1.50 1.50)) (justify bottom)))
+      (property "Evidence" "Phoenix Contact official US product pages for items 3211861 and 3030420; rechecked 2026-08-07." (at 299.72 204.47 0) (effects (font (size 1.50 1.50)) (hide yes)))
+      (property "Display" "Phoenix PT 4-HESI (5X20) item 3211861 holder with D-ST 4 item 3030420 end cover; fuse link SELECTION REQUIRED" (at 264.16 190.97 0) (effects (font (size 1.50 1.50)) (justify left bottom)))
       (pin "1")
       (pin "2")

Commit message: Freeze SD1 candidate and synchronize R64
Other:
- title: PB HR-V0 V3-P1.7 - 04 -> PB HR-V0 V3-P1.8 - 04
Changed lines of the file:
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@@
   (version 20250114) (generator "eeschema") (generator_version "10.0")
  (paper "A3")
-  (title_block (title "PB HR-V0 V3-P1.7 - 04") (date "2026-08-07") (rev "V3-P1.7")
+  (title_block (title "PB HR-V0 V3-P1.8 - 04") (date "2026-08-07") (rev "V3-P1.8")
     (company "Project Button") (comment 1 "PRELIMINARY - NOT APPROVED FOR FABRICATION OR ENERGIZATION") (comment 2 "CONNECTED DESIGN CANDIDATE - QUALIFIED REVIEW REQUIRED"))
   (text "PRELIMINARY - NOT APPROVED FOR FABRICATION OR ENERGIZATION" (exclude_from_sim no) (at 17.78 10.16 0)

Commit message: Add R79 E2 hardware slice and Electrical V3-P1.9
Other:
- title: PB HR-V0 V3-P1.8 - 04 -> PB HR-V0 V3-P1.9 - 04
Changed lines of the file:
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@@
   (version 20250114) (generator "eeschema") (generator_version "10.0")
  (paper "A3")
-  (title_block (title "PB HR-V0 V3-P1.8 - 04") (date "2026-08-07") (rev "V3-P1.8")
+  (title_block (title "PB HR-V0 V3-P1.9 - 04") (date "2026-08-08") (rev "V3-P1.9")
     (company "Project Button") (comment 1 "PRELIMINARY - NOT APPROVED FOR FABRICATION OR ENERGIZATION") (comment 2 "CONNECTED DESIGN CANDIDATE - QUALIFIED REVIEW REQUIRED"))
   (text "PRELIMINARY - NOT APPROVED FOR FABRICATION OR ENERGIZATION" (exclude_from_sim no) (at 17.78 10.16 0)
