File: electrical/kicad/project-button-v3/06_branches_and_injection.kicad_sch (KiCad schematic)
At the start: 6 parts

Commit message: Add native DYNAMIXEL star injection release candidate
Parts:
- removed INJ2: J2 data/power injection module, symbol PBV3:INJ2
- removed INJ3: Gripper data/power injection module, symbol PBV3:INJ3
- INJ1: value J1 data/power injection module -> HR-V0 DXL-STAR-P0.1 central branch-isolating injection board; Display J1 data/power injection module -> HR-V0 DXL-STAR-P0.1 central branch-isolating injection board; Status DESIGN REQUIRED -> PROPOSED - PCB/HARNESS/FAULT EVIDENCE REQUIRED
Connections:
- net ACT_0V_PE_BONDED: now also INJ1.ACT1:1 (J1 GND), INJ1.ACT2:1 (J2 GND), INJ1.ACT3:1 (J3 GND), INJ1.CTRL:1 (U2D2 GND), INJ1.PWR1:2 (J1 RETURN), INJ1.PWR2:2 (J2 RETURN), INJ1.PWR3:2 (J3 RETURN); no longer INJ1.TBD-A-G (ACT GND), INJ1.TBD-BI-G (BUS IN GND), INJ1.TBD-BO-G (BUS OUT GND)
- net DXL_TTL_DATA: now also INJ1.ACT1:3 (J1 DATA), INJ1.ACT2:3 (J2 DATA), INJ1.ACT3:3 (J3 DATA), INJ1.CTRL:3 (U2D2 DATA); no longer INJ1.TBD-A-D (ACT DATA), INJ1.TBD-BI-D (BUS IN DATA), INJ1.TBD-BO-D (BUS OUT DATA)
- net J1_VDD: now also INJ1.ACT1:2 (J1 VDD), INJ1.PWR1:1 (J1 FUSED VDD); no longer INJ1.TBD-A-V (ACT VDD), INJ1.TBD-P (FUSED VDD)
- net J2_VDD: now also INJ1.ACT2:2 (J2 VDD), INJ1.PWR2:1 (J2 FUSED VDD)
- net J3_VDD: now also INJ1.ACT3:2 (J3 VDD), INJ1.PWR3:1 (J3 FUSED VDD)
- new net INTENTIONALLY_UNUSED_U2D2_VDD: INJ1.CTRL:2 (U2D2 VDD OMITTED)
Other:
- note added: "06 Protected actuator branches and central DYNAMIXEL star injection"
- note added: "Each actuator has a separate protected VDD branch; U2D2 pin 2 and inter-actuator VDD paths are omitted."
- note added: "NOTE 1: INJ1 is a fixed central star: U2D2 pin 2 is unrouted and J1/J2/J3 positive rails"
- note added: "NOTE 2: Exact actuator cables, branch returns, enclosure, continuity, isolation, signal-"
- note added: "integrity, pull and no-backfeed tests remain release gates."
- note added: "never join."
- note removed: "06 Protected actuator branches and VDD-isolating injection"
- note removed: "Each actuator has a separate protected VDD branch; inter-actuator data cables must omit VDD."
- note removed: "NOTE 1: Standard fully populated ROBOTIS TTL daisy-chain cables are prohibited because they"
- note removed: "NOTE 2: Every injection module requires released source, continuity, isolation, pull and no-"
- note removed: "W6025"
- note removed: "W6026"
- note removed: "W6027"
- note removed: "W6028"
- note removed: "backfeed tests."
- note removed: "would parallel branch VDD."
- title: PB HR-V0 Electrical V3 - 06 -> PB HR-V0 V3-P1.2 - 06
- moved on the sheet: F1, F2, F3

Commit message: Document HR-V0 contactor application evidence
Other:
- title: PB HR-V0 V3-P1.2 - 06 -> PB HR-V0 V3-P1.3 - 06
Changed lines of the file:
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@@
   (version 20250114) (generator "eeschema") (generator_version "10.0")
  (paper "A3")
-  (title_block (title "PB HR-V0 V3-P1.2 - 06") (date "2026-08-07") (rev "V3-P1.2")
+  (title_block (title "PB HR-V0 V3-P1.3 - 06") (date "2026-08-07") (rev "V3-P1.3")
     (company "Project Button") (comment 1 "PRELIMINARY - NOT APPROVED FOR FABRICATION OR ENERGIZATION") (comment 2 "CONNECTED DESIGN CANDIDATE - QUALIFIED REVIEW REQUIRED"))
   (text "PRELIMINARY - NOT APPROVED FOR FABRICATION OR ENERGIZATION" (exclude_from_sim no) (at 17.78 10.16 0)

Commit message: Add received-lot control for reset and arm terminals
Other:
- title: PB HR-V0 V3-P1.3 - 06 -> PB HR-V0 V3-P1.4 - 06
Changed lines of the file:
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@@
   (version 20250114) (generator "eeschema") (generator_version "10.0")
  (paper "A3")
-  (title_block (title "PB HR-V0 V3-P1.3 - 06") (date "2026-08-07") (rev "V3-P1.3")
+  (title_block (title "PB HR-V0 V3-P1.4 - 06") (date "2026-08-07") (rev "V3-P1.4")
     (company "Project Button") (comment 1 "PRELIMINARY - NOT APPROVED FOR FABRICATION OR ENERGIZATION") (comment 2 "CONNECTED DESIGN CANDIDATE - QUALIFIED REVIEW REQUIRED"))
   (text "PRELIMINARY - NOT APPROVED FOR FABRICATION OR ENERGIZATION" (exclude_from_sim no) (at 17.78 10.16 0)

Commit message: Reconcile H1 pilot light in electrical V3
Other:
- title: PB HR-V0 V3-P1.4 - 06 -> PB HR-V0 V3-P1.5 - 06
Changed lines of the file:
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@@
   (version 20250114) (generator "eeschema") (generator_version "10.0")
  (paper "A3")
-  (title_block (title "PB HR-V0 V3-P1.4 - 06") (date "2026-08-07") (rev "V3-P1.4")
+  (title_block (title "PB HR-V0 V3-P1.5 - 06") (date "2026-08-07") (rev "V3-P1.5")
     (company "Project Button") (comment 1 "PRELIMINARY - NOT APPROVED FOR FABRICATION OR ENERGIZATION") (comment 2 "CONNECTED DESIGN CANDIDATE - QUALIFIED REVIEW REQUIRED"))
   (text "PRELIMINARY - NOT APPROVED FOR FABRICATION OR ENERGIZATION" (exclude_from_sim no) (at 17.78 10.16 0)

Commit message: Correct control-panel protection fit
Other:
- title: PB HR-V0 V3-P1.5 - 06 -> PB HR-V0 V3-P1.6 - 06
Changed lines of the file:
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@@
   (version 20250114) (generator "eeschema") (generator_version "10.0")
  (paper "A3")
-  (title_block (title "PB HR-V0 V3-P1.5 - 06") (date "2026-08-07") (rev "V3-P1.5")
+  (title_block (title "PB HR-V0 V3-P1.6 - 06") (date "2026-08-07") (rev "V3-P1.6")
     (company "Project Button") (comment 1 "PRELIMINARY - NOT APPROVED FOR FABRICATION OR ENERGIZATION") (comment 2 "CONNECTED DESIGN CANDIDATE - QUALIFIED REVIEW REQUIRED"))
   (text "PRELIMINARY - NOT APPROVED FOR FABRICATION OR ENERGIZATION" (exclude_from_sim no) (at 17.78 10.16 0)

Commit message: Screen service disconnect and freeze fuse end cover
Other:
- title: PB HR-V0 V3-P1.6 - 06 -> PB HR-V0 V3-P1.7 - 06
Changed lines of the file:
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@@
   (version 20250114) (generator "eeschema") (generator_version "10.0")
  (paper "A3")
-  (title_block (title "PB HR-V0 V3-P1.6 - 06") (date "2026-08-07") (rev "V3-P1.6")
+  (title_block (title "PB HR-V0 V3-P1.7 - 06") (date "2026-08-07") (rev "V3-P1.7")
     (company "Project Button") (comment 1 "PRELIMINARY - NOT APPROVED FOR FABRICATION OR ENERGIZATION") (comment 2 "CONNECTED DESIGN CANDIDATE - QUALIFIED REVIEW REQUIRED"))
   (text "PRELIMINARY - NOT APPROVED FOR FABRICATION OR ENERGIZATION" (exclude_from_sim no) (at 17.78 10.16 0)

Commit message: Freeze SD1 candidate and synchronize R64
Other:
- title: PB HR-V0 V3-P1.7 - 06 -> PB HR-V0 V3-P1.8 - 06
Changed lines of the file:
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@@
   (version 20250114) (generator "eeschema") (generator_version "10.0")
  (paper "A3")
-  (title_block (title "PB HR-V0 V3-P1.7 - 06") (date "2026-08-07") (rev "V3-P1.7")
+  (title_block (title "PB HR-V0 V3-P1.8 - 06") (date "2026-08-07") (rev "V3-P1.8")
     (company "Project Button") (comment 1 "PRELIMINARY - NOT APPROVED FOR FABRICATION OR ENERGIZATION") (comment 2 "CONNECTED DESIGN CANDIDATE - QUALIFIED REVIEW REQUIRED"))
   (text "PRELIMINARY - NOT APPROVED FOR FABRICATION OR ENERGIZATION" (exclude_from_sim no) (at 17.78 10.16 0)

Commit message: Add R79 E2 hardware slice and Electrical V3-P1.9
Other:
- title: PB HR-V0 V3-P1.8 - 06 -> PB HR-V0 V3-P1.9 - 06
Changed lines of the file:
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@@
   (version 20250114) (generator "eeschema") (generator_version "10.0")
  (paper "A3")
-  (title_block (title "PB HR-V0 V3-P1.8 - 06") (date "2026-08-07") (rev "V3-P1.8")
+  (title_block (title "PB HR-V0 V3-P1.9 - 06") (date "2026-08-08") (rev "V3-P1.9")
     (company "Project Button") (comment 1 "PRELIMINARY - NOT APPROVED FOR FABRICATION OR ENERGIZATION") (comment 2 "CONNECTED DESIGN CANDIDATE - QUALIFIED REVIEW REQUIRED"))
   (text "PRELIMINARY - NOT APPROVED FOR FABRICATION OR ENERGIZATION" (exclude_from_sim no) (at 17.78 10.16 0)
