File: electrical/kicad/project-button-v3/01_external_sources.kicad_sch (KiCad schematic)
At the start: 6 parts

Commit message: Freeze SD1 candidate and synchronize R64
Other:
- title: PB HR-V0 V3-P1.7 - 01 -> PB HR-V0 V3-P1.8 - 01
Changed lines of the file:
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@@
   (version 20250114) (generator "eeschema") (generator_version "10.0")
  (paper "A3")
-  (title_block (title "PB HR-V0 V3-P1.7 - 01") (date "2026-08-07") (rev "V3-P1.7")
+  (title_block (title "PB HR-V0 V3-P1.8 - 01") (date "2026-08-07") (rev "V3-P1.8")
     (company "Project Button") (comment 1 "PRELIMINARY - NOT APPROVED FOR FABRICATION OR ENERGIZATION") (comment 2 "CONNECTED DESIGN CANDIDATE - QUALIFIED REVIEW REQUIRED"))
   (text "PRELIMINARY - NOT APPROVED FOR FABRICATION OR ENERGIZATION" (exclude_from_sim no) (at 17.78 10.16 0)

Commit message: Add R79 E2 hardware slice and Electrical V3-P1.9
Other:
- title: PB HR-V0 V3-P1.8 - 01 -> PB HR-V0 V3-P1.9 - 01
Changed lines of the file:
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@@
   (version 20250114) (generator "eeschema") (generator_version "10.0")
  (paper "A3")
-  (title_block (title "PB HR-V0 V3-P1.8 - 01") (date "2026-08-07") (rev "V3-P1.8")
+  (title_block (title "PB HR-V0 V3-P1.9 - 01") (date "2026-08-08") (rev "V3-P1.9")
     (company "Project Button") (comment 1 "PRELIMINARY - NOT APPROVED FOR FABRICATION OR ENERGIZATION") (comment 2 "CONNECTED DESIGN CANDIDATE - QUALIFIED REVIEW REQUIRED"))
   (text "PRELIMINARY - NOT APPROVED FOR FABRICATION OR ENERGIZATION" (exclude_from_sim no) (at 17.78 10.16 0)

Commit message: Add held 24V source interface candidate
Parts:
- removed JC1: Locking 24 V DC inlet/interface, symbol PBV3:JC1
- added F24: 24 V control-source branch protection, symbol PBV3:F24
- added J24: Mean Well DC PLUG-P1J-R7B conversion candidate + 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, symbol PBV3:J24
- PSU2: Status PROPOSED - LOCKING DC INTERFACE OPEN -> PROPOSED - LOCKING CONVERSION COMPATIBILITY VERIFICATION RE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
Connections:
- net SAFETY_0V: now also J24.2 (0V A), J24.3 (0V B)
- net SAFETY_24V: now also F24.OUT (PROTECTED +24V)
- net SAFETY_24V_RAW: now also F24.IN (SOURCE +24V), J24.1 (+24V A), J24.4 (+24V B)
Other:
- note added: "W1022"
- note added: "W1023"
- title: PB HR-V0 V3-P1.9 - 01 -> PB HR-V0 V3-P1.10 - 01
- moved on the sheet: JA1, PSA1, PSU2, PSU3, SP1

Commit message: Issue R81 24 V factory-cord correction
Parts:
- J24: value Mean Well DC PLUG-P1J-R7B conversion candidate + Kycon KPJX-PM-4S panel jack -> Kycon KPJX-PM-4S panel jack candidate for GlobTek factory 4-pin locking output; Display Mean Well DC PLUG-P1J-R7B conversion candidate + Kycon KPJX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 -> Kycon KPJX-PM-4S panel jack candidate for GlobTek factory 4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; Evidence Mean Well current accessory page and industrial catalog rec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 -> GlobTek WR9QI1660YL4NKITR6B Rev B and YL4/KPPX-4P source re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; Status EXACT CATALOG/TOPOLOGY CANDIDATE - COMPATIBILITY AND PHYSIC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 -> EXACT JACK CANDIDATE - SOURCE-CORD FIT AND PHYSICAL VERIFIC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
- PSU2: value Mean Well GST40A24-P1J, 24 V 1.67 A 40 W -> GlobTek WR9QI1660YL4NKITR6B, 24 V 1.66 A 40 W, YL4/C40337 factory 4-pin locking cord; Display Mean Well GST40A24-P1J, 24 V 1.67 A 40 W -> GlobTek WR9QI1660YL4NKITR6B, 24 V 1.66 A 40 W, YL4/C40337 f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; Evidence GST40A-SPEC 2026-04-03 -> GlobTek WR9QI1660YL4NKITR6B specification Rev B; current ge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; Status PROPOSED - LOCKING CONVERSION COMPATIBILITY VERIFICATION RE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 -> EXACT SOURCE/OUTPUT-CORD CANDIDATE - RECEIVED AND APPLICATI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
Connections:
- net SAFETY_0V: now also PSU2.YL4-3 (0V / SHIELD RETURN); no longer J24.2 (0V A), PSU2.P1J-S (SLEEVE 0V)
- net SAFETY_24V_RAW: now also PSU2.YL4-1 (+24V); no longer J24.4 (+24V B), PSU2.P1J-C (CENTER +24V)
- no-connect marks 8 -> 11
Other:
- note removed: "W1022"
- note removed: "W1023"
- title: PB HR-V0 V3-P1.10 - 01 -> PB HR-V0 V3-P1.11 - 01

Commit message: Issue R82 compute and debug interface correction
Other:
- title: PB HR-V0 V3-P1.11 - 01 -> PB HR-V0 V3-P1.12 - 01
Changed lines of the file:
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@@
   (version 20250114) (generator "eeschema") (generator_version "10.0")
  (paper "A3")
-  (title_block (title "PB HR-V0 V3-P1.11 - 01") (date "2026-08-08") (rev "V3-P1.11")
+  (title_block (title "PB HR-V0 V3-P1.12 - 01") (date "2026-08-08") (rev "V3-P1.12")
     (company "Project Button") (comment 1 "PRELIMINARY - NOT APPROVED FOR FABRICATION OR ENERGIZATION") (comment 2 "CONNECTED DESIGN CANDIDATE - QUALIFIED REVIEW REQUIRED"))
   (text "PRELIMINARY - NOT APPROVED FOR FABRICATION OR ENERGIZATION" (exclude_from_sim no) (at 17.78 10.16 0)

Commit message: Add R87 watchdog-gated SR1 supply correction
Other:
- title: PB HR-V0 V3-P1.12 - 01 -> PB HR-V0 V3-P1.13 - 01
Changed lines of the file:
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@@
   (version 20250114) (generator "eeschema") (generator_version "10.0")
  (paper "A3")
-  (title_block (title "PB HR-V0 V3-P1.12 - 01") (date "2026-08-08") (rev "V3-P1.12")
+  (title_block (title "PB HR-V0 V3-P1.13 - 01") (date "2026-08-08") (rev "V3-P1.13")
     (company "Project Button") (comment 1 "PRELIMINARY - NOT APPROVED FOR FABRICATION OR ENERGIZATION") (comment 2 "CONNECTED DESIGN CANDIDATE - QUALIFIED REVIEW REQUIRED"))
   (text "PRELIMINARY - NOT APPROVED FOR FABRICATION OR ENERGIZATION" (exclude_from_sim no) (at 17.78 10.16 0)

Commit message: Add exact held Raspberry Pi compute candidates
Parts:
- PSU3: value Raspberry Pi 27W USB-C Power Supply US; color/SKU unresolved -> Raspberry Pi 27W USB-C Power Supply US Type A black, SC1158; Display Raspberry Pi 27W USB-C Power Supply US; color/SKU unresolved -> Raspberry Pi 27W USB-C Power Supply US Type A black, SC1158; Evidence Raspberry Pi product brief RP-008245-DS-1, published Octobe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 -> Raspberry Pi 27W USB-C Power Supply product brief RP-008245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; Status SELECTION REQUIRED - US SKU / COLOR / RETENTION -> EXACT CANDIDATE - RECEIVING / RETENTION / APPLICATION OPEN
Other:
- title: PB HR-V0 V3-P1.13 - 01 -> PB HR-V0 V3-P1.14 - 01
Changed lines of the file:
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@@
   (version 20250114) (generator "eeschema") (generator_version "10.0")
  (paper "A3")
-  (title_block (title "PB HR-V0 V3-P1.13 - 01") (date "2026-08-08") (rev "V3-P1.13")
+  (title_block (title "PB HR-V0 V3-P1.14 - 01") (date "2026-08-08") (rev "V3-P1.14")
     (company "Project Button") (comment 1 "PRELIMINARY - NOT APPROVED FOR FABRICATION OR ENERGIZATION") (comment 2 "CONNECTED DESIGN CANDIDATE - QUALIFIED REVIEW REQUIRED"))
   (text "PRELIMINARY - NOT APPROVED FOR FABRICATION OR ENERGIZATION" (exclude_from_sim no) (at 17.78 10.16 0)
@@
       (exclude_from_sim no) (in_bom yes) (on_board yes) (dnp no)
       (property "Reference" "PSU3" (at 285.75 192.85 0) (effects (font (size 1.50 1.50)) (justify left bottom)))
-      (property "Value" "Raspberry Pi 27W USB-C Power Supply US; color/SKU unresolved" (at 325.12 209.55 0) (effects (font (size 1.50 1.50)) (hide yes)))
+      (property "Value" "Raspberry Pi 27W USB-C Power Supply US Type A black, SC1158" (at 325.12 209.55 0) (effects (font (size 1.50 1.50)) (hide yes)))
       (property "Footprint" "" (at 325.12 209.55 0) (effects (font (size 1.50 1.50)) (hide yes)))
-      (property "Datasheet" "https://pip-assets.raspberrypi.com/categories/898-raspberry-pi-27w-usb-c-power-supply" (at 325.12 209.55 0) (effects (font (size 1.50 1.50)) (hide yes)))
-      (property "Description" "Official US Type-A regional model is frozen. Raspberry Pi's current primary portal lists twelve family SKUs without mapping each SKU to region/color, so the exact order code must not be inferred. Compute remains powered for diagnostics during E-stop and has no safety authority." (at 325.12 209.55 0) (effects (font (size 1.50 1.50)) (hide yes)))
-      (property "Status" "SELECTION REQUIRED - US SKU / COLOR / RETENTION" (at 325.12 225.25 0) (effects (font (size 1.50 1.50)) (justify bottom)))
-      (property "Evidence" "Raspberry Pi product brief RP-008245-DS-1, published October 2023 and portal-updated 2025-10-06; rechecked 2026-08-06." (at 325.12 209.55 0) (effects (font (size 1.50 1.50)) (hide yes)))
-      (property "Display" "Raspberry Pi 27W USB-C Power Supply US; color/SKU unresolved" (at 285.75 196.05 0) (effects (font (size 1.50 1.50)) (justify left bottom)))
+      (property "Datasheet" "https://www.raspberrypi.com/products/27w-power-supply/" (at 325.12 209.55 0) (effects (font (size 1.50 1.50)) (hide yes)))
+      (property "Description" "The current Raspberry Pi configurator maps the selected US Type-A black model to SC1158 through manufacturer-generated approved-reseller links. The product brief specifies 5.1 V / 5 A and a 1.2 m captive 17 AWG cable. Received identity, site/receptacle suitability, cable and USB-C retention, load/startup/brownout, thermal behavior and physical verification remain open. Compute remains powered for diagnostics during E-stop and has no safety authority." (at 325.12 209.55 0) (effects (font (size 1.50 1.50)) (hide yes)))
+      (property "Status" "EXACT CANDIDATE - RECEIVING / RETENTION / APPLICATION OPEN" (at 325.12 225.25 0) (effects (font (size 1.50 1.50)) (justify bottom)))
+      (property "Evidence" "Raspberry Pi 27W USB-C Power Supply product brief RP-008245-DS-1, published October 2023; portal/product/configurator and US authorization records rechecked 2026-08-08. Selected model: US Type A black; manufacturer-generated DigiKey/Mouser links identify SC1158." (at 325.12 209.55 0) (effects (font (size 1.50 1.50)) (hide yes)))
+      (property "Display" "Raspberry Pi 27W USB-C Power Supply US Type A black, SC1158" (at 285.75 196.05 0) (effects (font (size 1.50 1.50)) (justify left bottom)))
       (pin "USB-C-VBUS")
       (pin "USB-C-GND")
