File: electrical/kicad/project-button-v3/02_estop_eligibility.kicad_sch (KiCad schematic)
At the start: 4 parts

Commit message: Freeze SD1 candidate and synchronize R64
Other:
- title: PB HR-V0 V3-P1.7 - 02 -> PB HR-V0 V3-P1.8 - 02
Changed lines of the file:
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@@
   (version 20250114) (generator "eeschema") (generator_version "10.0")
  (paper "A3")
-  (title_block (title "PB HR-V0 V3-P1.7 - 02") (date "2026-08-07") (rev "V3-P1.7")
+  (title_block (title "PB HR-V0 V3-P1.8 - 02") (date "2026-08-07") (rev "V3-P1.8")
     (company "Project Button") (comment 1 "PRELIMINARY - NOT APPROVED FOR FABRICATION OR ENERGIZATION") (comment 2 "CONNECTED DESIGN CANDIDATE - QUALIFIED REVIEW REQUIRED"))
   (text "PRELIMINARY - NOT APPROVED FOR FABRICATION OR ENERGIZATION" (exclude_from_sim no) (at 17.78 10.16 0)

Commit message: Add R79 E2 hardware slice and Electrical V3-P1.9
Other:
- title: PB HR-V0 V3-P1.8 - 02 -> PB HR-V0 V3-P1.9 - 02
Changed lines of the file:
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@@
   (version 20250114) (generator "eeschema") (generator_version "10.0")
  (paper "A3")
-  (title_block (title "PB HR-V0 V3-P1.8 - 02") (date "2026-08-07") (rev "V3-P1.8")
+  (title_block (title "PB HR-V0 V3-P1.9 - 02") (date "2026-08-08") (rev "V3-P1.9")
     (company "Project Button") (comment 1 "PRELIMINARY - NOT APPROVED FOR FABRICATION OR ENERGIZATION") (comment 2 "CONNECTED DESIGN CANDIDATE - QUALIFIED REVIEW REQUIRED"))
   (text "PRELIMINARY - NOT APPROVED FOR FABRICATION OR ENERGIZATION" (exclude_from_sim no) (at 17.78 10.16 0)

Commit message: Add held 24V source interface candidate
Other:
- title: PB HR-V0 V3-P1.9 - 02 -> PB HR-V0 V3-P1.10 - 02
Changed lines of the file:
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@@
   (version 20250114) (generator "eeschema") (generator_version "10.0")
  (paper "A3")
-  (title_block (title "PB HR-V0 V3-P1.9 - 02") (date "2026-08-08") (rev "V3-P1.9")
+  (title_block (title "PB HR-V0 V3-P1.10 - 02") (date "2026-08-08") (rev "V3-P1.10")
     (company "Project Button") (comment 1 "PRELIMINARY - NOT APPROVED FOR FABRICATION OR ENERGIZATION") (comment 2 "CONNECTED DESIGN CANDIDATE - QUALIFIED REVIEW REQUIRED"))
   (text "PRELIMINARY - NOT APPROVED FOR FABRICATION OR ENERGIZATION" (exclude_from_sim no) (at 17.78 10.16 0)

Commit message: Issue R81 24 V factory-cord correction
Other:
- title: PB HR-V0 V3-P1.10 - 02 -> PB HR-V0 V3-P1.11 - 02
Changed lines of the file:
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@@
   (version 20250114) (generator "eeschema") (generator_version "10.0")
  (paper "A3")
-  (title_block (title "PB HR-V0 V3-P1.10 - 02") (date "2026-08-08") (rev "V3-P1.10")
+  (title_block (title "PB HR-V0 V3-P1.11 - 02") (date "2026-08-08") (rev "V3-P1.11")
     (company "Project Button") (comment 1 "PRELIMINARY - NOT APPROVED FOR FABRICATION OR ENERGIZATION") (comment 2 "CONNECTED DESIGN CANDIDATE - QUALIFIED REVIEW REQUIRED"))
   (text "PRELIMINARY - NOT APPROVED FOR FABRICATION OR ENERGIZATION" (exclude_from_sim no) (at 17.78 10.16 0)

Commit message: Issue R82 compute and debug interface correction
Other:
- title: PB HR-V0 V3-P1.11 - 02 -> PB HR-V0 V3-P1.12 - 02
Changed lines of the file:
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@@
   (version 20250114) (generator "eeschema") (generator_version "10.0")
  (paper "A3")
-  (title_block (title "PB HR-V0 V3-P1.11 - 02") (date "2026-08-08") (rev "V3-P1.11")
+  (title_block (title "PB HR-V0 V3-P1.12 - 02") (date "2026-08-08") (rev "V3-P1.12")
     (company "Project Button") (comment 1 "PRELIMINARY - NOT APPROVED FOR FABRICATION OR ENERGIZATION") (comment 2 "CONNECTED DESIGN CANDIDATE - QUALIFIED REVIEW REQUIRED"))
   (text "PRELIMINARY - NOT APPROVED FOR FABRICATION OR ENERGIZATION" (exclude_from_sim no) (at 17.78 10.16 0)

Commit message: Add R87 watchdog-gated SR1 supply correction
Connections:
- net WD1_SAFETY_IN is gone; now on net SR1_S12: S0.R-2 (CH1 RIGHT NC MARK 2)
- net WD2_SAFETY_IN is gone; now on net SR1_S22: S0.L-2 (CH2 LEFT NC MARK 2)
- net SAFETY_24V: no longer SR1.A1 (24V SUPPLY)
- new net SR1_A1_WD_GATED: SR1.A1 (24V SUPPLY)
Other:
- note added: "Each SR1 input return contains only one S0 NC contact; RESET cannot energize K1/K2."
- note added: "NOTE 1: S0 directly completes both SR1 input returns; ordinary KWD terminals are absent from"
- note added: "NOTE 2: Heartbeat loss removes SR1 A1 through the separate two-contact supply gate; recovery"
- note added: "alone cannot restore the monitored RESET stage."
- note added: "both loops."
- note removed: "Each SR1 input return contains one E-stop NC and one watchdog NO contact; RESET cannot energize K1/K2."
- note removed: "NOTE 1: Heartbeat loss opens both SR1 input returns; recovery alone cannot restore the"
- note removed: "NOTE 2: RESET release may make SR1 eligible, but SRA1 and K1/K2 remain de-energized until a"
- note removed: "later ARM."
- note removed: "monitored RESET stage."
- title: PB HR-V0 V3-P1.12 - 02 -> PB HR-V0 V3-P1.13 - 02
Changed lines of the file:
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@@
   (version 20250114) (generator "eeschema") (generator_version "10.0")
  (paper "A3")
-  (title_block (title "PB HR-V0 V3-P1.12 - 02") (date "2026-08-08") (rev "V3-P1.12")
+  (title_block (title "PB HR-V0 V3-P1.13 - 02") (date "2026-08-08") (rev "V3-P1.13")
     (company "Project Button") (comment 1 "PRELIMINARY - NOT APPROVED FOR FABRICATION OR ENERGIZATION") (comment 2 "CONNECTED DESIGN CANDIDATE - QUALIFIED REVIEW REQUIRED"))
   (text "PRELIMINARY - NOT APPROVED FOR FABRICATION OR ENERGIZATION" (exclude_from_sim no) (at 17.78 10.16 0)
       (effects (font (size 2.54 2.54)) (justify left bottom))) (text "02  Dual-channel E-stop and RESET eligibility" (exclude_from_sim no) (at 17.78 19.05 0)
-      (effects (font (size 2.20 2.20)) (justify left bottom))) (text "Each SR1 input return contains one E-stop NC and one watchdog NO contact; RESET cannot energize K1/K2." (exclude_from_sim no) (at 17.78 26.67 0)
+      (effects (font (size 2.20 2.20)) (justify left bottom))) (text "Each SR1 input return contains only one S0 NC contact; RESET cannot energize K1/K2." (exclude_from_sim no) (at 17.78 26.67 0)
       (effects (font (size 1.80 1.80)) (justify left bottom))) (rectangle (start 12.70 31.75) (end 406.40 281.94)
       (stroke (width 0.50) (type solid)) (fill (type none))) (wire (pts (xy 52.07 87.63) (xy 41.91 87.63))
@@
 (wire (pts (xy 138.43 87.63) (xy 148.59 87.63))
               (stroke (width 0) (type default)))
-(global_label "WD1_SAFETY_IN" (shape bidirectional) (at 148.59 87.63 0)
+(global_label "SR1_S12" (shape bidirectional) (at 148.59 87.63 0)
               (fields_autoplaced yes) (effects (font (size 1.50 1.50)) (justify left))
               (property "Intersheetrefs" "${INTERSHEET_REFS}" (at 148.59 90.17 0)
@@
 (wire (pts (xy 138.43 82.55) (xy 148.59 82.55))
               (stroke (width 0) (type default)))
-(global_label "WD2_SAFETY_IN" (shape bidirectional) (at 148.59 82.55 0)
+(global_label "SR1_S22" (shape bidirectional) (at 148.59 82.55 0)
               (fields_autoplaced yes) (effects (font (size 1.50 1.50)) (justify left))
               (property "Intersheetrefs" "${INTERSHEET_REFS}" (at 148.59 85.09 0)
@@
 ) (wire (pts (xy 256.54 110.49) (xy 246.38 110.49))
               (stroke (width 0) (type default)))
-(global_label "SAFETY_24V" (shape bidirectional) (at 246.38 110.49 180)
+(global_label "SR1_A1_WD_GATED" (shape bidirectional) (at 246.38 110.49 180)
               (fields_autoplaced yes) (effects (font (size 1.50 1.50)) (justify right))
               (property "Intersheetrefs" "${INTERSHEET_REFS}" (at 246.38 113.03 0)
@@
 (text "W2021" (exclude_from_sim no)
               (at 347.98 202.47 0) (effects (font (size 1.27 1.27)) (justify bottom))
-) (text "NOTE 1: Heartbeat loss opens both SR1 input returns; recovery alone cannot restore the" (exclude_from_sim no) (at 17.78 260.00 0)
-      (effects (font (size 1.50 1.50)) (justify left bottom))) (text "        monitored RESET stage." (exclude_from_sim no) (at 17.78 265.50 0)
-      (effects (font (size 1.50 1.50)) (justify left bottom))) (text "NOTE 2: RESET release may make SR1 eligible, but SRA1 and K1/K2 remain de-energized until a" (exclude_from_sim no) (at 17.78 271.00 0)
-      (effects (font (size 1.50 1.50)) (justify left bottom))) (text "        later ARM." (exclude_from_sim no) (at 17.78 276.50 0)
+) (text "NOTE 1: S0 directly completes both SR1 input returns; ordinary KWD terminals are absent from" (exclude_from_sim no) (at 17.78 260.00 0)
+      (effects (font (size 1.50 1.50)) (justify left bottom))) (text "        both loops." (exclude_from_sim no) (at 17.78 265.50 0)
+      (effects (font (size 1.50 1.50)) (justify left bottom))) (text "NOTE 2: Heartbeat loss removes SR1 A1 through the separate two-contact supply gate; recovery" (exclude_from_sim no) (at 17.78 271.00 0)
+      (effects (font (size 1.50 1.50)) (justify left bottom))) (text "        alone cannot restore the monitored RESET stage." (exclude_from_sim no) (at 17.78 276.50 0)
       (effects (font (size 1.50 1.50)) (justify left bottom)))
   (symbol

Commit message: Control PNOZ path conformance
Parts:
- SR1: Evidence Pilz operating manual 21396-EN-23, product file 2026-06-22;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 -> Pilz operating manual 21396-EN-23; PDF metadata 2026-06-17;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
Changed lines of the file:
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@@
       (property "Description" "First-stage E-stop eligibility relay. Mode: short-cross detection plus monitored start on falling edge; seal and inspect selector with power removed." (at 299.72 95.25 0) (effects (font (size 1.50 1.50)) (hide yes)))
       (property "Status" "PROPOSED - QUALIFIED APPLICATION REVIEW REQUIRED" (at 299.72 123.65 0) (effects (font (size 1.50 1.50)) (justify bottom)))
-      (property "Evidence" "Pilz operating manual 21396-EN-23, product file 2026-06-22; terminals and timing rechecked 2026-08-06." (at 299.72 95.25 0) (effects (font (size 1.50 1.50)) (hide yes)))
+      (property "Evidence" "Pilz operating manual 21396-EN-23; PDF metadata 2026-06-17; portal file 2026-06-22; SHA-256 4B6E4768CEFAEDAF54F006347D32A8A04964B59A16F3616D8AC43698D3626BB4; terminals and timing rechecked 2026-08-08." (at 299.72 95.25 0) (effects (font (size 1.50 1.50)) (hide yes)))
       (property "Display" "Pilz PNOZ s4 24 VDC 3 n/o 1 n/c, order 750104" (at 259.08 69.05 0) (effects (font (size 1.50 1.50)) (justify left bottom)))
       (pin "A1")

Commit message: Add exact held Raspberry Pi compute candidates
Other:
- title: PB HR-V0 V3-P1.13 - 02 -> PB HR-V0 V3-P1.14 - 02
Changed lines of the file:
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@@
   (version 20250114) (generator "eeschema") (generator_version "10.0")
  (paper "A3")
-  (title_block (title "PB HR-V0 V3-P1.13 - 02") (date "2026-08-08") (rev "V3-P1.13")
+  (title_block (title "PB HR-V0 V3-P1.14 - 02") (date "2026-08-08") (rev "V3-P1.14")
     (company "Project Button") (comment 1 "PRELIMINARY - NOT APPROVED FOR FABRICATION OR ENERGIZATION") (comment 2 "CONNECTED DESIGN CANDIDATE - QUALIFIED REVIEW REQUIRED"))
   (text "PRELIMINARY - NOT APPROVED FOR FABRICATION OR ENERGIZATION" (exclude_from_sim no) (at 17.78 10.16 0)
