File: electrical/kicad/project-button-v3/07_watchdog_control.kicad_sch (KiCad schematic)
At the start: 9 parts

Commit message: Freeze SD1 candidate and synchronize R64
Other:
- title: PB HR-V0 V3-P1.7 - 07 -> PB HR-V0 V3-P1.8 - 07
Changed lines of the file:
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@@
   (version 20250114) (generator "eeschema") (generator_version "10.0")
  (paper "A3")
-  (title_block (title "PB HR-V0 V3-P1.7 - 07") (date "2026-08-07") (rev "V3-P1.7")
+  (title_block (title "PB HR-V0 V3-P1.8 - 07") (date "2026-08-07") (rev "V3-P1.8")
     (company "Project Button") (comment 1 "PRELIMINARY - NOT APPROVED FOR FABRICATION OR ENERGIZATION") (comment 2 "CONNECTED DESIGN CANDIDATE - QUALIFIED REVIEW REQUIRED"))
   (text "PRELIMINARY - NOT APPROVED FOR FABRICATION OR ENERGIZATION" (exclude_from_sim no) (at 17.78 10.16 0)

Commit message: Add R79 E2 hardware slice and Electrical V3-P1.9
Other:
- title: PB HR-V0 V3-P1.8 - 07 -> PB HR-V0 V3-P1.9 - 07
Changed lines of the file:
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@@
   (version 20250114) (generator "eeschema") (generator_version "10.0")
  (paper "A3")
-  (title_block (title "PB HR-V0 V3-P1.8 - 07") (date "2026-08-07") (rev "V3-P1.8")
+  (title_block (title "PB HR-V0 V3-P1.9 - 07") (date "2026-08-08") (rev "V3-P1.9")
     (company "Project Button") (comment 1 "PRELIMINARY - NOT APPROVED FOR FABRICATION OR ENERGIZATION") (comment 2 "CONNECTED DESIGN CANDIDATE - QUALIFIED REVIEW REQUIRED"))
   (text "PRELIMINARY - NOT APPROVED FOR FABRICATION OR ENERGIZATION" (exclude_from_sim no) (at 17.78 10.16 0)

Commit message: Add held 24V source interface candidate
Other:
- title: PB HR-V0 V3-P1.9 - 07 -> PB HR-V0 V3-P1.10 - 07
Changed lines of the file:
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@@
   (version 20250114) (generator "eeschema") (generator_version "10.0")
  (paper "A3")
-  (title_block (title "PB HR-V0 V3-P1.9 - 07") (date "2026-08-08") (rev "V3-P1.9")
+  (title_block (title "PB HR-V0 V3-P1.10 - 07") (date "2026-08-08") (rev "V3-P1.10")
     (company "Project Button") (comment 1 "PRELIMINARY - NOT APPROVED FOR FABRICATION OR ENERGIZATION") (comment 2 "CONNECTED DESIGN CANDIDATE - QUALIFIED REVIEW REQUIRED"))
   (text "PRELIMINARY - NOT APPROVED FOR FABRICATION OR ENERGIZATION" (exclude_from_sim no) (at 17.78 10.16 0)

Commit message: Issue R81 24 V factory-cord correction
Other:
- title: PB HR-V0 V3-P1.10 - 07 -> PB HR-V0 V3-P1.11 - 07
Changed lines of the file:
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@@
   (version 20250114) (generator "eeschema") (generator_version "10.0")
  (paper "A3")
-  (title_block (title "PB HR-V0 V3-P1.10 - 07") (date "2026-08-08") (rev "V3-P1.10")
+  (title_block (title "PB HR-V0 V3-P1.11 - 07") (date "2026-08-08") (rev "V3-P1.11")
     (company "Project Button") (comment 1 "PRELIMINARY - NOT APPROVED FOR FABRICATION OR ENERGIZATION") (comment 2 "CONNECTED DESIGN CANDIDATE - QUALIFIED REVIEW REQUIRED"))
   (text "PRELIMINARY - NOT APPROVED FOR FABRICATION OR ENERGIZATION" (exclude_from_sim no) (at 17.78 10.16 0)

Commit message: Issue R82 compute and debug interface correction
Other:
- title: PB HR-V0 V3-P1.11 - 07 -> PB HR-V0 V3-P1.12 - 07
Changed lines of the file:
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@@
   (version 20250114) (generator "eeschema") (generator_version "10.0")
  (paper "A3")
-  (title_block (title "PB HR-V0 V3-P1.11 - 07") (date "2026-08-08") (rev "V3-P1.11")
+  (title_block (title "PB HR-V0 V3-P1.12 - 07") (date "2026-08-08") (rev "V3-P1.12")
     (company "Project Button") (comment 1 "PRELIMINARY - NOT APPROVED FOR FABRICATION OR ENERGIZATION") (comment 2 "CONNECTED DESIGN CANDIDATE - QUALIFIED REVIEW REQUIRED"))
   (text "PRELIMINARY - NOT APPROVED FOR FABRICATION OR ENERGIZATION" (exclude_from_sim no) (at 17.78 10.16 0)

Commit message: Add R87 watchdog-gated SR1 supply correction
Other:
- title: PB HR-V0 V3-P1.12 - 07 -> PB HR-V0 V3-P1.13 - 07
Changed lines of the file:
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@@
   (version 20250114) (generator "eeschema") (generator_version "10.0")
  (paper "A3")
-  (title_block (title "PB HR-V0 V3-P1.12 - 07") (date "2026-08-08") (rev "V3-P1.12")
+  (title_block (title "PB HR-V0 V3-P1.13 - 07") (date "2026-08-08") (rev "V3-P1.13")
     (company "Project Button") (comment 1 "PRELIMINARY - NOT APPROVED FOR FABRICATION OR ENERGIZATION") (comment 2 "CONNECTED DESIGN CANDIDATE - QUALIFIED REVIEW REQUIRED"))
   (text "PRELIMINARY - NOT APPROVED FOR FABRICATION OR ENERGIZATION" (exclude_from_sim no) (at 17.78 10.16 0)

Commit message: Correct watchdog PCB land patterns and supersede P0.5 CAM
Parts:
- CDRV1, CDRV2: footprint Capacitor_SMD:C_0805_2012Metric_Pad1.18x1.45mm_HandSolder -> PBV3_Footprints:Murata_GRM21_Reflow_Nominal
- RHB1, RHP1: footprint Resistor_SMD:R_0805_2012Metric_Pad1.20x1.40mm_HandSolder -> PBV3_Footprints:Panasonic_ERJ6_Reflow_Nominal
- UDRV1, UDRV2: footprint Package_SO:TSSOP-16_4.4x5mm_P0.65mm -> PBV3_Footprints:TI_PW0016A_Example_Land
Changed lines of the file:
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@@
       (property "Reference" "RHB1" (at 149.86 63.31 0) (effects (font (size 1.50 1.50)) (justify left bottom)))
       (property "Value" "Panasonic ERJ6ENF9100V, 910 Ohm 1% 0805 0.125 W" (at 190.50 80.01 0) (effects (font (size 1.50 1.50)) (hide yes)))
-      (property "Footprint" "Resistor_SMD:R_0805_2012Metric_Pad1.20x1.40mm_HandSolder" (at 190.50 80.01 0) (effects (font (size 1.50 1.50)) (hide yes)))
+      (property "Footprint" "PBV3_Footprints:Panasonic_ERJ6_Reflow_Nominal" (at 190.50 80.01 0) (effects (font (size 1.50 1.50)) (hide yes)))
       (property "Datasheet" "https://industrial.panasonic.com/ww/products/pt/general-purpose-chip-resistors/models/ERJ6ENF9100V" (at 190.50 80.01 0) (effects (font (size 1.50 1.50)) (hide yes)))
       (property "Description" "Screens approximately 1.04 mA at a project 2.6 V GPIO-high floor and 1.65 V LED maximum, and 2.53 mA at 3.3 V with 1.0 V LED minimum. The 2.6 V floor is a project screen, not a released Raspberry Pi 5 guarantee; measure the actual source across load and temperature." (at 190.50 80.01 0) (effects (font (size 1.50 1.50)) (hide yes)))
@@
       (property "Reference" "RHP1" (at 299.72 98.87 0) (effects (font (size 1.50 1.50)) (justify left bottom)))
       (property "Value" "Panasonic ERJ6ENF1002V, 10.0 kOhm 1% 0805 0.125 W" (at 340.36 115.57 0) (effects (font (size 1.50 1.50)) (hide yes)))
-      (property "Footprint" "Resistor_SMD:R_0805_2012Metric_Pad1.20x1.40mm_HandSolder" (at 340.36 115.57 0) (effects (font (size 1.50 1.50)) (hide yes)))
+      (property "Footprint" "PBV3_Footprints:Panasonic_ERJ6_Reflow_Nominal" (at 340.36 115.57 0) (effects (font (size 1.50 1.50)) (hide yes)))
       (property "Datasheet" "https://industrial.panasonic.com/ww/products/pt/general-purpose-chip-resistors/models/ERJ6ENF1002V" (at 340.36 115.57 0) (effects (font (size 1.50 1.50)) (hide yes)))
       (property "Description" "The 10 kOhm pullup draws 0.33 mA at 3.3 V. Confirm logic thresholds, leakage, power sequencing, waveform rise/fall time and fault response on the released PCB." (at 340.36 115.57 0) (effects (font (size 1.50 1.50)) (hide yes)))
@@
       (property "Reference" "UDRV1" (at 209.55 120.46 0) (effects (font (size 1.50 1.50)) (justify left bottom)))
       (property "Value" "Texas Instruments TPL7407LPWR channel-1 relay driver" (at 250.19 149.86 0) (effects (font (size 1.50 1.50)) (hide yes)))
-      (property "Footprint" "Package_SO:TSSOP-16_4.4x5mm_P0.65mm" (at 250.19 149.86 0) (effects (font (size 1.50 1.50)) (hide yes)))
+      (property "Footprint" "PBV3_Footprints:TI_PW0016A_Example_Land" (at 250.19 149.86 0) (effects (font (size 1.50 1.50)) (hide yes)))
       (property "Datasheet" "https://www.ti.com/lit/ds/symlink/tpl7407l.pdf" (at 250.19 149.86 0) (effects (font (size 1.50 1.50)) (hide yes)))
       (property "Description" "Dedicated package for channel 1. COM is tied to the 24 V coil rail for the internal clamp; unused inputs are tied low and unused outputs are no-connect. Default-off, hot-plug/COM slew, clamp interaction with the relay module, thermal, brownout, open/short and cross-channel faults remain open." (at 250.19 149.86 0) (effects (font (size 1.50 1.50)) (hide yes)))
@@
       (property "Reference" "CDRV1" (at 54.61 102.68 0) (effects (font (size 1.50 1.50)) (justify left bottom)))
       (property "Value" "Murata GRM21BR71H104KA01L, 100 nF 50 V X7R 0805" (at 95.25 119.38 0) (effects (font (size 1.50 1.50)) (hide yes)))
-      (property "Footprint" "Capacitor_SMD:C_0805_2012Metric_Pad1.18x1.45mm_HandSolder" (at 95.25 119.38 0) (effects (font (size 1.50 1.50)) (hide yes)))
+      (property "Footprint" "PBV3_Footprints:Murata_GRM21_Reflow_Nominal" (at 95.25 119.38 0) (effects (font (size 1.50 1.50)) (hide yes)))
       (property "Datasheet" "https://pim.murata.com/asset/pim4/ceramicCapacitorSMD/GRM21BR71H104KA01-01-EN_PDF_CERAMICCAPACITORSMD?lastModifiedDatetime=20250707233810" (at 95.25 119.38 0) (effects (font (size 1.50 1.50)) (hide yes)))
       (property "Description" "Local COM bypass candidate for UDRV1. Capacitance alone does not prove TI's less-than-0.5 V/us COM slew requirement; scope hot-plug and repetitive transients in the released layout." (at 95.25 119.38 0) (effects (font (size 1.50 1.50)) (hide yes)))
@@
       (property "Reference" "UDRV2" (at 209.55 200.47 0) (effects (font (size 1.50 1.50)) (justify left bottom)))
       (property "Value" "Texas Instruments TPL7407LPWR channel-2 relay driver" (at 250.19 229.87 0) (effects (font (size 1.50 1.50)) (hide yes)))
-      (property "Footprint" "Package_SO:TSSOP-16_4.4x5mm_P0.65mm" (at 250.19 229.87 0) (effects (font (size 1.50 1.50)) (hide yes)))
+      (property "Footprint" "PBV3_Footprints:TI_PW0016A_Example_Land" (at 250.19 229.87 0) (effects (font (size 1.50 1.50)) (hide yes)))
       (property "Datasheet" "https://www.ti.com/lit/ds/symlink/tpl7407l.pdf" (at 250.19 229.87 0) (effects (font (size 1.50 1.50)) (hide yes)))
       (property "Description" "Separate package for channel 2 to avoid one driver-package fault controlling both coils. The controller, supplies, clock and firmware remain common causes; no safety credit is claimed." (at 250.19 229.87 0) (effects (font (size 1.50 1.50)) (hide yes)))
@@
       (property "Reference" "CDRV2" (at 54.61 143.32 0) (effects (font (size 1.50 1.50)) (justify left bottom)))
       (property "Value" "Murata GRM21BR71H104KA01L, 100 nF 50 V X7R 0805" (at 95.25 160.02 0) (effects (font (size 1.50 1.50)) (hide yes)))
-      (property "Footprint" "Capacitor_SMD:C_0805_2012Metric_Pad1.18x1.45mm_HandSolder" (at 95.25 160.02 0) (effects (font (size 1.50 1.50)) (hide yes)))
+      (property "Footprint" "PBV3_Footprints:Murata_GRM21_Reflow_Nominal" (at 95.25 160.02 0) (effects (font (size 1.50 1.50)) (hide yes)))
       (property "Datasheet" "https://pim.murata.com/asset/pim4/ceramicCapacitorSMD/GRM21BR71H104KA01-01-EN_PDF_CERAMICCAPACITORSMD?lastModifiedDatetime=20250707233810" (at 95.25 160.02 0) (effects (font (size 1.50 1.50)) (hide yes)))
       (property "Description" "Local COM bypass candidate for UDRV2; the same physical slew and fault evidence remains mandatory." (at 95.25 160.02 0) (effects (font (size 1.50 1.50)) (hide yes)))

Commit message: Add exact held Raspberry Pi compute candidates
Other:
- title: PB HR-V0 V3-P1.13 - 07 -> PB HR-V0 V3-P1.14 - 07
Changed lines of the file:
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@@
   (version 20250114) (generator "eeschema") (generator_version "10.0")
  (paper "A3")
-  (title_block (title "PB HR-V0 V3-P1.13 - 07") (date "2026-08-08") (rev "V3-P1.13")
+  (title_block (title "PB HR-V0 V3-P1.14 - 07") (date "2026-08-08") (rev "V3-P1.14")
     (company "Project Button") (comment 1 "PRELIMINARY - NOT APPROVED FOR FABRICATION OR ENERGIZATION") (comment 2 "CONNECTED DESIGN CANDIDATE - QUALIFIED REVIEW REQUIRED"))
   (text "PRELIMINARY - NOT APPROVED FOR FABRICATION OR ENERGIZATION" (exclude_from_sim no) (at 17.78 10.16 0)
