File: hr30/whole-body-p0.1/electrical/kicad/hr30-whole-body-electrical-p0.1/06_right_leg_rs485.kicad_sch (KiCad schematic)
At the start: 8 parts

Commit message: Add HR-30 whole-body harness architecture
Parts:
- AX_R_ANKLE_PITCH, AX_R_ANKLE_ROLL, AX_R_HIP_PITCH, AX_R_HIP_ROLL, AX_R_HIP_YAW, AX_R_KNEE_PITCH: Evidence Official ROBOTIS e-Manual interface family checked 2026-08-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 -> Current official ROBOTIS Docs checked 2026-08-14: actuator-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; Status SELECTION REQUIRED - LOGICAL CONNECTIVITY ONLY -> ACTUATOR-SIDE PINOUT VERIFIED - HARNESS AND CONTROLLER SIDE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
Connections:
- net RS-RLEG_DN: now also AX_R_ANKLE_PITCH.4 (DATA-), AX_R_ANKLE_ROLL.4 (DATA-), AX_R_HIP_PITCH.4 (DATA-), AX_R_HIP_ROLL.4 (DATA-), AX_R_HIP_YAW.4 (DATA-), AX_R_KNEE_PITCH.4 (DATA-); no longer AX_R_ANKLE_PITCH.LOG-DN (RS-485 DATA-), AX_R_ANKLE_ROLL.LOG-DN (RS-485 DATA-), AX_R_HIP_PITCH.LOG-DN (RS-485 DATA-), AX_R_HIP_ROLL.LOG-DN (RS-485 DATA-), AX_R_HIP_YAW.LOG-DN (RS-485 DATA-), AX_R_KNEE_PITCH.LOG-DN (RS-485 DATA-)
- net RS-RLEG_DP: now also AX_R_ANKLE_PITCH.3 (DATA+), AX_R_ANKLE_ROLL.3 (DATA+), AX_R_HIP_PITCH.3 (DATA+), AX_R_HIP_ROLL.3 (DATA+), AX_R_HIP_YAW.3 (DATA+), AX_R_KNEE_PITCH.3 (DATA+); no longer AX_R_ANKLE_PITCH.LOG-DP (RS-485 DATA+), AX_R_ANKLE_ROLL.LOG-DP (RS-485 DATA+), AX_R_HIP_PITCH.LOG-DP (RS-485 DATA+), AX_R_HIP_ROLL.LOG-DP (RS-485 DATA+), AX_R_HIP_YAW.LOG-DP (RS-485 DATA+), AX_R_KNEE_PITCH.LOG-DP (RS-485 DATA+)
- net RS-RLEG_RET: now also AX_R_ANKLE_PITCH.1 (GND), AX_R_ANKLE_ROLL.1 (GND), AX_R_HIP_PITCH.1 (GND), AX_R_HIP_ROLL.1 (GND), AX_R_HIP_YAW.1 (GND), AX_R_KNEE_PITCH.1 (GND); no longer AX_R_ANKLE_PITCH.LOG-RET (BRANCH RETURN), AX_R_ANKLE_ROLL.LOG-RET (BRANCH RETURN), AX_R_HIP_PITCH.LOG-RET (BRANCH RETURN), AX_R_HIP_ROLL.LOG-RET (BRANCH RETURN), AX_R_HIP_YAW.LOG-RET (BRANCH RETURN), AX_R_KNEE_PITCH.LOG-RET (BRANCH RETURN)
- net RS-RLEG_VDD: now also AX_R_ANKLE_PITCH.2 (VDD), AX_R_ANKLE_ROLL.2 (VDD), AX_R_HIP_PITCH.2 (VDD), AX_R_HIP_ROLL.2 (VDD), AX_R_HIP_YAW.2 (VDD), AX_R_KNEE_PITCH.2 (VDD); no longer AX_R_ANKLE_PITCH.LOG-PWR (BRANCH VDD), AX_R_ANKLE_ROLL.LOG-PWR (BRANCH VDD), AX_R_HIP_PITCH.LOG-PWR (BRANCH VDD), AX_R_HIP_ROLL.LOG-PWR (BRANCH VDD), AX_R_HIP_YAW.LOG-PWR (BRANCH VDD), AX_R_KNEE_PITCH.LOG-PWR (BRANCH VDD)
Other:
- note added: "NOTE 2: AX_* terminals use current official ROBOTIS actuator-side pin numbers; all LOG-*"
- note added: "identifiers remain functional ports, not physical connector or IC pins."
- note removed: "NOTE 2: All terminal identifiers beginning LOG- are functional ports, not manufacturer"
- note removed: "connector or package pin numbers."
