File: hr30/whole-body-p0.1/electrical/kicad/hr30-whole-body-electrical-p0.1/08_right_arm_rs485.kicad_sch (KiCad schematic)
At the start: 5 parts

Commit message: Add HR-30 whole-body harness architecture
Parts:
- AX_R_ELBOW_PITCH, AX_R_SHOULDER_PITCH, AX_R_SHOULDER_ROLL: Evidence Official ROBOTIS e-Manual interface family checked 2026-08-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 -> Current official ROBOTIS Docs checked 2026-08-14: actuator-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; Status SELECTION REQUIRED - LOGICAL CONNECTIVITY ONLY -> ACTUATOR-SIDE PINOUT VERIFIED - HARNESS AND CONTROLLER SIDE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
Connections:
- net RS-RARM_DN: now also AX_R_ELBOW_PITCH.4 (DATA-), AX_R_SHOULDER_PITCH.4 (DATA-), AX_R_SHOULDER_ROLL.4 (DATA-); no longer AX_R_ELBOW_PITCH.LOG-DN (RS-485 DATA-), AX_R_SHOULDER_PITCH.LOG-DN (RS-485 DATA-), AX_R_SHOULDER_ROLL.LOG-DN (RS-485 DATA-)
- net RS-RARM_DP: now also AX_R_ELBOW_PITCH.3 (DATA+), AX_R_SHOULDER_PITCH.3 (DATA+), AX_R_SHOULDER_ROLL.3 (DATA+); no longer AX_R_ELBOW_PITCH.LOG-DP (RS-485 DATA+), AX_R_SHOULDER_PITCH.LOG-DP (RS-485 DATA+), AX_R_SHOULDER_ROLL.LOG-DP (RS-485 DATA+)
- net RS-RARM_RET: now also AX_R_ELBOW_PITCH.1 (GND), AX_R_SHOULDER_PITCH.1 (GND), AX_R_SHOULDER_ROLL.1 (GND); no longer AX_R_ELBOW_PITCH.LOG-RET (BRANCH RETURN), AX_R_SHOULDER_PITCH.LOG-RET (BRANCH RETURN), AX_R_SHOULDER_ROLL.LOG-RET (BRANCH RETURN)
- net RS-RARM_VDD: now also AX_R_ELBOW_PITCH.2 (VDD), AX_R_SHOULDER_PITCH.2 (VDD), AX_R_SHOULDER_ROLL.2 (VDD); no longer AX_R_ELBOW_PITCH.LOG-PWR (BRANCH VDD), AX_R_SHOULDER_PITCH.LOG-PWR (BRANCH VDD), AX_R_SHOULDER_ROLL.LOG-PWR (BRANCH VDD)
Other:
- note added: "NOTE 2: AX_* terminals use current official ROBOTIS actuator-side pin numbers; all LOG-*"
- note added: "identifiers remain functional ports, not physical connector or IC pins."
- note removed: "NOTE 2: All terminal identifiers beginning LOG- are functional ports, not manufacturer"
- note removed: "connector or package pin numbers."
Changed lines of the file:
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@@
 ) (text "NOTE 1: The segment shares data and branch power only among the listed axes; it does not" (exclude_from_sim no) (at 17.78 260.00 0)
       (effects (font (size 1.50 1.50)) (justify left bottom))) (text "        join any other protected branch VDD." (exclude_from_sim no) (at 17.78 265.50 0)
-      (effects (font (size 1.50 1.50)) (justify left bottom))) (text "NOTE 2: All terminal identifiers beginning LOG- are functional ports, not manufacturer" (exclude_from_sim no) (at 17.78 271.00 0)
-      (effects (font (size 1.50 1.50)) (justify left bottom))) (text "        connector or package pin numbers." (exclude_from_sim no) (at 17.78 276.50 0)
+      (effects (font (size 1.50 1.50)) (justify left bottom))) (text "NOTE 2: AX_* terminals use current official ROBOTIS actuator-side pin numbers; all LOG-*" (exclude_from_sim no) (at 17.78 271.00 0)
+      (effects (font (size 1.50 1.50)) (justify left bottom))) (text "        identifiers remain functional ports, not physical connector or IC pins." (exclude_from_sim no) (at 17.78 276.50 0)
       (effects (font (size 1.50 1.50)) (justify left bottom))) (text "NOTE 3: Termination, bias, actuator IDs, baud rate, cable length, waveform, latency, EMC," (exclude_from_sim no) (at 17.78 282.00 0)
       (effects (font (size 1.50 1.50)) (justify left bottom))) (text "        thermal and fault behavior remain unvalidated." (exclude_from_sim no) (at 17.78 287.50 0)
@@
       (property "Value" "ROBOTIS XM540-W270-R candidate" (at 144.78 144.78 0) (effects (font (size 1.50 1.50)) (hide yes)))
       (property "Footprint" "" (at 144.78 144.78 0) (effects (font (size 1.50 1.50)) (hide yes)))
-      (property "Datasheet" "https://emanual.robotis.com/docs/en/dxl/x/xm540-w270/" (at 144.78 144.78 0) (effects (font (size 1.50 1.50)) (hide yes)))
-      (property "Description" "Axis identity and protocol are allocated. Exact order code, actuator ID, physical connector pins, cable, branch current/protection and installed thermal/communication behavior remain selection and test work." (at 144.78 144.78 0) (effects (font (size 1.50 1.50)) (hide yes)))
-      (property "Status" "SELECTION REQUIRED - LOGICAL CONNECTIVITY ONLY" (at 144.78 160.48 0) (effects (font (size 1.50 1.50)) (justify bottom)))
-      (property "Evidence" "Official ROBOTIS e-Manual interface family checked 2026-08-14; no physical robot pin map released." (at 144.78 144.78 0) (effects (font (size 1.50 1.50)) (hide yes)))
+      (property "Datasheet" "https://docs.robotis.com/docs/dxl/model_reference/x_series/xm_series/xm540-w270/" (at 144.78 144.78 0) (effects (font (size 1.50 1.50)) (hide yes)))
+      (property "Description" "Axis identity, protocol and manufacturer actuator-side pins are allocated. Exact order code, actuator ID, cable assembly, controller-side connector, branch current/protection and installed thermal/communication behavior remain selection and test work." (at 144.78 144.78 0) (effects (font (size 1.50 1.50)) (hide yes)))
+      (property "Status" "ACTUATOR-SIDE PINOUT VERIFIED - HARNESS AND CONTROLLER SIDE SELECTION REQUIRED" (at 144.78 160.48 0) (effects (font (size 1.50 1.50)) (justify bottom)))
+      (property "Evidence" "Current official ROBOTIS Docs checked 2026-08-14: actuator-side 1=GND, 2=VDD and 3=DATA (TTL) or 3=DATA+/4=DATA- (RS-485)." (at 144.78 144.78 0) (effects (font (size 1.50 1.50)) (hide yes)))
       (property "Display" "ROBOTIS XM540-W270-R candidate" (at 107.95 131.28 0) (effects (font (size 1.50 1.50)) (justify left bottom)))
-      (pin "LOG-PWR")
-      (pin "LOG-RET")
-      (pin "LOG-DP")
-      (pin "LOG-DN")
+      (pin "2")
+      (pin "1")
+      (pin "3")
+      (pin "4")
       (instances (project "hr30-whole-body-electrical-p0.1" (path "/6dbc6f1c-d05b-56f0-8b51-042e5f8599ba/f7394767-33e6-5313-82f8-29f392882afa" (reference "AX_R_SHOULDER_PITCH") (unit 1)))))
 (symbol
@@
       (property "Value" "ROBOTIS XM430-W350-R candidate" (at 330.20 144.78 0) (effects (font (size 1.50 1.50)) (hide yes)))
       (property "Footprint" "" (at 330.20 144.78 0) (effects (font (size 1.50 1.50)) (hide yes)))
-      (property "Datasheet" "https://emanual.robotis.com/docs/en/dxl/x/xm430-w350/" (at 330.20 144.78 0) (effects (font (size 1.50 1.50)) (hide yes)))
-      (property "Description" "Axis identity and protocol are allocated. Exact order code, actuator ID, physical connector pins, cable, branch current/protection and installed thermal/communication behavior remain selection and test work." (at 330.20 144.78 0) (effects (font (size 1.50 1.50)) (hide yes)))
-      (property "Status" "SELECTION REQUIRED - LOGICAL CONNECTIVITY ONLY" (at 330.20 160.48 0) (effects (font (size 1.50 1.50)) (justify bottom)))
-      (property "Evidence" "Official ROBOTIS e-Manual interface family checked 2026-08-14; no physical robot pin map released." (at 330.20 144.78 0) (effects (font (size 1.50 1.50)) (hide yes)))
+      (property "Datasheet" "https://docs.robotis.com/docs/dxl/model_reference/x_series/xm_series/xm430-w350/" (at 330.20 144.78 0) (effects (font (size 1.50 1.50)) (hide yes)))
+      (property "Description" "Axis identity, protocol and manufacturer actuator-side pins are allocated. Exact order code, actuator ID, cable assembly, controller-side connector, branch current/protection and installed thermal/communication behavior remain selection and test work." (at 330.20 144.78 0) (effects (font (size 1.50 1.50)) (hide yes)))
+      (property "Status" "ACTUATOR-SIDE PINOUT VERIFIED - HARNESS AND CONTROLLER SIDE SELECTION REQUIRED" (at 330.20 160.48 0) (effects (font (size 1.50 1.50)) (justify bottom)))
+      (property "Evidence" "Current official ROBOTIS Docs checked 2026-08-14: actuator-side 1=GND, 2=VDD and 3=DATA (TTL) or 3=DATA+/4=DATA- (RS-485)." (at 330.20 144.78 0) (effects (font (size 1.50 1.50)) (hide yes)))
       (property "Display" "ROBOTIS XM430-W350-R candidate" (at 293.37 131.28 0) (effects (font (size 1.50 1.50)) (justify left bottom)))
-      (pin "LOG-PWR")
-      (pin "LOG-RET")
-      (pin "LOG-DP")
-      (pin "LOG-DN")
+      (pin "2")
+      (pin "1")
+      (pin "3")
+      (pin "4")
       (instances (project "hr30-whole-body-electrical-p0.1" (path "/6dbc6f1c-d05b-56f0-8b51-042e5f8599ba/f7394767-33e6-5313-82f8-29f392882afa" (reference "AX_R_SHOULDER_ROLL") (unit 1)))))
 (symbol
@@
       (property "Value" "ROBOTIS XM430-W350-R candidate" (at 240.03 209.55 0) (effects (font (size 1.50 1.50)) (hide yes)))
       (property "Footprint" "" (at 240.03 209.55 0) (effects (font (size 1.50 1.50)) (hide yes)))
-      (property "Datasheet" "https://emanual.robotis.com/docs/en/dxl/x/xm430-w350/" (at 240.03 209.55 0) (effects (font (size 1.50 1.50)) (hide yes)))
-      (property "Description" "Axis identity and protocol are allocated. Exact order code, actuator ID, physical connector pins, cable, branch current/protection and installed thermal/communication behavior remain selection and test work." (at 240.03 209.55 0) (effects (font (size 1.50 1.50)) (hide yes)))
-      (property "Status" "SELECTION REQUIRED - LOGICAL CONNECTIVITY ONLY" (at 240.03 225.25 0) (effects (font (size 1.50 1.50)) (justify bottom)))
-      (property "Evidence" "Official ROBOTIS e-Manual interface family checked 2026-08-14; no physical robot pin map released." (at 240.03 209.55 0) (effects (font (size 1.50 1.50)) (hide yes)))
+      (property "Datasheet" "https://docs.robotis.com/docs/dxl/model_reference/x_series/xm_series/xm430-w350/" (at 240.03 209.55 0) (effects (font (size 1.50 1.50)) (hide yes)))
+      (property "Description" "Axis identity, protocol and manufacturer actuator-side pins are allocated. Exact order code, actuator ID, cable assembly, controller-side connector, branch current/protection and installed thermal/communication behavior remain selection and test work." (at 240.03 209.55 0) (effects (font (size 1.50 1.50)) (hide yes)))
+      (property "Status" "ACTUATOR-SIDE PINOUT VERIFIED - HARNESS AND CONTROLLER SIDE SELECTION REQUIRED" (at 240.03 225.25 0) (effects (font (size 1.50 1.50)) (justify bottom)))
+      (property "Evidence" "Current official ROBOTIS Docs checked 2026-08-14: actuator-side 1=GND, 2=VDD and 3=DATA (TTL) or 3=DATA+/4=DATA- (RS-485)." (at 240.03 209.55 0) (effects (font (size 1.50 1.50)) (hide yes)))
       (property "Display" "ROBOTIS XM430-W350-R candidate" (at 203.20 196.05 0) (effects (font (size 1.50 1.50)) (justify left bottom)))
-      (pin "LOG-PWR")
-      (pin "LOG-RET")
-      (pin "LOG-DP")
-      (pin "LOG-DN")
+      (pin "2")
+      (pin "1")
+      (pin "3")
+      (pin "4")
       (instances (project "hr30-whole-body-electrical-p0.1" (path "/6dbc6f1c-d05b-56f0-8b51-042e5f8599ba/f7394767-33e6-5313-82f8-29f392882afa" (reference "AX_R_ELBOW_PITCH") (unit 1)))))
   (embedded_fonts no))
