File: hr30/whole-body-p0.1/electrical/kicad/hr30-whole-body-electrical-p0.1/10_left_distal_ttl.kicad_sch (KiCad schematic)
At the start: 4 parts

Commit message: Add HR-30 whole-body harness architecture
Parts:
- AX_L_GRIPPER, AX_L_WRIST_ROTATION: Evidence Official ROBOTIS e-Manual interface family checked 2026-08-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 -> Current official ROBOTIS Docs checked 2026-08-14: actuator-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; Status SELECTION REQUIRED - LOGICAL CONNECTIVITY ONLY -> ACTUATOR-SIDE PINOUT VERIFIED - HARNESS AND CONTROLLER SIDE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
Connections:
- net TTL-LDIST_DATA: now also AX_L_GRIPPER.3 (DATA), AX_L_WRIST_ROTATION.3 (DATA); no longer AX_L_GRIPPER.LOG-DATA (TTL HALF-DUPLEX DATA), AX_L_WRIST_ROTATION.LOG-DATA (TTL HALF-DUPLEX DATA)
- net TTL-LDIST_RET: now also AX_L_GRIPPER.1 (GND), AX_L_WRIST_ROTATION.1 (GND); no longer AX_L_GRIPPER.LOG-RET (BRANCH RETURN), AX_L_WRIST_ROTATION.LOG-RET (BRANCH RETURN)
- net TTL-LDIST_VDD: now also AX_L_GRIPPER.2 (VDD), AX_L_WRIST_ROTATION.2 (VDD); no longer AX_L_GRIPPER.LOG-PWR (BRANCH VDD), AX_L_WRIST_ROTATION.LOG-PWR (BRANCH VDD)
Other:
- note added: "NOTE 2: AX_* terminals use current official ROBOTIS actuator-side pin numbers; all LOG-*"
- note added: "identifiers remain functional ports, not physical connector or IC pins."
- note removed: "NOTE 2: All terminal identifiers beginning LOG- are functional ports, not manufacturer"
- note removed: "connector or package pin numbers."
Changed lines of the file:
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@@
 ) (text "NOTE 1: The segment shares data and branch power only among the listed axes; it does not" (exclude_from_sim no) (at 17.78 260.00 0)
       (effects (font (size 1.50 1.50)) (justify left bottom))) (text "        join any other protected branch VDD." (exclude_from_sim no) (at 17.78 265.50 0)
-      (effects (font (size 1.50 1.50)) (justify left bottom))) (text "NOTE 2: All terminal identifiers beginning LOG- are functional ports, not manufacturer" (exclude_from_sim no) (at 17.78 271.00 0)
-      (effects (font (size 1.50 1.50)) (justify left bottom))) (text "        connector or package pin numbers." (exclude_from_sim no) (at 17.78 276.50 0)
+      (effects (font (size 1.50 1.50)) (justify left bottom))) (text "NOTE 2: AX_* terminals use current official ROBOTIS actuator-side pin numbers; all LOG-*" (exclude_from_sim no) (at 17.78 271.00 0)
+      (effects (font (size 1.50 1.50)) (justify left bottom))) (text "        identifiers remain functional ports, not physical connector or IC pins." (exclude_from_sim no) (at 17.78 276.50 0)
       (effects (font (size 1.50 1.50)) (justify left bottom))) (text "NOTE 3: Termination, bias, actuator IDs, baud rate, cable length, waveform, latency, EMC," (exclude_from_sim no) (at 17.78 282.00 0)
       (effects (font (size 1.50 1.50)) (justify left bottom))) (text "        thermal and fault behavior remain unvalidated." (exclude_from_sim no) (at 17.78 287.50 0)
@@
       (property "Value" "ROBOTIS XC330-T288-T candidate" (at 144.78 175.26 0) (effects (font (size 1.50 1.50)) (hide yes)))
       (property "Footprint" "" (at 144.78 175.26 0) (effects (font (size 1.50 1.50)) (hide yes)))
-      (property "Datasheet" "https://emanual.robotis.com/docs/en/dxl/x/xc330-m288/" (at 144.78 175.26 0) (effects (font (size 1.50 1.50)) (hide yes)))
-      (property "Description" "Axis identity and protocol are allocated. Exact order code, actuator ID, physical connector pins, cable, branch current/protection and installed thermal/communication behavior remain selection and test work." (at 144.78 175.26 0) (effects (font (size 1.50 1.50)) (hide yes)))
-      (property "Status" "SELECTION REQUIRED - LOGICAL CONNECTIVITY ONLY" (at 144.78 190.96 0) (effects (font (size 1.50 1.50)) (justify bottom)))
-      (property "Evidence" "Official ROBOTIS e-Manual interface family checked 2026-08-14; no physical robot pin map released." (at 144.78 175.26 0) (effects (font (size 1.50 1.50)) (hide yes)))
+      (property "Datasheet" "https://docs.robotis.com/docs/dxl/model_reference/x_series/xc_series/xc330-t288/" (at 144.78 175.26 0) (effects (font (size 1.50 1.50)) (hide yes)))
+      (property "Description" "Axis identity, protocol and manufacturer actuator-side pins are allocated. Exact order code, actuator ID, cable assembly, controller-side connector, branch current/protection and installed thermal/communication behavior remain selection and test work." (at 144.78 175.26 0) (effects (font (size 1.50 1.50)) (hide yes)))
+      (property "Status" "ACTUATOR-SIDE PINOUT VERIFIED - HARNESS AND CONTROLLER SIDE SELECTION REQUIRED" (at 144.78 190.96 0) (effects (font (size 1.50 1.50)) (justify bottom)))
+      (property "Evidence" "Current official ROBOTIS Docs checked 2026-08-14: actuator-side 1=GND, 2=VDD and 3=DATA (TTL) or 3=DATA+/4=DATA- (RS-485)." (at 144.78 175.26 0) (effects (font (size 1.50 1.50)) (hide yes)))
       (property "Display" "ROBOTIS XC330-T288-T candidate" (at 107.95 161.76 0) (effects (font (size 1.50 1.50)) (justify left bottom)))
-      (pin "LOG-PWR")
-      (pin "LOG-RET")
-      (pin "LOG-DATA")
+      (pin "2")
+      (pin "1")
+      (pin "3")
       (instances (project "hr30-whole-body-electrical-p0.1" (path "/6dbc6f1c-d05b-56f0-8b51-042e5f8599ba/6dc96b4c-da73-57e4-b9d2-048189eb899f" (reference "AX_L_WRIST_ROTATION") (unit 1)))))
 (symbol
@@
       (property "Value" "ROBOTIS XC330-class compact candidate" (at 330.20 175.26 0) (effects (font (size 1.50 1.50)) (hide yes)))
       (property "Footprint" "" (at 330.20 175.26 0) (effects (font (size 1.50 1.50)) (hide yes)))
-      (property "Datasheet" "https://emanual.robotis.com/docs/en/dxl/x/xc330-m288/" (at 330.20 175.26 0) (effects (font (size 1.50 1.50)) (hide yes)))
-      (property "Description" "Axis identity and protocol are allocated. Exact order code, actuator ID, physical connector pins, cable, branch current/protection and installed thermal/communication behavior remain selection and test work." (at 330.20 175.26 0) (effects (font (size 1.50 1.50)) (hide yes)))
-      (property "Status" "SELECTION REQUIRED - LOGICAL CONNECTIVITY ONLY" (at 330.20 190.96 0) (effects (font (size 1.50 1.50)) (justify bottom)))
-      (property "Evidence" "Official ROBOTIS e-Manual interface family checked 2026-08-14; no physical robot pin map released." (at 330.20 175.26 0) (effects (font (size 1.50 1.50)) (hide yes)))
+      (property "Datasheet" "https://docs.robotis.com/docs/dxl/model_reference/x_series/xc_series/xc330-t288/" (at 330.20 175.26 0) (effects (font (size 1.50 1.50)) (hide yes)))
+      (property "Description" "Axis identity, protocol and manufacturer actuator-side pins are allocated. Exact order code, actuator ID, cable assembly, controller-side connector, branch current/protection and installed thermal/communication behavior remain selection and test work." (at 330.20 175.26 0) (effects (font (size 1.50 1.50)) (hide yes)))
+      (property "Status" "ACTUATOR-SIDE PINOUT VERIFIED - HARNESS AND CONTROLLER SIDE SELECTION REQUIRED" (at 330.20 190.96 0) (effects (font (size 1.50 1.50)) (justify bottom)))
+      (property "Evidence" "Current official ROBOTIS Docs checked 2026-08-14: actuator-side 1=GND, 2=VDD and 3=DATA (TTL) or 3=DATA+/4=DATA- (RS-485)." (at 330.20 175.26 0) (effects (font (size 1.50 1.50)) (hide yes)))
       (property "Display" "ROBOTIS XC330-class compact candidate" (at 293.37 161.76 0) (effects (font (size 1.50 1.50)) (justify left bottom)))
-      (pin "LOG-PWR")
-      (pin "LOG-RET")
-      (pin "LOG-DATA")
+      (pin "2")
+      (pin "1")
+      (pin "3")
       (instances (project "hr30-whole-body-electrical-p0.1" (path "/6dbc6f1c-d05b-56f0-8b51-042e5f8599ba/6dc96b4c-da73-57e4-b9d2-048189eb899f" (reference "AX_L_GRIPPER") (unit 1)))))
   (embedded_fonts no))
