File: hr30/whole-body-p0.1/electrical/kicad/hr30-whole-body-electrical-p0.1/12_head_ttl_sensors_hmi.kicad_sch (KiCad schematic)
At the start: 7 parts

Commit message: Add HR-30 whole-body harness architecture
Parts:
- AX_HEAD_PAN, AX_HEAD_TILT: Evidence Official ROBOTIS e-Manual interface family checked 2026-08-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 -> Current official ROBOTIS Docs checked 2026-08-14: actuator-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; Status SELECTION REQUIRED - LOGICAL CONNECTIVITY ONLY -> ACTUATOR-SIDE PINOUT VERIFIED - HARNESS AND CONTROLLER SIDE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
Connections:
- net TTL-HEAD_DATA: now also AX_HEAD_PAN.3 (DATA), AX_HEAD_TILT.3 (DATA); no longer AX_HEAD_PAN.LOG-DATA (TTL HALF-DUPLEX DATA), AX_HEAD_TILT.LOG-DATA (TTL HALF-DUPLEX DATA)
- net TTL-HEAD_RET: now also AX_HEAD_PAN.1 (GND), AX_HEAD_TILT.1 (GND); no longer AX_HEAD_PAN.LOG-RET (BRANCH RETURN), AX_HEAD_TILT.LOG-RET (BRANCH RETURN)
- net TTL-HEAD_VDD: now also AX_HEAD_PAN.2 (VDD), AX_HEAD_TILT.2 (VDD); no longer AX_HEAD_PAN.LOG-PWR (BRANCH VDD), AX_HEAD_TILT.LOG-PWR (BRANCH VDD)
Other:
- note added: "NOTE 2: AX_* terminals use current official ROBOTIS actuator-side pin numbers; all LOG-*"
- note added: "identifiers remain functional ports, not physical connector or IC pins."
- note removed: "NOTE 2: All terminal identifiers beginning LOG- are functional ports, not manufacturer"
- note removed: "connector or package pin numbers."
Changed lines of the file:
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@@
 ) (text "NOTE 1: The segment shares data and branch power only among the listed axes; it does not" (exclude_from_sim no) (at 17.78 260.00 0)
       (effects (font (size 1.50 1.50)) (justify left bottom))) (text "        join any other protected branch VDD." (exclude_from_sim no) (at 17.78 265.50 0)
-      (effects (font (size 1.50 1.50)) (justify left bottom))) (text "NOTE 2: All terminal identifiers beginning LOG- are functional ports, not manufacturer" (exclude_from_sim no) (at 17.78 271.00 0)
-      (effects (font (size 1.50 1.50)) (justify left bottom))) (text "        connector or package pin numbers." (exclude_from_sim no) (at 17.78 276.50 0)
+      (effects (font (size 1.50 1.50)) (justify left bottom))) (text "NOTE 2: AX_* terminals use current official ROBOTIS actuator-side pin numbers; all LOG-*" (exclude_from_sim no) (at 17.78 271.00 0)
+      (effects (font (size 1.50 1.50)) (justify left bottom))) (text "        identifiers remain functional ports, not physical connector or IC pins." (exclude_from_sim no) (at 17.78 276.50 0)
       (effects (font (size 1.50 1.50)) (justify left bottom))) (text "NOTE 3: Termination, bias, actuator IDs, baud rate, cable length, waveform, latency, EMC," (exclude_from_sim no) (at 17.78 282.00 0)
       (effects (font (size 1.50 1.50)) (justify left bottom))) (text "        thermal and fault behavior remain unvalidated." (exclude_from_sim no) (at 17.78 287.50 0)
@@
       (property "Value" "ROBOTIS XC330-class compact X-series candidate" (at 144.78 175.26 0) (effects (font (size 1.50 1.50)) (hide yes)))
       (property "Footprint" "" (at 144.78 175.26 0) (effects (font (size 1.50 1.50)) (hide yes)))
-      (property "Datasheet" "https://emanual.robotis.com/docs/en/dxl/x/xc330-m288/" (at 144.78 175.26 0) (effects (font (size 1.50 1.50)) (hide yes)))
-      (property "Description" "Axis identity and protocol are allocated. Exact order code, actuator ID, physical connector pins, cable, branch current/protection and installed thermal/communication behavior remain selection and test work." (at 144.78 175.26 0) (effects (font (size 1.50 1.50)) (hide yes)))
-      (property "Status" "SELECTION REQUIRED - LOGICAL CONNECTIVITY ONLY" (at 144.78 190.96 0) (effects (font (size 1.50 1.50)) (justify bottom)))
-      (property "Evidence" "Official ROBOTIS e-Manual interface family checked 2026-08-14; no physical robot pin map released." (at 144.78 175.26 0) (effects (font (size 1.50 1.50)) (hide yes)))
+      (property "Datasheet" "https://docs.robotis.com/docs/dxl/model_reference/x_series/xc_series/xc330-t288/" (at 144.78 175.26 0) (effects (font (size 1.50 1.50)) (hide yes)))
+      (property "Description" "Axis identity, protocol and manufacturer actuator-side pins are allocated. Exact order code, actuator ID, cable assembly, controller-side connector, branch current/protection and installed thermal/communication behavior remain selection and test work." (at 144.78 175.26 0) (effects (font (size 1.50 1.50)) (hide yes)))
+      (property "Status" "ACTUATOR-SIDE PINOUT VERIFIED - HARNESS AND CONTROLLER SIDE SELECTION REQUIRED" (at 144.78 190.96 0) (effects (font (size 1.50 1.50)) (justify bottom)))
+      (property "Evidence" "Current official ROBOTIS Docs checked 2026-08-14: actuator-side 1=GND, 2=VDD and 3=DATA (TTL) or 3=DATA+/4=DATA- (RS-485)." (at 144.78 175.26 0) (effects (font (size 1.50 1.50)) (hide yes)))
       (property "Display" "ROBOTIS XC330-class compact X-series candidate" (at 107.95 161.76 0) (effects (font (size 1.50 1.50)) (justify left bottom)))
-      (pin "LOG-PWR")
-      (pin "LOG-RET")
-      (pin "LOG-DATA")
+      (pin "2")
+      (pin "1")
+      (pin "3")
       (instances (project "hr30-whole-body-electrical-p0.1" (path "/6dbc6f1c-d05b-56f0-8b51-042e5f8599ba/2c0d00f0-93a8-543c-ac01-83696100d78d" (reference "AX_HEAD_PAN") (unit 1)))))
 (symbol
@@
       (property "Value" "ROBOTIS XC330-class compact X-series candidate" (at 330.20 175.26 0) (effects (font (size 1.50 1.50)) (hide yes)))
       (property "Footprint" "" (at 330.20 175.26 0) (effects (font (size 1.50 1.50)) (hide yes)))
-      (property "Datasheet" "https://emanual.robotis.com/docs/en/dxl/x/xc330-m288/" (at 330.20 175.26 0) (effects (font (size 1.50 1.50)) (hide yes)))
-      (property "Description" "Axis identity and protocol are allocated. Exact order code, actuator ID, physical connector pins, cable, branch current/protection and installed thermal/communication behavior remain selection and test work." (at 330.20 175.26 0) (effects (font (size 1.50 1.50)) (hide yes)))
-      (property "Status" "SELECTION REQUIRED - LOGICAL CONNECTIVITY ONLY" (at 330.20 190.96 0) (effects (font (size 1.50 1.50)) (justify bottom)))
-      (property "Evidence" "Official ROBOTIS e-Manual interface family checked 2026-08-14; no physical robot pin map released." (at 330.20 175.26 0) (effects (font (size 1.50 1.50)) (hide yes)))
+      (property "Datasheet" "https://docs.robotis.com/docs/dxl/model_reference/x_series/xc_series/xc330-t288/" (at 330.20 175.26 0) (effects (font (size 1.50 1.50)) (hide yes)))
+      (property "Description" "Axis identity, protocol and manufacturer actuator-side pins are allocated. Exact order code, actuator ID, cable assembly, controller-side connector, branch current/protection and installed thermal/communication behavior remain selection and test work." (at 330.20 175.26 0) (effects (font (size 1.50 1.50)) (hide yes)))
+      (property "Status" "ACTUATOR-SIDE PINOUT VERIFIED - HARNESS AND CONTROLLER SIDE SELECTION REQUIRED" (at 330.20 190.96 0) (effects (font (size 1.50 1.50)) (justify bottom)))
+      (property "Evidence" "Current official ROBOTIS Docs checked 2026-08-14: actuator-side 1=GND, 2=VDD and 3=DATA (TTL) or 3=DATA+/4=DATA- (RS-485)." (at 330.20 175.26 0) (effects (font (size 1.50 1.50)) (hide yes)))
       (property "Display" "ROBOTIS XC330-class compact X-series candidate" (at 293.37 161.76 0) (effects (font (size 1.50 1.50)) (justify left bottom)))
-      (pin "LOG-PWR")
-      (pin "LOG-RET")
-      (pin "LOG-DATA")
+      (pin "2")
+      (pin "1")
+      (pin "3")
       (instances (project "hr30-whole-body-electrical-p0.1" (path "/6dbc6f1c-d05b-56f0-8b51-042e5f8599ba/2c0d00f0-93a8-543c-ac01-83696100d78d" (reference "AX_HEAD_TILT") (unit 1)))))
 (symbol

Commit message: Expand HR-30 whole-body electrical architecture
Parts:
- removed HMI1: FACE DISPLAY / MICROPHONES / SPEAKERS - SELECTION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, symbol PBV3:HMI1
- added AMP1: AUDIO AMPLIFIER - SELECTION REQUIRED, symbol PBV3:AMP1
- added DISP1: FACE DISPLAY - SELECTION REQUIRED, symbol PBV3:DISP1
- added FAN1: HEAD COOLING FAN - SELECTION REQUIRED, symbol PBV3:FAN1
- added HPWR1: PROTECTED HEAD AUXILIARY DISTRIBUTION - DESIGN RE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, symbol PBV3:HPWR1
- added MIC1: MICROPHONE ARRAY - SELECTION REQUIRED, symbol PBV3:MIC1
- added SPK1: LEFT SPEAKER - SELECTION REQUIRED, symbol PBV3:SPK1
- added SPK2: RIGHT SPEAKER - SELECTION REQUIRED, symbol PBV3:SPK2
Connections:
- net HMI_SENSOR_IPC renamed HEAD_CAM_L_IPC
- net HEAD_CAM_L_IPC: no longer CAM2.LOG-IPC (VISION IPC)
- new net AUX_0V: HPWR1.LOG-RET-IN (AUXILIARY RETURN)
- new net AUX_5V_SAFE: HPWR1.LOG-IN (AUXILIARY 5 V INPUT)
- new net HEAD_0V: AMP1.LOG-RET (RETURN), CAM1.LOG-RET (RETURN), CAM2.LOG-RET (RETURN), DISP1.LOG-RET (RETURN), FAN1.LOG-RET (RETURN), HPWR1.LOG-RET-OUT (HEAD RETURN), MIC1.LOG-RET (RETURN)
- new net HEAD_5V: AMP1.LOG-5V (5 V POWER), CAM1.LOG-5V (5 V POWER), CAM2.LOG-5V (5 V POWER), DISP1.LOG-5V (5 V POWER), FAN1.LOG-5V (5 V POWER), HPWR1.LOG-OUT (HEAD 5 V), MIC1.LOG-5V (5 V POWER)
- new net HEAD_AUDIO_IPC: AMP1.LOG-IN (AUDIO INPUT IPC)
- new net HEAD_CAM_R_IPC: CAM2.LOG-IPC (VISION IPC)
- new net HEAD_DISPLAY_IPC: DISP1.LOG-IPC (DISPLAY IPC)
- new net HEAD_FAN_PWM: FAN1.LOG-PWM (PWM)
- new net HEAD_FAN_TACH: FAN1.LOG-TACH (TACHOMETER)
- new net HEAD_MIC_IPC: MIC1.LOG-IPC (AUDIO INPUT IPC)
- new net HEAD_TOUCH_IPC: DISP1.LOG-TOUCH (TOUCH IPC)
- new net SPK_L_NEG: AMP1.LOG-LN (LEFT SPEAKER -), SPK1.LOG-N (SPEAKER -)
- new net SPK_L_POS: AMP1.LOG-LP (LEFT SPEAKER +), SPK1.LOG-P (SPEAKER +)
- new net SPK_R_NEG: AMP1.LOG-RN (RIGHT SPEAKER -), SPK2.LOG-N (SPEAKER -)
- new net SPK_R_POS: AMP1.LOG-RP (RIGHT SPEAKER +), SPK2.LOG-P (SPEAKER +)
Other:
- note added: "12 Head TTL, cameras, face display, audio and cooling"
- note added: "W12016"
- note added: "W12017"
- note added: "W12018"
- note added: "W12019"
- note added: "W12020"
- note added: "W12021"
- note added: "W12022"
- note added: "W12023"
- note added: "W12024"
- note added: "W12025"
- note added: "W12026"
- note added: "W12027"
- note added: "W12028"
- note added: "W12029"
- note added: "W12030"
- note added: "W12031"
- note added: "W12032"
- note added: "W12033"
- note added: "W12034"
- note added: "W12035"
- note added: "W12036"
- note added: "W12037"
- note added: "W12038"
- note added: "W12039"
- note added: "W12040"
- note added: "W12041"
- note added: "W12042"
- note added: "W12043"
- note added: "W12044"
- note removed: "12 Head TTL, sensing, display and audio"
