File: hr30/whole-body-p0.1/electrical/kicad/hr30-whole-body-electrical-p0.1/02_estop_permit_contactors.kicad_sch (KiCad schematic)
At the start: 5 parts, among them K1 DC CONTACTOR 1 WITH MIRROR CO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, K2 DC CONTACTOR 2 WITH MIRROR CO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

Commit message: Correct HR-30 whole-body electrical architecture
Parts:
- added WD_INH1: ORDINARY WATCHDOG INHIBIT INTERFACE - DESIGN REQU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, symbol PBV3:WD_INH1
- K1: value DC CONTACTOR 1 WITH MIRROR CONTACT - SELECTION REQUIRED -> SENSATA GIGAVAC GV12-FAMILY DC CONTACTOR 1 CANDIDATE; Display DC CONTACTOR 1 WITH MIRROR CONTACT - SELECTION REQUIRED -> SENSATA GIGAVAC GV12-FAMILY DC CONTACTOR 1 CANDIDATE
- K2: value DC CONTACTOR 2 WITH MIRROR CONTACT - SELECTION REQUIRED -> SENSATA GIGAVAC GV12-FAMILY DC CONTACTOR 2 CANDIDATE; Display DC CONTACTOR 2 WITH MIRROR CONTACT - SELECTION REQUIRED -> SENSATA GIGAVAC GV12-FAMILY DC CONTACTOR 2 CANDIDATE
- S0: value DUAL-CHANNEL E-STOP DEVICE - SELECTION REQUIRED -> IDEC XW DUAL-NC E-STOP FAMILY CANDIDATE - EXACT ORDER CODE REQUIRED; Display DUAL-CHANNEL E-STOP DEVICE - SELECTION REQUIRED -> IDEC XW DUAL-NC E-STOP FAMILY CANDIDATE - EXACT ORDER CODE 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
- S1: value MONITORED MANUAL RESET DEVICE - SELECTION REQUIRED -> IDEC HW1B-M1F11-G MANUAL RESET CANDIDATE; Display MONITORED MANUAL RESET DEVICE - SELECTION REQUIRED -> IDEC HW1B-M1F11-G MANUAL RESET CANDIDATE
- SR1: value SAFETY CONTROL / EDM FUNCTION - APPLICATION SELECTION REQUIRED -> PILZ PNOZ s4 750104 SAFETY-RELAY CANDIDATE - APPLICATION OPEN; Display SAFETY CONTROL / EDM FUNCTION - APPLICATION SELECTION REQUI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 -> PILZ PNOZ s4 750104 SAFETY-RELAY CANDIDATE - APPLICATION OP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; Evidence (none) -> Pilz manual 21396-EN-23 dated 2026-06-22; accessed 2026-08-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; Status SELECTION REQUIRED - LOGICAL CONNECTIVITY ONLY -> SAFETY-RELAY CANDIDATE - NO FUNCTIONAL-SAFETY APPROVAL
Connections:
- net SAFETY_PERMIT_HARDWIRED: no longer K1.LOG-COIL (COIL PERMIT), K2.LOG-COIL (COIL PERMIT)
- net ACT_14V8_SAFE renamed TETHER_MAIN_POS
- net CONTACTOR_POS_IN renamed PANEL_DC_POS_RAW
- net EDM_K1 renamed EDM_K1_AUX
- net EDM_K1_AUX: now also K1.LOG-AUX (MECHANICALLY LINKED AUXILIARY CANDIDATE); no longer K1.LOG-MIR (MIRROR / EDM)
- net EDM_K2 renamed EDM_K2_AUX
- net EDM_K2_AUX: now also K2.LOG-AUX (MECHANICALLY LINKED AUXILIARY CANDIDATE); no longer K2.LOG-MIR (MIRROR / EDM)
- new net SAFETY_0V: K1.LOG-COIL-N (COIL RETURN), K2.LOG-COIL-N (COIL RETURN), SR1.LOG-0V (CONTROL RETURN)
- new net SAFETY_24V: SR1.LOG-24V (24 V CONTROL)
- new net SAFETY_OUT_K1: K1.LOG-COIL-P (COIL POSITIVE), SR1.LOG-OUT1 (SAFETY OUTPUT TO K1)
- new net SAFETY_OUT_K2: K2.LOG-COIL-P (COIL POSITIVE), SR1.LOG-OUT2 (SAFETY OUTPUT TO K2)
- new net WATCHDOG_INHIBIT_OK: SR1.LOG-WD (ORDINARY WATCHDOG INHIBIT), WD_INH1.LOG-OUT (FAIL-LOW INHIBIT ELIGIBILITY)
- new net WD_PERMIT_REQUEST: WD_INH1.LOG-IN (WATCHDOG REQUEST)
Other:
- note added: "W2025"
- note added: "W2026"
- note added: "W2027"
- note added: "W2028"
- note added: "W2029"
- note added: "W2030"
- note added: "W2031"
- note added: "W2032"
- note added: "W2033"
- moved on the sheet: S0, S1
