File: hr30/whole-body-p0.1/electrical/kicad/hr30-whole-body-electrical-p0.1/07_left_leg_rs485.kicad_sch (KiCad schematic)
At the start: 8 parts

Commit message: Correct HR-30 whole-body electrical architecture
Parts:
- removed PBR_RS_LLEG: RS-LLEG BRANCH PROTECTION / TELEMETRY - SELECTION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, symbol PBV3:PBR_RS_LLEG
- added PBR_L_ANKLE_PITCH: L_ANKLE_PITCH INDIVIDUAL PROTECTION / TELEMETRY -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, symbol PBV3:PBR_L_ANKLE_PITCH
- added PBR_L_ANKLE_ROLL: L_ANKLE_ROLL INDIVIDUAL PROTECTION / TELEMETRY - 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, symbol PBV3:PBR_L_ANKLE_ROLL
- added PBR_L_HIP_PITCH: L_HIP_PITCH INDIVIDUAL PROTECTION / TELEMETRY - S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, symbol PBV3:PBR_L_HIP_PITCH
- added PBR_L_HIP_ROLL: L_HIP_ROLL INDIVIDUAL PROTECTION / TELEMETRY - SE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, symbol PBV3:PBR_L_HIP_ROLL
- added PBR_L_HIP_YAW: L_HIP_YAW INDIVIDUAL PROTECTION / TELEMETRY - SEL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, symbol PBV3:PBR_L_HIP_YAW
- added PBR_L_KNEE_PITCH: L_KNEE_PITCH INDIVIDUAL PROTECTION / TELEMETRY - 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, symbol PBV3:PBR_L_KNEE_PITCH
- AX_L_ANKLE_PITCH, AX_L_ANKLE_ROLL, AX_L_HIP_PITCH, AX_L_HIP_ROLL, AX_L_HIP_YAW, AX_L_KNEE_PITCH: Status ACTUATOR-SIDE PINOUT VERIFIED - HARNESS AND CONTROLLER SIDE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 -> (none)
- PORT_RS_LLEG: Status SELECTION REQUIRED - LOGICAL CONNECTIVITY ONLY -> (none)
Connections:
- net ACT_0V_CONTROLLED: now also PBR_L_ANKLE_PITCH.LOG-RET-IN (SOURCE RETURN), PBR_L_ANKLE_ROLL.LOG-RET-IN (SOURCE RETURN), PBR_L_HIP_PITCH.LOG-RET-IN (SOURCE RETURN), PBR_L_HIP_ROLL.LOG-RET-IN (SOURCE RETURN), PBR_L_HIP_YAW.LOG-RET-IN (SOURCE RETURN), PBR_L_KNEE_PITCH.LOG-RET-IN (SOURCE RETURN)
- net RS-LLEG_RET: now also PBR_L_ANKLE_PITCH.LOG-RET-OUT (ACTUATOR / DATA REFERENCE), PBR_L_ANKLE_ROLL.LOG-RET-OUT (ACTUATOR / DATA REFERENCE), PBR_L_HIP_PITCH.LOG-RET-OUT (ACTUATOR / DATA REFERENCE), PBR_L_HIP_ROLL.LOG-RET-OUT (ACTUATOR / DATA REFERENCE), PBR_L_HIP_YAW.LOG-RET-OUT (ACTUATOR / DATA REFERENCE), PBR_L_KNEE_PITCH.LOG-RET-OUT (ACTUATOR / DATA REFERENCE)
- removed net RS-LLEG_VDD: AX_L_ANKLE_PITCH.2 (VDD), AX_L_ANKLE_ROLL.2 (VDD), AX_L_HIP_PITCH.2 (VDD), AX_L_HIP_ROLL.2 (VDD), AX_L_HIP_YAW.2 (VDD), AX_L_KNEE_PITCH.2 (VDD)
- new net ACT_MAIN_SAFE_12V: PBR_L_ANKLE_PITCH.LOG-IN (INTERRUPTED SOURCE), PBR_L_ANKLE_ROLL.LOG-IN (INTERRUPTED SOURCE), PBR_L_HIP_PITCH.LOG-IN (INTERRUPTED SOURCE), PBR_L_HIP_ROLL.LOG-IN (INTERRUPTED SOURCE), PBR_L_HIP_YAW.LOG-IN (INTERRUPTED SOURCE), PBR_L_KNEE_PITCH.LOG-IN (INTERRUPTED SOURCE)
- new net L_ANKLE_PITCH_VDD: AX_L_ANKLE_PITCH.2 (VDD), PBR_L_ANKLE_PITCH.LOG-OUT (PROTECTED ACTUATOR VDD)
- new net L_ANKLE_ROLL_VDD: AX_L_ANKLE_ROLL.2 (VDD), PBR_L_ANKLE_ROLL.LOG-OUT (PROTECTED ACTUATOR VDD)
- new net L_HIP_PITCH_VDD: AX_L_HIP_PITCH.2 (VDD), PBR_L_HIP_PITCH.LOG-OUT (PROTECTED ACTUATOR VDD)
- new net L_HIP_ROLL_VDD: AX_L_HIP_ROLL.2 (VDD), PBR_L_HIP_ROLL.LOG-OUT (PROTECTED ACTUATOR VDD)
- new net L_HIP_YAW_VDD: AX_L_HIP_YAW.2 (VDD), PBR_L_HIP_YAW.LOG-OUT (PROTECTED ACTUATOR VDD)
- new net L_KNEE_PITCH_VDD: AX_L_KNEE_PITCH.2 (VDD), PBR_L_KNEE_PITCH.LOG-OUT (PROTECTED ACTUATOR VDD)
- no-connect marks 1 -> 6
Other:
- note added: "07 Left-leg RS-485 data bus and individual feeds"
- note added: "Connected RS-LLEG data-only segment and one separately protected power feed per actuator."
- note added: "W7032"
- note added: "W7033"
- note added: "W7034"
- note added: "W7035"
- note added: "W7036"
- note added: "W7037"
- note added: "W7038"
- note added: "W7039"
- note added: "W7040"
- note added: "W7041"
- note added: "W7042"
- note added: "W7043"
- note added: "W7044"
- note added: "W7045"
- note added: "W7046"
- note added: "W7047"
- note added: "W7048"
- note added: "W7049"
- note added: "W7050"
- note added: "W7051"
- note removed: "07 Left-leg RS-485 and protected branch"
- note removed: "Connected RS-LLEG data segment and separately protected actuator-power branch."
- note removed: "NOTE 1: The segment shares data and branch power only among the listed axes; it does not"
- note removed: "NOTE 2: AX_* terminals use current official ROBOTIS actuator-side pin numbers; all LOG-*"
- note removed: "NOTE 3: Termination, bias, actuator IDs, baud rate, cable length, waveform, latency, EMC,"
- note removed: "identifiers remain functional ports, not physical connector or IC pins."
- note removed: "join any other protected branch VDD."
- note removed: "thermal and fault behavior remain unvalidated."
- moved on the sheet: AX_L_ANKLE_PITCH, AX_L_ANKLE_ROLL, AX_L_HIP_PITCH, AX_L_HIP_ROLL, AX_L_HIP_YAW, AX_L_KNEE_PITCH, PORT_RS_LLEG
