File: hr30/whole-body-p0.1/electrical/kicad/hr30-whole-body-electrical-p0.1/08_right_leg_rs485.kicad_sch (KiCad schematic)
At the start: 8 parts

Commit message: Correct HR-30 whole-body electrical architecture
Parts:
- removed PBR_RS_RLEG: RS-RLEG BRANCH PROTECTION / TELEMETRY - SELECTION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, symbol PBV3:PBR_RS_RLEG
- added PBR_R_ANKLE_PITCH: R_ANKLE_PITCH INDIVIDUAL PROTECTION / TELEMETRY -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, symbol PBV3:PBR_R_ANKLE_PITCH
- added PBR_R_ANKLE_ROLL: R_ANKLE_ROLL INDIVIDUAL PROTECTION / TELEMETRY - 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, symbol PBV3:PBR_R_ANKLE_ROLL
- added PBR_R_HIP_PITCH: R_HIP_PITCH INDIVIDUAL PROTECTION / TELEMETRY - S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, symbol PBV3:PBR_R_HIP_PITCH
- added PBR_R_HIP_ROLL: R_HIP_ROLL INDIVIDUAL PROTECTION / TELEMETRY - SE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, symbol PBV3:PBR_R_HIP_ROLL
- added PBR_R_HIP_YAW: R_HIP_YAW INDIVIDUAL PROTECTION / TELEMETRY - SEL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, symbol PBV3:PBR_R_HIP_YAW
- added PBR_R_KNEE_PITCH: R_KNEE_PITCH INDIVIDUAL PROTECTION / TELEMETRY - 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, symbol PBV3:PBR_R_KNEE_PITCH
- AX_R_ANKLE_PITCH, AX_R_ANKLE_ROLL, AX_R_HIP_PITCH, AX_R_HIP_ROLL, AX_R_HIP_YAW, AX_R_KNEE_PITCH: Status ACTUATOR-SIDE PINOUT VERIFIED - HARNESS AND CONTROLLER SIDE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 -> (none)
- PORT_RS_RLEG: Status SELECTION REQUIRED - LOGICAL CONNECTIVITY ONLY -> (none)
Connections:
- net ACT_0V_CONTROLLED: now also PBR_R_ANKLE_PITCH.LOG-RET-IN (SOURCE RETURN), PBR_R_ANKLE_ROLL.LOG-RET-IN (SOURCE RETURN), PBR_R_HIP_PITCH.LOG-RET-IN (SOURCE RETURN), PBR_R_HIP_ROLL.LOG-RET-IN (SOURCE RETURN), PBR_R_HIP_YAW.LOG-RET-IN (SOURCE RETURN), PBR_R_KNEE_PITCH.LOG-RET-IN (SOURCE RETURN)
- net RS-RLEG_RET: now also PBR_R_ANKLE_PITCH.LOG-RET-OUT (ACTUATOR / DATA REFERENCE), PBR_R_ANKLE_ROLL.LOG-RET-OUT (ACTUATOR / DATA REFERENCE), PBR_R_HIP_PITCH.LOG-RET-OUT (ACTUATOR / DATA REFERENCE), PBR_R_HIP_ROLL.LOG-RET-OUT (ACTUATOR / DATA REFERENCE), PBR_R_HIP_YAW.LOG-RET-OUT (ACTUATOR / DATA REFERENCE), PBR_R_KNEE_PITCH.LOG-RET-OUT (ACTUATOR / DATA REFERENCE)
- removed net RS-RLEG_VDD: AX_R_ANKLE_PITCH.2 (VDD), AX_R_ANKLE_ROLL.2 (VDD), AX_R_HIP_PITCH.2 (VDD), AX_R_HIP_ROLL.2 (VDD), AX_R_HIP_YAW.2 (VDD), AX_R_KNEE_PITCH.2 (VDD)
- new net ACT_MAIN_SAFE_12V: PBR_R_ANKLE_PITCH.LOG-IN (INTERRUPTED SOURCE), PBR_R_ANKLE_ROLL.LOG-IN (INTERRUPTED SOURCE), PBR_R_HIP_PITCH.LOG-IN (INTERRUPTED SOURCE), PBR_R_HIP_ROLL.LOG-IN (INTERRUPTED SOURCE), PBR_R_HIP_YAW.LOG-IN (INTERRUPTED SOURCE), PBR_R_KNEE_PITCH.LOG-IN (INTERRUPTED SOURCE)
- new net R_ANKLE_PITCH_VDD: AX_R_ANKLE_PITCH.2 (VDD), PBR_R_ANKLE_PITCH.LOG-OUT (PROTECTED ACTUATOR VDD)
- new net R_ANKLE_ROLL_VDD: AX_R_ANKLE_ROLL.2 (VDD), PBR_R_ANKLE_ROLL.LOG-OUT (PROTECTED ACTUATOR VDD)
- new net R_HIP_PITCH_VDD: AX_R_HIP_PITCH.2 (VDD), PBR_R_HIP_PITCH.LOG-OUT (PROTECTED ACTUATOR VDD)
- new net R_HIP_ROLL_VDD: AX_R_HIP_ROLL.2 (VDD), PBR_R_HIP_ROLL.LOG-OUT (PROTECTED ACTUATOR VDD)
- new net R_HIP_YAW_VDD: AX_R_HIP_YAW.2 (VDD), PBR_R_HIP_YAW.LOG-OUT (PROTECTED ACTUATOR VDD)
- new net R_KNEE_PITCH_VDD: AX_R_KNEE_PITCH.2 (VDD), PBR_R_KNEE_PITCH.LOG-OUT (PROTECTED ACTUATOR VDD)
- no-connect marks 1 -> 6
Other:
- note added: "08 Right-leg RS-485 data bus and individual feeds"
- note added: "Connected RS-RLEG data-only segment and one separately protected power feed per actuator."
- note added: "W8032"
- note added: "W8033"
- note added: "W8034"
- note added: "W8035"
- note added: "W8036"
- note added: "W8037"
- note added: "W8038"
- note added: "W8039"
- note added: "W8040"
- note added: "W8041"
- note added: "W8042"
- note added: "W8043"
- note added: "W8044"
- note added: "W8045"
- note added: "W8046"
- note added: "W8047"
- note added: "W8048"
- note added: "W8049"
- note added: "W8050"
- note added: "W8051"
- note removed: "08 Right-leg RS-485 and protected branch"
- note removed: "Connected RS-RLEG data segment and separately protected actuator-power branch."
- note removed: "NOTE 1: The segment shares data and branch power only among the listed axes; it does not"
- note removed: "NOTE 2: AX_* terminals use current official ROBOTIS actuator-side pin numbers; all LOG-*"
- note removed: "NOTE 3: Termination, bias, actuator IDs, baud rate, cable length, waveform, latency, EMC,"
- note removed: "identifiers remain functional ports, not physical connector or IC pins."
- note removed: "join any other protected branch VDD."
- note removed: "thermal and fault behavior remain unvalidated."
- moved on the sheet: AX_R_ANKLE_PITCH, AX_R_ANKLE_ROLL, AX_R_HIP_PITCH, AX_R_HIP_ROLL, AX_R_HIP_YAW, AX_R_KNEE_PITCH, PORT_RS_RLEG
