File: hr30/whole-body-p0.1/electrical/kicad/hr30-whole-body-electrical-p0.1/12_left_distal_ttl.kicad_sch (KiCad schematic)
At the start: 4 parts

Commit message: Correct HR-30 whole-body electrical architecture
Parts:
- removed PBR_TTL_LDIST: TTL-LDIST BRANCH PROTECTION / TELEMETRY - SELECTI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, symbol PBV3:PBR_TTL_LDIST
- added PBR_L_GRIPPER: L_GRIPPER INDIVIDUAL PROTECTION / TELEMETRY - SEL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, symbol PBV3:PBR_L_GRIPPER
- added PBR_L_WRIST_ROTATION: L_WRIST_ROTATION INDIVIDUAL PROTECTION / TELEMETR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, symbol PBV3:PBR_L_WRIST_ROTATION
Connections:
- net ACT_0V_CONTROLLED: now also PBR_L_GRIPPER.LOG-RET-IN (SOURCE RETURN), PBR_L_WRIST_ROTATION.LOG-RET-IN (SOURCE RETURN)
- net TTL-LDIST_RET: now also PBR_L_GRIPPER.LOG-RET-OUT (ACTUATOR / DATA REFERENCE), PBR_L_WRIST_ROTATION.LOG-RET-OUT (ACTUATOR / DATA REFERENCE)
- net TTL-LDIST_VDD renamed L_GRIPPER_VDD
- net L_GRIPPER_VDD: now also PBR_L_GRIPPER.LOG-OUT (PROTECTED ACTUATOR VDD); no longer AX_L_WRIST_ROTATION.2 (VDD)
- new net L_WRIST_ROTATION_VDD: AX_L_WRIST_ROTATION.2 (VDD), PBR_L_WRIST_ROTATION.LOG-OUT (PROTECTED ACTUATOR VDD)
- new net TTL_LDIST_SAFE_9V: PBR_L_GRIPPER.LOG-IN (INTERRUPTED SOURCE), PBR_L_WRIST_ROTATION.LOG-IN (INTERRUPTED SOURCE)
- no-connect marks 1 -> 2
Other:
- note added: "12 Left wrist/gripper TTL data bus and individual feeds"
- note added: "Connected TTL-LDIST data-only segment and one separately protected power feed per actuator."
- note added: "IDs, baud rate, cable, EMC, thermal and fault behavior remain unvalidated."
- note added: "NOTE 1: The listed axes share only data and reference. Each pin-2 VDD has a distinct"
- note added: "NOTE 3: A custom/de-pinned data-only harness or breakout is SELECTION REQUIRED. Termination,"
- note added: "W12013"
- note added: "W12014"
- note added: "W12015"
- note added: "W12016"
- note added: "protected feed; no standard VDD-carrying daisy cable may parallel those feeds."
- note removed: "12 Left wrist/gripper TTL and protected branch"
- note removed: "Connected TTL-LDIST data segment and separately protected actuator-power branch."
- note removed: "NOTE 1: The segment shares data and branch power only among the listed axes; it does not"
- note removed: "NOTE 3: Termination, bias, actuator IDs, baud rate, cable length, waveform, latency, EMC,"
- note removed: "join any other protected branch VDD."
- note removed: "thermal and fault behavior remain unvalidated."
- moved on the sheet: AX_L_GRIPPER, AX_L_WRIST_ROTATION, PORT_TTL_LDIST
