File: hr30/whole-body-p0.1/electrical/kicad/hr30-whole-body-electrical-p0.1/10_right_arm_rs485.kicad_sch (KiCad schematic)
At the start: 5 parts

Commit message: Correct HR-30 whole-body electrical architecture
Parts:
- removed PBR_RS_RARM: RS-RARM BRANCH PROTECTION / TELEMETRY - SELECTION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, symbol PBV3:PBR_RS_RARM
- added PBR_R_ELBOW_PITCH: R_ELBOW_PITCH INDIVIDUAL PROTECTION / TELEMETRY -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, symbol PBV3:PBR_R_ELBOW_PITCH
- added PBR_R_SHOULDER_PITCH: R_SHOULDER_PITCH INDIVIDUAL PROTECTION / TELEMETR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, symbol PBV3:PBR_R_SHOULDER_PITCH
- added PBR_R_SHOULDER_ROLL: R_SHOULDER_ROLL INDIVIDUAL PROTECTION / TELEMETRY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, symbol PBV3:PBR_R_SHOULDER_ROLL
Connections:
- net ACT_0V_CONTROLLED: now also PBR_R_ELBOW_PITCH.LOG-RET-IN (SOURCE RETURN), PBR_R_SHOULDER_PITCH.LOG-RET-IN (SOURCE RETURN), PBR_R_SHOULDER_ROLL.LOG-RET-IN (SOURCE RETURN)
- net RS-RARM_RET: now also PBR_R_ELBOW_PITCH.LOG-RET-OUT (ACTUATOR / DATA REFERENCE), PBR_R_SHOULDER_PITCH.LOG-RET-OUT (ACTUATOR / DATA REFERENCE), PBR_R_SHOULDER_ROLL.LOG-RET-OUT (ACTUATOR / DATA REFERENCE)
- removed net RS-RARM_VDD: AX_R_ELBOW_PITCH.2 (VDD), AX_R_SHOULDER_PITCH.2 (VDD), AX_R_SHOULDER_ROLL.2 (VDD)
- new net ACT_MAIN_SAFE_12V: PBR_R_ELBOW_PITCH.LOG-IN (INTERRUPTED SOURCE), PBR_R_SHOULDER_PITCH.LOG-IN (INTERRUPTED SOURCE), PBR_R_SHOULDER_ROLL.LOG-IN (INTERRUPTED SOURCE)
- new net R_ELBOW_PITCH_VDD: AX_R_ELBOW_PITCH.2 (VDD), PBR_R_ELBOW_PITCH.LOG-OUT (PROTECTED ACTUATOR VDD)
- new net R_SHOULDER_PITCH_VDD: AX_R_SHOULDER_PITCH.2 (VDD), PBR_R_SHOULDER_PITCH.LOG-OUT (PROTECTED ACTUATOR VDD)
- new net R_SHOULDER_ROLL_VDD: AX_R_SHOULDER_ROLL.2 (VDD), PBR_R_SHOULDER_ROLL.LOG-OUT (PROTECTED ACTUATOR VDD)
- no-connect marks 1 -> 3
Other:
- note added: "10 Right proximal-arm RS-485 data bus and individual feeds"
- note added: "Connected RS-RARM data-only segment and one separately protected power feed per actuator."
- note added: "IDs, baud rate, cable, EMC, thermal and fault behavior remain unvalidated."
- note added: "NOTE 1: The listed axes share only data and reference. Each pin-2 VDD has a distinct"
- note added: "NOTE 3: A custom/de-pinned data-only harness or breakout is SELECTION REQUIRED. Termination,"
- note added: "W10020"
- note added: "W10021"
- note added: "W10022"
- note added: "W10023"
- note added: "W10024"
- note added: "W10025"
- note added: "W10026"
- note added: "W10027"
- note added: "protected feed; no standard VDD-carrying daisy cable may parallel those feeds."
- note removed: "10 Right proximal-arm RS-485 and protected branch"
- note removed: "Connected RS-RARM data segment and separately protected actuator-power branch."
- note removed: "NOTE 1: The segment shares data and branch power only among the listed axes; it does not"
- note removed: "NOTE 3: Termination, bias, actuator IDs, baud rate, cable length, waveform, latency, EMC,"
- note removed: "join any other protected branch VDD."
- note removed: "thermal and fault behavior remain unvalidated."
- moved on the sheet: AX_R_ELBOW_PITCH, AX_R_SHOULDER_PITCH, AX_R_SHOULDER_ROLL, PORT_RS_RARM

Commit message: Close HR-30 whole-body mass and shoulder architecture
Parts:
- AX_R_SHOULDER_PITCH: value ROBOTIS XM540-W270-R candidate -> ROBOTIS XM430-W350-R candidate; Display ROBOTIS XM540-W270-R candidate -> ROBOTIS XM430-W350-R candidate
Changed lines of the file:
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@@
       (exclude_from_sim no) (in_bom yes) (on_board yes) (dnp no)
       (property "Reference" "AX_R_SHOULDER_PITCH" (at 278.13 83.63 0) (effects (font (size 1.50 1.50)) (justify left bottom)))
-      (property "Value" "ROBOTIS XM540-W270-R candidate" (at 314.96 100.33 0) (effects (font (size 1.50 1.50)) (hide yes)))
+      (property "Value" "ROBOTIS XM430-W350-R candidate" (at 314.96 100.33 0) (effects (font (size 1.50 1.50)) (hide yes)))
       (property "Footprint" "" (at 314.96 100.33 0) (effects (font (size 1.50 1.50)) (hide yes)))
-      (property "Datasheet" "https://docs.robotis.com/docs/dxl/model_reference/x_series/xm_series/xm540-w270/" (at 314.96 100.33 0) (effects (font (size 1.50 1.50)) (hide yes)))
+      (property "Datasheet" "https://docs.robotis.com/docs/dxl/model_reference/x_series/xm_series/xm430-w350/" (at 314.96 100.33 0) (effects (font (size 1.50 1.50)) (hide yes)))
       (property "Description" "Axis identity, protocol and manufacturer actuator-side pins are allocated. Exact order code, actuator ID, cable assembly, controller-side connector, branch current/protection and installed thermal/communication behavior remain selection and test work." (at 314.96 100.33 0) (effects (font (size 1.50 1.50)) (hide yes)))
       (property "Status" "ACTUATOR-SIDE PINOUT VERIFIED - HARNESS AND CONTROLLER SIDE SELECTION REQUIRED" (at 314.96 116.03 0) (effects (font (size 1.50 1.50)) (justify bottom)))
       (property "Evidence" "Current official ROBOTIS Docs checked 2026-08-14: actuator-side 1=GND, 2=VDD and 3=DATA (TTL) or 3=DATA+/4=DATA- (RS-485)." (at 314.96 100.33 0) (effects (font (size 1.50 1.50)) (hide yes)))
-      (property "Display" "ROBOTIS XM540-W270-R candidate" (at 278.13 86.83 0) (effects (font (size 1.50 1.50)) (justify left bottom)))
+      (property "Display" "ROBOTIS XM430-W350-R candidate" (at 278.13 86.83 0) (effects (font (size 1.50 1.50)) (justify left bottom)))
       (pin "2")
       (pin "1")
