File: hr30/whole-body-p0.1/electrical/kicad/hr30-whole-body-electrical-p0.1/05_carrier_a_four_isolated_rs485.kicad_sch (KiCad schematic)
At the start: 9 parts

Commit message: Add HR-30 motion controller candidate
Connections:
- net CTRL_3V3: now also JCA1.3 (CONTROL 3.3 V); no longer JCA1.2 (CONTROL 3.3 V)
- net CTRL_5V: now also JCA1.2 (CONTROL 5 V); no longer JCA1.1 (CONTROL 5 V)
- net CTRL_GND: now also JCA1.1 (CONTROL GROUND); no longer JCA1.3 (CONTROL GROUND)
Changed lines of the file:
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@@
       (stroke (width 0.50) (type solid)) (fill (type none))) (wire (pts (xy 151.13 64.77) (xy 140.97 64.77))
               (stroke (width 0) (type default)))
-(global_label "CTRL_5V" (shape bidirectional) (at 140.97 64.77 180)
+(global_label "CTRL_GND" (shape bidirectional) (at 140.97 64.77 180)
               (fields_autoplaced yes) (effects (font (size 1.50 1.50)) (justify right))
               (property "Intersheetrefs" "${INTERSHEET_REFS}" (at 140.97 67.31 0)
@@
 (wire (pts (xy 151.13 59.69) (xy 140.97 59.69))
               (stroke (width 0) (type default)))
-(global_label "CTRL_3V3" (shape bidirectional) (at 140.97 59.69 180)
+(global_label "CTRL_5V" (shape bidirectional) (at 140.97 59.69 180)
               (fields_autoplaced yes) (effects (font (size 1.50 1.50)) (justify right))
               (property "Intersheetrefs" "${INTERSHEET_REFS}" (at 140.97 62.23 0)
@@
 (wire (pts (xy 151.13 54.61) (xy 140.97 54.61))
               (stroke (width 0) (type default)))
-(global_label "CTRL_GND" (shape bidirectional) (at 140.97 54.61 180)
+(global_label "CTRL_3V3" (shape bidirectional) (at 140.97 54.61 180)
               (fields_autoplaced yes) (effects (font (size 1.50 1.50)) (justify right))
               (property "Intersheetrefs" "${INTERSHEET_REFS}" (at 140.97 57.15 0)

Commit message: Integrate HR-30 PA field connector harnesses
Parts:
- J_RS_LARM, J_RS_LLEG, J_RS_RARM, J_RS_RLEG: value JST BM03B-GHS-TBT DATA-ONLY FIELD HEADER -> JST B03B-PASK-1 DATA-ONLY FIELD HEADER; Display JST BM03B-GHS-TBT DATA-ONLY FIELD HEADER -> JST B03B-PASK-1 DATA-ONLY FIELD HEADER; Evidence JST GH official eGH catalog checked 2026-08-14. -> JST PA official ePA-F catalog checked 2026-08-18: 2.0 mm se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
Changed lines of the file:
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@@
       (exclude_from_sim no) (in_bom yes) (on_board yes) (dnp no)
       (property "Reference" "J_RS_LLEG" (at 19.05 225.87 0) (effects (font (size 1.50 1.50)) (justify left bottom)))
-      (property "Value" "JST BM03B-GHS-TBT DATA-ONLY FIELD HEADER" (at 54.61 242.57 0) (effects (font (size 1.50 1.50)) (hide yes)))
+      (property "Value" "JST B03B-PASK-1 DATA-ONLY FIELD HEADER" (at 54.61 242.57 0) (effects (font (size 1.50 1.50)) (hide yes)))
       (property "Footprint" "" (at 54.61 242.57 0) (effects (font (size 1.50 1.50)) (hide yes)))
-      (property "Datasheet" "https://www.jst-mfg.com/product/pdf/eng/eGH.pdf" (at 54.61 242.57 0) (effects (font (size 1.50 1.50)) (hide yes)))
-      (property "Description" "Three-contact data-only connector. It intentionally has no actuator VDD contact. Mating GHR-03V-S/SSHL-002T-P0.2 cable, shield/bond, termination, protection and routing remain open." (at 54.61 242.57 0) (effects (font (size 1.50 1.50)) (hide yes)))
+      (property "Datasheet" "https://www.jst-mfg.com/product/pdf/eng/ePA-F.pdf" (at 54.61 242.57 0) (effects (font (size 1.50 1.50)) (hide yes)))
+      (property "Description" "Three-contact data-only connector. It intentionally has no actuator VDD contact. Mating PAP-03V-S/SPHD-001T-P0.5 cable, shield/bond, termination, protection and routing remain open." (at 54.61 242.57 0) (effects (font (size 1.50 1.50)) (hide yes)))
       (property "Status" "EXACT DATA-ONLY CONNECTOR CANDIDATE - HARNESS/EMC VALIDATION REQUIRED" (at 54.61 258.27 0) (effects (font (size 1.50 1.50)) (justify bottom)))
-      (property "Evidence" "JST GH official eGH catalog checked 2026-08-14." (at 54.61 242.57 0) (effects (font (size 1.50 1.50)) (hide yes)))
-      (property "Display" "JST BM03B-GHS-TBT DATA-ONLY FIELD HEADER" (at 19.05 229.07 0) (effects (font (size 1.50 1.50)) (justify left bottom)))
+      (property "Evidence" "JST PA official ePA-F catalog checked 2026-08-18: 2.0 mm secure lock; 0.13-0.33 mm2 SPHD-001T-P0.5 contact range includes the 0.25 mm2 RS candidate conductor." (at 54.61 242.57 0) (effects (font (size 1.50 1.50)) (hide yes)))
+      (property "Display" "JST B03B-PASK-1 DATA-ONLY FIELD HEADER" (at 19.05 229.07 0) (effects (font (size 1.50 1.50)) (justify left bottom)))
       (pin "1")
       (pin "2")
@@
       (exclude_from_sim no) (in_bom yes) (on_board yes) (dnp no)
       (property "Reference" "J_RS_RLEG" (at 119.38 225.87 0) (effects (font (size 1.50 1.50)) (justify left bottom)))
-      (property "Value" "JST BM03B-GHS-TBT DATA-ONLY FIELD HEADER" (at 154.94 242.57 0) (effects (font (size 1.50 1.50)) (hide yes)))
+      (property "Value" "JST B03B-PASK-1 DATA-ONLY FIELD HEADER" (at 154.94 242.57 0) (effects (font (size 1.50 1.50)) (hide yes)))
       (property "Footprint" "" (at 154.94 242.57 0) (effects (font (size 1.50 1.50)) (hide yes)))
-      (property "Datasheet" "https://www.jst-mfg.com/product/pdf/eng/eGH.pdf" (at 154.94 242.57 0) (effects (font (size 1.50 1.50)) (hide yes)))
-      (property "Description" "Three-contact data-only connector. It intentionally has no actuator VDD contact. Mating GHR-03V-S/SSHL-002T-P0.2 cable, shield/bond, termination, protection and routing remain open." (at 154.94 242.57 0) (effects (font (size 1.50 1.50)) (hide yes)))
+      (property "Datasheet" "https://www.jst-mfg.com/product/pdf/eng/ePA-F.pdf" (at 154.94 242.57 0) (effects (font (size 1.50 1.50)) (hide yes)))
+      (property "Description" "Three-contact data-only connector. It intentionally has no actuator VDD contact. Mating PAP-03V-S/SPHD-001T-P0.5 cable, shield/bond, termination, protection and routing remain open." (at 154.94 242.57 0) (effects (font (size 1.50 1.50)) (hide yes)))
       (property "Status" "EXACT DATA-ONLY CONNECTOR CANDIDATE - HARNESS/EMC VALIDATION REQUIRED" (at 154.94 258.27 0) (effects (font (size 1.50 1.50)) (justify bottom)))
-      (property "Evidence" "JST GH official eGH catalog checked 2026-08-14." (at 154.94 242.57 0) (effects (font (size 1.50 1.50)) (hide yes)))
-      (property "Display" "JST BM03B-GHS-TBT DATA-ONLY FIELD HEADER" (at 119.38 229.07 0) (effects (font (size 1.50 1.50)) (justify left bottom)))
+      (property "Evidence" "JST PA official ePA-F catalog checked 2026-08-18: 2.0 mm secure lock; 0.13-0.33 mm2 SPHD-001T-P0.5 contact range includes the 0.25 mm2 RS candidate conductor." (at 154.94 242.57 0) (effects (font (size 1.50 1.50)) (hide yes)))
+      (property "Display" "JST B03B-PASK-1 DATA-ONLY FIELD HEADER" (at 119.38 229.07 0) (effects (font (size 1.50 1.50)) (justify left bottom)))
       (pin "1")
       (pin "2")
@@
       (exclude_from_sim no) (in_bom yes) (on_board yes) (dnp no)
       (property "Reference" "J_RS_LARM" (at 219.71 225.87 0) (effects (font (size 1.50 1.50)) (justify left bottom)))
-      (property "Value" "JST BM03B-GHS-TBT DATA-ONLY FIELD HEADER" (at 255.27 242.57 0) (effects (font (size 1.50 1.50)) (hide yes)))
+      (property "Value" "JST B03B-PASK-1 DATA-ONLY FIELD HEADER" (at 255.27 242.57 0) (effects (font (size 1.50 1.50)) (hide yes)))
       (property "Footprint" "" (at 255.27 242.57 0) (effects (font (size 1.50 1.50)) (hide yes)))
-      (property "Datasheet" "https://www.jst-mfg.com/product/pdf/eng/eGH.pdf" (at 255.27 242.57 0) (effects (font (size 1.50 1.50)) (hide yes)))
-      (property "Description" "Three-contact data-only connector. It intentionally has no actuator VDD contact. Mating GHR-03V-S/SSHL-002T-P0.2 cable, shield/bond, termination, protection and routing remain open." (at 255.27 242.57 0) (effects (font (size 1.50 1.50)) (hide yes)))
+      (property "Datasheet" "https://www.jst-mfg.com/product/pdf/eng/ePA-F.pdf" (at 255.27 242.57 0) (effects (font (size 1.50 1.50)) (hide yes)))
+      (property "Description" "Three-contact data-only connector. It intentionally has no actuator VDD contact. Mating PAP-03V-S/SPHD-001T-P0.5 cable, shield/bond, termination, protection and routing remain open." (at 255.27 242.57 0) (effects (font (size 1.50 1.50)) (hide yes)))
       (property "Status" "EXACT DATA-ONLY CONNECTOR CANDIDATE - HARNESS/EMC VALIDATION REQUIRED" (at 255.27 258.27 0) (effects (font (size 1.50 1.50)) (justify bottom)))
-      (property "Evidence" "JST GH official eGH catalog checked 2026-08-14." (at 255.27 242.57 0) (effects (font (size 1.50 1.50)) (hide yes)))
-      (property "Display" "JST BM03B-GHS-TBT DATA-ONLY FIELD HEADER" (at 219.71 229.07 0) (effects (font (size 1.50 1.50)) (justify left bottom)))
+      (property "Evidence" "JST PA official ePA-F catalog checked 2026-08-18: 2.0 mm secure lock; 0.13-0.33 mm2 SPHD-001T-P0.5 contact range includes the 0.25 mm2 RS candidate conductor." (at 255.27 242.57 0) (effects (font (size 1.50 1.50)) (hide yes)))
+      (property "Display" "JST B03B-PASK-1 DATA-ONLY FIELD HEADER" (at 219.71 229.07 0) (effects (font (size 1.50 1.50)) (justify left bottom)))
       (pin "1")
       (pin "2")
@@
       (exclude_from_sim no) (in_bom yes) (on_board yes) (dnp no)
       (property "Reference" "J_RS_RARM" (at 320.04 225.87 0) (effects (font (size 1.50 1.50)) (justify left bottom)))
-      (property "Value" "JST BM03B-GHS-TBT DATA-ONLY FIELD HEADER" (at 355.60 242.57 0) (effects (font (size 1.50 1.50)) (hide yes)))
+      (property "Value" "JST B03B-PASK-1 DATA-ONLY FIELD HEADER" (at 355.60 242.57 0) (effects (font (size 1.50 1.50)) (hide yes)))
       (property "Footprint" "" (at 355.60 242.57 0) (effects (font (size 1.50 1.50)) (hide yes)))
-      (property "Datasheet" "https://www.jst-mfg.com/product/pdf/eng/eGH.pdf" (at 355.60 242.57 0) (effects (font (size 1.50 1.50)) (hide yes)))
-      (property "Description" "Three-contact data-only connector. It intentionally has no actuator VDD contact. Mating GHR-03V-S/SSHL-002T-P0.2 cable, shield/bond, termination, protection and routing remain open." (at 355.60 242.57 0) (effects (font (size 1.50 1.50)) (hide yes)))
+      (property "Datasheet" "https://www.jst-mfg.com/product/pdf/eng/ePA-F.pdf" (at 355.60 242.57 0) (effects (font (size 1.50 1.50)) (hide yes)))
+      (property "Description" "Three-contact data-only connector. It intentionally has no actuator VDD contact. Mating PAP-03V-S/SPHD-001T-P0.5 cable, shield/bond, termination, protection and routing remain open." (at 355.60 242.57 0) (effects (font (size 1.50 1.50)) (hide yes)))
       (property "Status" "EXACT DATA-ONLY CONNECTOR CANDIDATE - HARNESS/EMC VALIDATION REQUIRED" (at 355.60 258.27 0) (effects (font (size 1.50 1.50)) (justify bottom)))
-      (property "Evidence" "JST GH official eGH catalog checked 2026-08-14." (at 355.60 242.57 0) (effects (font (size 1.50 1.50)) (hide yes)))
-      (property "Display" "JST BM03B-GHS-TBT DATA-ONLY FIELD HEADER" (at 320.04 229.07 0) (effects (font (size 1.50 1.50)) (justify left bottom)))
+      (property "Evidence" "JST PA official ePA-F catalog checked 2026-08-18: 2.0 mm secure lock; 0.13-0.33 mm2 SPHD-001T-P0.5 contact range includes the 0.25 mm2 RS candidate conductor." (at 355.60 242.57 0) (effects (font (size 1.50 1.50)) (hide yes)))
+      (property "Display" "JST B03B-PASK-1 DATA-ONLY FIELD HEADER" (at 320.04 229.07 0) (effects (font (size 1.50 1.50)) (justify left bottom)))
       (pin "1")
       (pin "2")
