File: hr30/whole-body-p0.1/electrical/kicad/hr30-whole-body-electrical-p0.1/06_carrier_b_waist_and_ttl.kicad_sch (KiCad schematic)
At the start: 9 parts

Commit message: Add HR-30 motion controller candidate
Connections:
- net CTRL_3V3: now also JCB1.3 (CONTROL 3.3 V); no longer JCB1.2 (CONTROL 3.3 V)
- net CTRL_5V: now also JCB1.2 (CONTROL 5 V); no longer JCB1.1 (CONTROL 5 V)
- net CTRL_GND: now also JCB1.1 (CONTROL GROUND); no longer JCB1.3 (CONTROL GROUND)
Changed lines of the file:
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@@
       (stroke (width 0.50) (type solid)) (fill (type none))) (wire (pts (xy 151.13 64.77) (xy 140.97 64.77))
               (stroke (width 0) (type default)))
-(global_label "CTRL_5V" (shape bidirectional) (at 140.97 64.77 180)
+(global_label "CTRL_GND" (shape bidirectional) (at 140.97 64.77 180)
               (fields_autoplaced yes) (effects (font (size 1.50 1.50)) (justify right))
               (property "Intersheetrefs" "${INTERSHEET_REFS}" (at 140.97 67.31 0)
@@
 (wire (pts (xy 151.13 59.69) (xy 140.97 59.69))
               (stroke (width 0) (type default)))
-(global_label "CTRL_3V3" (shape bidirectional) (at 140.97 59.69 180)
+(global_label "CTRL_5V" (shape bidirectional) (at 140.97 59.69 180)
               (fields_autoplaced yes) (effects (font (size 1.50 1.50)) (justify right))
               (property "Intersheetrefs" "${INTERSHEET_REFS}" (at 140.97 62.23 0)
@@
 (wire (pts (xy 151.13 54.61) (xy 140.97 54.61))
               (stroke (width 0) (type default)))
-(global_label "CTRL_GND" (shape bidirectional) (at 140.97 54.61 180)
+(global_label "CTRL_3V3" (shape bidirectional) (at 140.97 54.61 180)
               (fields_autoplaced yes) (effects (font (size 1.50 1.50)) (justify right))
               (property "Intersheetrefs" "${INTERSHEET_REFS}" (at 140.97 57.15 0)

Commit message: Integrate HR-30 PA field connector harnesses
Parts:
- J_RS_WAIST: value JST BM03B-GHS-TBT DATA-ONLY FIELD HEADER -> JST B03B-PASK-1 DATA-ONLY FIELD HEADER; Display JST BM03B-GHS-TBT DATA-ONLY FIELD HEADER -> JST B03B-PASK-1 DATA-ONLY FIELD HEADER; Evidence JST GH official eGH catalog checked 2026-08-14. -> JST PA official ePA-F catalog checked 2026-08-18: 2.0 mm se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
- J_TTL_HEAD, J_TTL_LDIST, J_TTL_RDIST: value JST BM02B-GHS-TBT DATA-ONLY FIELD HEADER -> JST B02B-PASK-1 DATA-ONLY FIELD HEADER; Display JST BM02B-GHS-TBT DATA-ONLY FIELD HEADER -> JST B02B-PASK-1 DATA-ONLY FIELD HEADER; Evidence JST GH official eGH catalog checked 2026-08-14. -> JST PA official ePA-F catalog checked 2026-08-18: 2.0 mm se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
Changed lines of the file:
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@@
       (exclude_from_sim no) (in_bom yes) (on_board yes) (dnp no)
       (property "Reference" "J_RS_WAIST" (at 284.48 112.84 0) (effects (font (size 1.50 1.50)) (justify left bottom)))
-      (property "Value" "JST BM03B-GHS-TBT DATA-ONLY FIELD HEADER" (at 320.04 129.54 0) (effects (font (size 1.50 1.50)) (hide yes)))
+      (property "Value" "JST B03B-PASK-1 DATA-ONLY FIELD HEADER" (at 320.04 129.54 0) (effects (font (size 1.50 1.50)) (hide yes)))
       (property "Footprint" "" (at 320.04 129.54 0) (effects (font (size 1.50 1.50)) (hide yes)))
-      (property "Datasheet" "https://www.jst-mfg.com/product/pdf/eng/eGH.pdf" (at 320.04 129.54 0) (effects (font (size 1.50 1.50)) (hide yes)))
-      (property "Description" "Three-contact data-only connector. It intentionally has no actuator VDD contact. Mating GHR-03V-S/SSHL-002T-P0.2 cable, shield/bond, termination, protection and routing remain open." (at 320.04 129.54 0) (effects (font (size 1.50 1.50)) (hide yes)))
+      (property "Datasheet" "https://www.jst-mfg.com/product/pdf/eng/ePA-F.pdf" (at 320.04 129.54 0) (effects (font (size 1.50 1.50)) (hide yes)))
+      (property "Description" "Three-contact data-only connector. It intentionally has no actuator VDD contact. Mating PAP-03V-S/SPHD-001T-P0.5 cable, shield/bond, termination, protection and routing remain open." (at 320.04 129.54 0) (effects (font (size 1.50 1.50)) (hide yes)))
       (property "Status" "EXACT DATA-ONLY CONNECTOR CANDIDATE - HARNESS/EMC VALIDATION REQUIRED" (at 320.04 145.24 0) (effects (font (size 1.50 1.50)) (justify bottom)))
-      (property "Evidence" "JST GH official eGH catalog checked 2026-08-14." (at 320.04 129.54 0) (effects (font (size 1.50 1.50)) (hide yes)))
-      (property "Display" "JST BM03B-GHS-TBT DATA-ONLY FIELD HEADER" (at 284.48 116.04 0) (effects (font (size 1.50 1.50)) (justify left bottom)))
+      (property "Evidence" "JST PA official ePA-F catalog checked 2026-08-18: 2.0 mm secure lock; 0.13-0.33 mm2 SPHD-001T-P0.5 contact range includes the 0.25 mm2 RS candidate conductor." (at 320.04 129.54 0) (effects (font (size 1.50 1.50)) (hide yes)))
+      (property "Display" "JST B03B-PASK-1 DATA-ONLY FIELD HEADER" (at 284.48 116.04 0) (effects (font (size 1.50 1.50)) (justify left bottom)))
       (pin "1")
       (pin "2")
@@
       (exclude_from_sim no) (in_bom yes) (on_board yes) (dnp no)
       (property "Reference" "J_TTL_LDIST" (at 34.29 228.41 0) (effects (font (size 1.50 1.50)) (justify left bottom)))
-      (property "Value" "JST BM02B-GHS-TBT DATA-ONLY FIELD HEADER" (at 80.01 245.11 0) (effects (font (size 1.50 1.50)) (hide yes)))
+      (property "Value" "JST B02B-PASK-1 DATA-ONLY FIELD HEADER" (at 80.01 245.11 0) (effects (font (size 1.50 1.50)) (hide yes)))
       (property "Footprint" "" (at 80.01 245.11 0) (effects (font (size 1.50 1.50)) (hide yes)))
-      (property "Datasheet" "https://www.jst-mfg.com/product/pdf/eng/eGH.pdf" (at 80.01 245.11 0) (effects (font (size 1.50 1.50)) (hide yes)))
-      (property "Description" "Two-contact data-only connector; no actuator VDD contact. Mating GHR-02V-S/SSHL-002T-P0.2 cable, protection and routing remain open." (at 80.01 245.11 0) (effects (font (size 1.50 1.50)) (hide yes)))
+      (property "Datasheet" "https://www.jst-mfg.com/product/pdf/eng/ePA-F.pdf" (at 80.01 245.11 0) (effects (font (size 1.50 1.50)) (hide yes)))
+      (property "Description" "Two-contact data-only connector; no actuator VDD contact. Mating PAP-02V-S/SPHD-002T-P0.5 cable, protection and routing remain open." (at 80.01 245.11 0) (effects (font (size 1.50 1.50)) (hide yes)))
       (property "Status" "EXACT DATA-ONLY CONNECTOR CANDIDATE - HARNESS/EMC VALIDATION REQUIRED" (at 80.01 260.81 0) (effects (font (size 1.50 1.50)) (justify bottom)))
-      (property "Evidence" "JST GH official eGH catalog checked 2026-08-14." (at 80.01 245.11 0) (effects (font (size 1.50 1.50)) (hide yes)))
-      (property "Display" "JST BM02B-GHS-TBT DATA-ONLY FIELD HEADER" (at 34.29 231.61 0) (effects (font (size 1.50 1.50)) (justify left bottom)))
+      (property "Evidence" "JST PA official ePA-F catalog checked 2026-08-18: 2.0 mm secure lock; 0.08-0.21 mm2 SPHD-002T-P0.5 contact range includes the 0.14 mm2 TTL candidate conductor." (at 80.01 245.11 0) (effects (font (size 1.50 1.50)) (hide yes)))
+      (property "Display" "JST B02B-PASK-1 DATA-ONLY FIELD HEADER" (at 34.29 231.61 0) (effects (font (size 1.50 1.50)) (justify left bottom)))
       (pin "1")
       (pin "2")
@@
       (exclude_from_sim no) (in_bom yes) (on_board yes) (dnp no)
       (property "Reference" "J_TTL_RDIST" (at 163.83 228.41 0) (effects (font (size 1.50 1.50)) (justify left bottom)))
-      (property "Value" "JST BM02B-GHS-TBT DATA-ONLY FIELD HEADER" (at 209.55 245.11 0) (effects (font (size 1.50 1.50)) (hide yes)))
+      (property "Value" "JST B02B-PASK-1 DATA-ONLY FIELD HEADER" (at 209.55 245.11 0) (effects (font (size 1.50 1.50)) (hide yes)))
       (property "Footprint" "" (at 209.55 245.11 0) (effects (font (size 1.50 1.50)) (hide yes)))
-      (property "Datasheet" "https://www.jst-mfg.com/product/pdf/eng/eGH.pdf" (at 209.55 245.11 0) (effects (font (size 1.50 1.50)) (hide yes)))
-      (property "Description" "Two-contact data-only connector; no actuator VDD contact. Mating GHR-02V-S/SSHL-002T-P0.2 cable, protection and routing remain open." (at 209.55 245.11 0) (effects (font (size 1.50 1.50)) (hide yes)))
+      (property "Datasheet" "https://www.jst-mfg.com/product/pdf/eng/ePA-F.pdf" (at 209.55 245.11 0) (effects (font (size 1.50 1.50)) (hide yes)))
+      (property "Description" "Two-contact data-only connector; no actuator VDD contact. Mating PAP-02V-S/SPHD-002T-P0.5 cable, protection and routing remain open." (at 209.55 245.11 0) (effects (font (size 1.50 1.50)) (hide yes)))
       (property "Status" "EXACT DATA-ONLY CONNECTOR CANDIDATE - HARNESS/EMC VALIDATION REQUIRED" (at 209.55 260.81 0) (effects (font (size 1.50 1.50)) (justify bottom)))
-      (property "Evidence" "JST GH official eGH catalog checked 2026-08-14." (at 209.55 245.11 0) (effects (font (size 1.50 1.50)) (hide yes)))
-      (property "Display" "JST BM02B-GHS-TBT DATA-ONLY FIELD HEADER" (at 163.83 231.61 0) (effects (font (size 1.50 1.50)) (justify left bottom)))
+      (property "Evidence" "JST PA official ePA-F catalog checked 2026-08-18: 2.0 mm secure lock; 0.08-0.21 mm2 SPHD-002T-P0.5 contact range includes the 0.14 mm2 TTL candidate conductor." (at 209.55 245.11 0) (effects (font (size 1.50 1.50)) (hide yes)))
+      (property "Display" "JST B02B-PASK-1 DATA-ONLY FIELD HEADER" (at 163.83 231.61 0) (effects (font (size 1.50 1.50)) (justify left bottom)))
       (pin "1")
       (pin "2")
@@
       (exclude_from_sim no) (in_bom yes) (on_board yes) (dnp no)
       (property "Reference" "J_TTL_HEAD" (at 294.64 228.41 0) (effects (font (size 1.50 1.50)) (justify left bottom)))
-      (property "Value" "JST BM02B-GHS-TBT DATA-ONLY FIELD HEADER" (at 340.36 245.11 0) (effects (font (size 1.50 1.50)) (hide yes)))
+      (property "Value" "JST B02B-PASK-1 DATA-ONLY FIELD HEADER" (at 340.36 245.11 0) (effects (font (size 1.50 1.50)) (hide yes)))
       (property "Footprint" "" (at 340.36 245.11 0) (effects (font (size 1.50 1.50)) (hide yes)))
-      (property "Datasheet" "https://www.jst-mfg.com/product/pdf/eng/eGH.pdf" (at 340.36 245.11 0) (effects (font (size 1.50 1.50)) (hide yes)))
-      (property "Description" "Two-contact data-only connector; no actuator VDD contact. Mating GHR-02V-S/SSHL-002T-P0.2 cable, protection and routing remain open." (at 340.36 245.11 0) (effects (font (size 1.50 1.50)) (hide yes)))
+      (property "Datasheet" "https://www.jst-mfg.com/product/pdf/eng/ePA-F.pdf" (at 340.36 245.11 0) (effects (font (size 1.50 1.50)) (hide yes)))
+      (property "Description" "Two-contact data-only connector; no actuator VDD contact. Mating PAP-02V-S/SPHD-002T-P0.5 cable, protection and routing remain open." (at 340.36 245.11 0) (effects (font (size 1.50 1.50)) (hide yes)))
       (property "Status" "EXACT DATA-ONLY CONNECTOR CANDIDATE - HARNESS/EMC VALIDATION REQUIRED" (at 340.36 260.81 0) (effects (font (size 1.50 1.50)) (justify bottom)))
-      (property "Evidence" "JST GH official eGH catalog checked 2026-08-14." (at 340.36 245.11 0) (effects (font (size 1.50 1.50)) (hide yes)))
-      (property "Display" "JST BM02B-GHS-TBT DATA-ONLY FIELD HEADER" (at 294.64 231.61 0) (effects (font (size 1.50 1.50)) (justify left bottom)))
+      (property "Evidence" "JST PA official ePA-F catalog checked 2026-08-18: 2.0 mm secure lock; 0.08-0.21 mm2 SPHD-002T-P0.5 contact range includes the 0.14 mm2 TTL candidate conductor." (at 340.36 245.11 0) (effects (font (size 1.50 1.50)) (hide yes)))
+      (property "Display" "JST B02B-PASK-1 DATA-ONLY FIELD HEADER" (at 294.64 231.61 0) (effects (font (size 1.50 1.50)) (justify left bottom)))
       (pin "1")
       (pin "2")
