File: hr30/whole-body-p0.1/electrical/kicad/hr30-whole-body-electrical-p0.1/01_energy_precharge_conversion.kicad_sch (KiCad schematic)
At the start: 6 parts

Commit message: Correct HR-30 whole-body electrical architecture
Parts:
- removed BATT1: 4S 14.8 V 12 Ah PACK EVALUATION CANDIDATE - COMPL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, symbol PBV3:BATT1
- removed CHG1: CHARGER PORT / INTERLOCK - SELECTION REQUIRED, symbol PBV3:CHG1
- removed DCDC1: INTERRUPTED 14.8 V TO 12 V CONVERTER - SELECTION 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, symbol PBV3:DCDC1
- removed PRE1: PRECHARGE / DISCHARGE NETWORK - DESIGN REQUIRED, symbol PBV3:PRE1
- removed RET1: DC RETURN / FRAME / PE BOUNDARY - DESIGN REQUIRED, symbol PBV3:RET1
- removed SD1: DC SERVICE DISCONNECT - SELECTION REQUIRED, symbol PBV3:SD1
- added ACB1: FACILITY AC / PE PANEL BOUNDARY - SELECTION REQUI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, symbol PBV3:ACB1
- added CTRLPS1: MEAN WELL SD-15A-24 SAFETY-CONTROL SUPPLY CANDIDA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, symbol PBV3:CTRLPS1
- added PS1: MEAN WELL RSP-500-12 TETHER SUPPLY CANDIDATE, symbol PBV3:PS1
- added REG_TTL_H: HEAD 9 V BUCK-BOOST CANDIDATE - POLOLU S18V20F9, symbol PBV3:REG_TTL_H
- added REG_TTL_L: LEFT DISTAL 9 V BUCK-BOOST CANDIDATE - POLOLU S18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, symbol PBV3:REG_TTL_L
- added REG_TTL_R: RIGHT DISTAL 9 V BUCK-BOOST CANDIDATE - POLOLU S1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, symbol PBV3:REG_TTL_R
- added TETH1: TOUCH-SAFE ROBOT DC / PE TETHER BOUNDARY - SELECT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, symbol PBV3:TETH1
Connections:
- net ACT_0V_CONTROLLED: now also REG_TTL_H.LOG-RET-IN (CONTROLLED RETURN), REG_TTL_H.LOG-RET-OUT (RETURN), REG_TTL_L.LOG-RET-IN (CONTROLLED RETURN), REG_TTL_L.LOG-RET-OUT (RETURN), REG_TTL_R.LOG-RET-IN (CONTROLLED RETURN), REG_TTL_R.LOG-RET-OUT (RETURN), TETH1.LOG-ROBOT-N (ROBOT CONTROLLED RETURN)
- new net ACT_MAIN_SAFE_12V: REG_TTL_H.LOG-IN (CONTROLLED 12 V INPUT), REG_TTL_L.LOG-IN (CONTROLLED 12 V INPUT), REG_TTL_R.LOG-IN (CONTROLLED 12 V INPUT), TETH1.LOG-ROBOT-P (ROBOT CONTROLLED MAIN)
- new net FACILITY_AC_L: ACB1.LOG-L (FACILITY LINE), PS1.LOG-L (AC LINE FUNCTION)
- new net FACILITY_AC_N: ACB1.LOG-N (FACILITY NEUTRAL), PS1.LOG-N (AC NEUTRAL FUNCTION)
- new net PANEL_DC_POS_RAW: CTRLPS1.LOG-IN (PANEL DC POSITIVE), PS1.LOG-VPOS (12 V PANEL OUTPUT)
- new net PANEL_DC_RET: CTRLPS1.LOG-RET-IN (PANEL DC RETURN), PS1.LOG-VNEG (PANEL DC RETURN), TETH1.LOG-PANEL-N (PANEL DC RETURN)
- new net PANEL_PE: ACB1.LOG-PE (FACILITY PROTECTIVE EARTH), PS1.LOG-PE (PROTECTIVE EARTH FUNCTION), TETH1.LOG-PANEL-PE (PANEL PE)
- new net SAFETY_0V: CTRLPS1.LOG-RET-OUT (SAFETY CONTROL RETURN)
- new net SAFETY_24V: CTRLPS1.LOG-OUT (24 V SAFETY CONTROL)
- new net TETHER_MAIN_POS: TETH1.LOG-PANEL-P (CONTACTOR-SWITCHED PANEL POSITIVE)
- new net TTL_HEAD_SAFE_9V: REG_TTL_H.LOG-OUT (HEAD ACTUATOR 9 V)
- new net TTL_LDIST_SAFE_9V: REG_TTL_L.LOG-OUT (LEFT DISTAL 9 V)
- new net TTL_RDIST_SAFE_9V: REG_TTL_R.LOG-OUT (RIGHT DISTAL 9 V)
- no-connect marks 6 -> 4
Other:
- note added: "01 Tether-first energy, regulated rails and onboard-later boundary"
- note added: "ACT_MAIN_SAFE_12V until a separate reviewed change closes its holds."
- note added: "External 12 V tether-first source, three regulated 9 V TTL rails and a disconnected onboard-later evaluation boundary."
- note added: "NOTE 1: The 14.8 V direct-actuator architecture is absent. No fuse value, conductor size,"
- note added: "NOTE 2: The onboard-later battery/precharge/charger path is deliberately disconnected from"
- note added: "W1017"
- note added: "W1018"
- note added: "W1019"
- note added: "W1020"
- note added: "W1021"
- note added: "W1022"
- note added: "W1023"
- note added: "W1024"
- note added: "W1025"
- note added: "W1026"
- note added: "W1027"
- note added: "W1028"
- note added: "W1029"
- note added: "connector rating or unresolved physical pin is released."
- note removed: "01 Energy, service disconnect, precharge and conversion"
- note removed: "NOTE 1: No fuse value, conductor size, connector rating or physical pin is released."
- note removed: "NOTE 2: Charger presence must inhibit actuator permit, but the exact fail-safe"
- note removed: "Whole-body DC source and interrupted 14.8/12 V boundaries; every physical selection remains open."
- note removed: "implementation is not selected."

Commit message: Integrate HR-30 three-rail auxiliary power
Connections:
- net FRAME_PE_BOUNDARY: now reaches TETH1.LOG-ROBOT-PE (ROBOT FRAME / PE BOUNDARY)
- no-connect marks 4 -> 3
Other:
- note added: "W1030"
Changed lines of the file:
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@@
               (at 182.88 188.50 0) (effects (font (size 1.27 1.27)) (justify bottom))
 )
-(no_connect (at 177.80 185.42)
+(wire (pts (xy 177.80 185.42) (xy 187.96 185.42))
+              (stroke (width 0) (type default)))
+(global_label "FRAME_PE_BOUNDARY" (shape bidirectional) (at 187.96 185.42 0)
+              (fields_autoplaced yes) (effects (font (size 1.50 1.50)) (justify left))
+              (property "Intersheetrefs" "${INTERSHEET_REFS}" (at 187.96 187.96 0)
+                (effects (font (size 1.27 1.27)) (hide yes))))
+(text "W1018" (exclude_from_sim no)
+              (at 182.88 183.42 0) (effects (font (size 1.27 1.27)) (justify bottom))
 ) (wire (pts (xy 228.60 121.92) (xy 218.44 121.92))
               (stroke (width 0) (type default)))
@@
               (property "Intersheetrefs" "${INTERSHEET_REFS}" (at 218.44 124.46 0)
                 (effects (font (size 1.27 1.27)) (hide yes))))
-(text "W1018" (exclude_from_sim no)
+(text "W1019" (exclude_from_sim no)
               (at 223.52 119.92 0) (effects (font (size 1.27 1.27)) (justify bottom))
 )
@@
               (property "Intersheetrefs" "${INTERSHEET_REFS}" (at 218.44 119.38 0)
                 (effects (font (size 1.27 1.27)) (hide yes))))
-(text "W1019" (exclude_from_sim no)
+(text "W1020" (exclude_from_sim no)
               (at 223.52 114.84 0) (effects (font (size 1.27 1.27)) (justify bottom))
 )
@@
               (property "Intersheetrefs" "${INTERSHEET_REFS}" (at 340.36 127.00 0)
                 (effects (font (size 1.27 1.27)) (hide yes))))
-(text "W1020" (exclude_from_sim no)
+(text "W1021" (exclude_from_sim no)
               (at 335.28 122.46 0) (effects (font (size 1.27 1.27)) (justify bottom))
 )
@@
               (property "Intersheetrefs" "${INTERSHEET_REFS}" (at 340.36 121.92 0)
                 (effects (font (size 1.27 1.27)) (hide yes))))
-(text "W1021" (exclude_from_sim no)
+(text "W1022" (exclude_from_sim no)
               (at 335.28 117.38 0) (effects (font (size 1.27 1.27)) (justify bottom))
 )
@@
               (property "Intersheetrefs" "${INTERSHEET_REFS}" (at 218.44 180.34 0)
                 (effects (font (size 1.27 1.27)) (hide yes))))
-(text "W1022" (exclude_from_sim no)
+(text "W1023" (exclude_from_sim no)
               (at 223.52 175.80 0) (effects (font (size 1.27 1.27)) (justify bottom))
 )
@@
               (property "Intersheetrefs" "${INTERSHEET_REFS}" (at 218.44 175.26 0)
                 (effects (font (size 1.27 1.27)) (hide yes))))
-(text "W1023" (exclude_from_sim no)
+(text "W1024" (exclude_from_sim no)
               (at 223.52 170.72 0) (effects (font (size 1.27 1.27)) (justify bottom))
 )
@@
               (property "Intersheetrefs" "${INTERSHEET_REFS}" (at 340.36 182.88 0)
                 (effects (font (size 1.27 1.27)) (hide yes))))
-(text "W1024" (exclude_from_sim no)
+(text "W1025" (exclude_from_sim no)
               (at 335.28 178.34 0) (effects (font (size 1.27 1.27)) (justify bottom))
 )
@@
               (property "Intersheetrefs" "${INTERSHEET_REFS}" (at 340.36 177.80 0)
                 (effects (font (size 1.27 1.27)) (hide yes))))
-(text "W1025" (exclude_from_sim no)
+(text "W1026" (exclude_from_sim no)
               (at 335.28 173.26 0) (effects (font (size 1.27 1.27)) (justify bottom))
 )
@@
               (property "Intersheetrefs" "${INTERSHEET_REFS}" (at 218.44 234.95 0)
                 (effects (font (size 1.27 1.27)) (hide yes))))
-(text "W1026" (exclude_from_sim no)
+(text "W1027" (exclude_from_sim no)
               (at 223.52 230.41 0) (effects (font (size 1.27 1.27)) (justify bottom))
 )
@@
               (property "Intersheetrefs" "${INTERSHEET_REFS}" (at 218.44 229.87 0)
                 (effects (font (size 1.27 1.27)) (hide yes))))
-(text "W1027" (exclude_from_sim no)
+(text "W1028" (exclude_from_sim no)
               (at 223.52 225.33 0) (effects (font (size 1.27 1.27)) (justify bottom))
 )
@@
               (property "Intersheetrefs" "${INTERSHEET_REFS}" (at 340.36 237.49 0)
                 (effects (font (size 1.27 1.27)) (hide yes))))
-(text "W1028" (exclude_from_sim no)
+(text "W1029" (exclude_from_sim no)
               (at 335.28 232.95 0) (effects (font (size 1.27 1.27)) (justify bottom))
 )
@@
               (property "Intersheetrefs" "${INTERSHEET_REFS}" (at 340.36 232.41 0)
                 (effects (font (size 1.27 1.27)) (hide yes))))
-(text "W1029" (exclude_from_sim no)
+(text "W1030" (exclude_from_sim no)
               (at 335.28 227.87 0) (effects (font (size 1.27 1.27)) (justify bottom))
 )
