File: hr30/whole-body-p0.1/electrical/kicad/hr30-whole-body-electrical-p0.1/03_compute_motion_watchdog.kicad_sch (KiCad schematic)
At the start: 11 parts

Commit message: Expand HR-30 whole-body electrical architecture
Connections:
- net HMI_SENSOR_IPC renamed HEAD_AUDIO_IPC
- new net HEAD_CAM_L_IPC: CPU1.LOG-CAM-L (LEFT CAMERA IPC)
- new net HEAD_CAM_R_IPC: CPU1.LOG-CAM-R (RIGHT CAMERA IPC)
- new net HEAD_DISPLAY_IPC: CPU1.LOG-DISPLAY (FACE DISPLAY IPC)
- new net HEAD_FAN_PWM: CPU1.LOG-FAN-PWM (HEAD FAN PWM)
- new net HEAD_FAN_TACH: CPU1.LOG-FAN-TACH (HEAD FAN TACH)
- new net HEAD_MIC_IPC: CPU1.LOG-MIC (MICROPHONE IPC)
- new net HEAD_TOUCH_IPC: CPU1.LOG-TOUCH (FACE TOUCH IPC)
Other:
- note added: "W3033"
- note added: "W3034"
- note added: "W3035"
- note added: "W3036"
- note added: "W3037"
- note added: "W3038"
- note added: "W3039"

Commit message: Add pin-level HR-30 actuator interface carriers
Parts:
- MCU1: value DETERMINISTIC MOTION CONTROLLER - EXACT BOARD SELECTION REQUIRED -> STM32H743ZIT6 LQFP144 MOTION-CONTROL CARRIER CANDIDATE; Display DETERMINISTIC MOTION CONTROLLER - EXACT BOARD SELECTION REQ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 -> STM32H743ZIT6 LQFP144 MOTION-CONTROL CARRIER CANDIDATE; Evidence (none) -> ST DS12110 Rev 11 and current product page checked 2026-08-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; Status SELECTION REQUIRED - LOGICAL CONNECTIVITY ONLY -> EXACT MCU ORDER-CODE CANDIDATE - BOARD DESIGN AND VALIDATIO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
- MCU_IO_RS_LARM: value MCU1 LOGICAL UART BANK - RS-LARM -> MCU1 USART3 PHYSICAL PIN UNIT - RS-LARM; Display MCU1 LOGICAL UART BANK - RS-LARM -> MCU1 USART3 PHYSICAL PIN UNIT - RS-LARM; Evidence (none) -> ST DS12110 Rev 11 LQFP144 pinout and alternate-function tab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; Status SELECTION REQUIRED - LOGICAL CONNECTIVITY ONLY -> PHYSICAL MCU PACKAGE PIN AND ALTERNATE FUNCTION VERIFIED - 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
- MCU_IO_RS_LLEG: value MCU1 LOGICAL UART BANK - RS-LLEG -> MCU1 USART1 PHYSICAL PIN UNIT - RS-LLEG; Display MCU1 LOGICAL UART BANK - RS-LLEG -> MCU1 USART1 PHYSICAL PIN UNIT - RS-LLEG; Evidence (none) -> ST DS12110 Rev 11 LQFP144 pinout and alternate-function tab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; Status SELECTION REQUIRED - LOGICAL CONNECTIVITY ONLY -> PHYSICAL MCU PACKAGE PIN AND ALTERNATE FUNCTION VERIFIED - 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
- MCU_IO_RS_RARM: value MCU1 LOGICAL UART BANK - RS-RARM -> MCU1 USART6 PHYSICAL PIN UNIT - RS-RARM; Display MCU1 LOGICAL UART BANK - RS-RARM -> MCU1 USART6 PHYSICAL PIN UNIT - RS-RARM; Evidence (none) -> ST DS12110 Rev 11 LQFP144 pinout and alternate-function tab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; Status SELECTION REQUIRED - LOGICAL CONNECTIVITY ONLY -> PHYSICAL MCU PACKAGE PIN AND ALTERNATE FUNCTION VERIFIED - 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
- MCU_IO_RS_RLEG: value MCU1 LOGICAL UART BANK - RS-RLEG -> MCU1 USART2 PHYSICAL PIN UNIT - RS-RLEG; Display MCU1 LOGICAL UART BANK - RS-RLEG -> MCU1 USART2 PHYSICAL PIN UNIT - RS-RLEG; Evidence (none) -> ST DS12110 Rev 11 LQFP144 pinout and alternate-function tab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; Status SELECTION REQUIRED - LOGICAL CONNECTIVITY ONLY -> PHYSICAL MCU PACKAGE PIN AND ALTERNATE FUNCTION VERIFIED - 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
- MCU_IO_RS_WAIST: value MCU1 LOGICAL UART BANK - RS-WAIST -> MCU1 UART4 PHYSICAL PIN UNIT - RS-WAIST; Display MCU1 LOGICAL UART BANK - RS-WAIST -> MCU1 UART4 PHYSICAL PIN UNIT - RS-WAIST; Evidence (none) -> ST DS12110 Rev 11 LQFP144 pinout and alternate-function tab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; Status SELECTION REQUIRED - LOGICAL CONNECTIVITY ONLY -> PHYSICAL MCU PACKAGE PIN AND ALTERNATE FUNCTION VERIFIED - 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
- MCU_IO_TTL_HEAD: value MCU1 LOGICAL UART BANK - TTL-HEAD -> MCU1 UART8 PHYSICAL PIN UNIT - TTL-HEAD; Display MCU1 LOGICAL UART BANK - TTL-HEAD -> MCU1 UART8 PHYSICAL PIN UNIT - TTL-HEAD; Evidence (none) -> ST DS12110 Rev 11 LQFP144 pinout and alternate-function tab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; Status SELECTION REQUIRED - LOGICAL CONNECTIVITY ONLY -> PHYSICAL MCU PACKAGE PIN AND ALTERNATE FUNCTION VERIFIED - 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
- MCU_IO_TTL_LDIST: value MCU1 LOGICAL UART BANK - TTL-LDIST -> MCU1 UART5 PHYSICAL PIN UNIT - TTL-LDIST; Display MCU1 LOGICAL UART BANK - TTL-LDIST -> MCU1 UART5 PHYSICAL PIN UNIT - TTL-LDIST; Evidence (none) -> ST DS12110 Rev 11 LQFP144 pinout and alternate-function tab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; Status SELECTION REQUIRED - LOGICAL CONNECTIVITY ONLY -> PHYSICAL MCU PACKAGE PIN AND ALTERNATE FUNCTION VERIFIED - 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
- MCU_IO_TTL_RDIST: value MCU1 LOGICAL UART BANK - TTL-RDIST -> MCU1 UART7 PHYSICAL PIN UNIT - TTL-RDIST; Display MCU1 LOGICAL UART BANK - TTL-RDIST -> MCU1 UART7 PHYSICAL PIN UNIT - TTL-RDIST; Evidence (none) -> ST DS12110 Rev 11 LQFP144 pinout and alternate-function tab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; Status SELECTION REQUIRED - LOGICAL CONNECTIVITY ONLY -> PHYSICAL MCU PACKAGE PIN AND ALTERNATE FUNCTION VERIFIED - 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
Connections:
- net UART_RS-LARM_DIR: now also MCU_IO_RS_LARM.81 (PD12 AF7 RTS/DE); no longer MCU_IO_RS_LARM.LOG-RS-LARM-DIR (DIRECTION)
- net UART_RS-LARM_RX: now also MCU_IO_RS_LARM.78 (PD9 AF7 RX); no longer MCU_IO_RS_LARM.LOG-RS-LARM-RX (UART RX)
- net UART_RS-LARM_TX: now also MCU_IO_RS_LARM.77 (PD8 AF7 TX); no longer MCU_IO_RS_LARM.LOG-RS-LARM-TX (UART TX)
- net UART_RS-LLEG_DIR: now also MCU_IO_RS_LLEG.104 (PA12 AF7 RTS/DE); no longer MCU_IO_RS_LLEG.LOG-RS-LLEG-DIR (DIRECTION)
- net UART_RS-LLEG_RX: now also MCU_IO_RS_LLEG.102 (PA10 AF7 RX); no longer MCU_IO_RS_LLEG.LOG-RS-LLEG-RX (UART RX)
- net UART_RS-LLEG_TX: now also MCU_IO_RS_LLEG.101 (PA9 AF7 TX); no longer MCU_IO_RS_LLEG.LOG-RS-LLEG-TX (UART TX)
- net UART_RS-RARM_DIR: now also MCU_IO_RS_RARM.93 (PG8 AF7 RTS/DE); no longer MCU_IO_RS_RARM.LOG-RS-RARM-DIR (DIRECTION)
- net UART_RS-RARM_RX: now also MCU_IO_RS_RARM.97 (PC7 AF7 RX); no longer MCU_IO_RS_RARM.LOG-RS-RARM-RX (UART RX)
- net UART_RS-RARM_TX: now also MCU_IO_RS_RARM.96 (PC6 AF7 TX); no longer MCU_IO_RS_RARM.LOG-RS-RARM-TX (UART TX)
- net UART_RS-RLEG_DIR: now also MCU_IO_RS_RLEG.118 (PD4 AF7 RTS/DE); no longer MCU_IO_RS_RLEG.LOG-RS-RLEG-DIR (DIRECTION)
- net UART_RS-RLEG_RX: now also MCU_IO_RS_RLEG.122 (PD6 AF7 RX); no longer MCU_IO_RS_RLEG.LOG-RS-RLEG-RX (UART RX)
- net UART_RS-RLEG_TX: now also MCU_IO_RS_RLEG.119 (PD5 AF7 TX); no longer MCU_IO_RS_RLEG.LOG-RS-RLEG-TX (UART TX)
- net UART_RS-WAIST_DIR: now also MCU_IO_RS_WAIST.110 (PA15 AF8 RTS/DE); no longer MCU_IO_RS_WAIST.LOG-RS-WAIST-DIR (DIRECTION)
- net UART_RS-WAIST_RX: now also MCU_IO_RS_WAIST.112 (PC11 AF8 RX); no longer MCU_IO_RS_WAIST.LOG-RS-WAIST-RX (UART RX)
- net UART_RS-WAIST_TX: now also MCU_IO_RS_WAIST.111 (PC10 AF8 TX); no longer MCU_IO_RS_WAIST.LOG-RS-WAIST-TX (UART TX)
- net UART_TTL-HEAD_DIR: now also MCU_IO_TTL_HEAD.86 (PD15 AF8 RTS/DE); no longer MCU_IO_TTL_HEAD.LOG-TTL-HEAD-DIR (DIRECTION)
- net UART_TTL-HEAD_TX: now also MCU_IO_TTL_HEAD.142 (PE1 AF8 HALF-DUPLEX IO); no longer MCU_IO_TTL_HEAD.LOG-TTL-HEAD-TX (UART TX)
- net UART_TTL-LDIST_DIR: now also MCU_IO_TTL_LDIST.98 (PC8 AF8 RTS/DE); no longer MCU_IO_TTL_LDIST.LOG-TTL-LDIST-DIR (DIRECTION)
- net UART_TTL-LDIST_TX: now also MCU_IO_TTL_LDIST.113 (PC12 AF8 HALF-DUPLEX IO); no longer MCU_IO_TTL_LDIST.LOG-TTL-LDIST-TX (UART TX)
- net UART_TTL-RDIST_DIR: now also MCU_IO_TTL_RDIST.63 (PE9 AF7 RTS/DE); no longer MCU_IO_TTL_RDIST.LOG-TTL-RDIST-DIR (DIRECTION)
- net UART_TTL-RDIST_TX: now also MCU_IO_TTL_RDIST.62 (PE8 AF7 HALF-DUPLEX IO); no longer MCU_IO_TTL_RDIST.LOG-TTL-RDIST-TX (UART TX)
- removed net UART_TTL-HEAD_RX: MCU_IO_TTL_HEAD.LOG-TTL-HEAD-RX (UART RX)
- removed net UART_TTL-LDIST_RX: MCU_IO_TTL_LDIST.LOG-TTL-LDIST-RX (UART RX)
- removed net UART_TTL-RDIST_RX: MCU_IO_TTL_RDIST.LOG-TTL-RDIST-RX (UART RX)
- no-connect marks 2 -> 5
Other:
- note removed: "W3037"
- note removed: "W3038"
- note removed: "W3039"
- moved on the sheet: MCU_IO_RS_LARM, MCU_IO_RS_LLEG, MCU_IO_RS_RARM, MCU_IO_RS_RLEG, MCU_IO_RS_WAIST, MCU_IO_TTL_HEAD, MCU_IO_TTL_LDIST, MCU_IO_TTL_RDIST

Commit message: Correct HR-30 whole-body electrical architecture
Connections:
- net WD_PERMIT_REQUEST: now reaches WD1.LOG-REQ (PERMIT REQUEST DIAGNOSTIC)
- no-connect marks 5 -> 4
Other:
- note added: "W3037"
Changed lines of the file:
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@@
               (at 309.88 52.61 0) (effects (font (size 1.27 1.27)) (justify bottom))
 )
-(no_connect (at 396.24 54.61)
+(wire (pts (xy 396.24 54.61) (xy 406.40 54.61))
+              (stroke (width 0) (type default)))
+(global_label "WD_PERMIT_REQUEST" (shape bidirectional) (at 406.40 54.61 0)
+              (fields_autoplaced yes) (effects (font (size 1.50 1.50)) (justify left))
+              (property "Intersheetrefs" "${INTERSHEET_REFS}" (at 406.40 57.15 0)
+                (effects (font (size 1.27 1.27)) (hide yes))))
+(text "W3016" (exclude_from_sim no)
+              (at 401.32 52.61 0) (effects (font (size 1.27 1.27)) (justify bottom))
 ) (wire (pts (xy 57.15 129.54) (xy 46.99 129.54))
               (stroke (width 0) (type default)))
@@
               (property "Intersheetrefs" "${INTERSHEET_REFS}" (at 46.99 132.08 0)
                 (effects (font (size 1.27 1.27)) (hide yes))))
-(text "W3016" (exclude_from_sim no)
+(text "W3017" (exclude_from_sim no)
               (at 52.07 127.54 0) (effects (font (size 1.27 1.27)) (justify bottom))
 )
@@
               (property "Intersheetrefs" "${INTERSHEET_REFS}" (at 46.99 127.00 0)
                 (effects (font (size 1.27 1.27)) (hide yes))))
-(text "W3017" (exclude_from_sim no)
+(text "W3018" (exclude_from_sim no)
               (at 52.07 122.46 0) (effects (font (size 1.27 1.27)) (justify bottom))
 )
@@
               (property "Intersheetrefs" "${INTERSHEET_REFS}" (at 46.99 121.92 0)
                 (effects (font (size 1.27 1.27)) (hide yes))))
-(text "W3018" (exclude_from_sim no)
+(text "W3019" (exclude_from_sim no)
               (at 52.07 117.38 0) (effects (font (size 1.27 1.27)) (justify bottom))
 ) (wire (pts (xy 373.38 129.54) (xy 383.54 129.54))
@@
               (property "Intersheetrefs" "${INTERSHEET_REFS}" (at 383.54 132.08 0)
                 (effects (font (size 1.27 1.27)) (hide yes))))
-(text "W3019" (exclude_from_sim no)
+(text "W3020" (exclude_from_sim no)
               (at 378.46 127.54 0) (effects (font (size 1.27 1.27)) (justify bottom))
 )
@@
               (property "Intersheetrefs" "${INTERSHEET_REFS}" (at 383.54 127.00 0)
                 (effects (font (size 1.27 1.27)) (hide yes))))
-(text "W3020" (exclude_from_sim no)
+(text "W3021" (exclude_from_sim no)
               (at 378.46 122.46 0) (effects (font (size 1.27 1.27)) (justify bottom))
 )
@@
               (property "Intersheetrefs" "${INTERSHEET_REFS}" (at 383.54 121.92 0)
                 (effects (font (size 1.27 1.27)) (hide yes))))
-(text "W3021" (exclude_from_sim no)
+(text "W3022" (exclude_from_sim no)
               (at 378.46 117.38 0) (effects (font (size 1.27 1.27)) (justify bottom))
 ) (wire (pts (xy 57.15 170.18) (xy 46.99 170.18))
@@
               (property "Intersheetrefs" "${INTERSHEET_REFS}" (at 46.99 172.72 0)
                 (effects (font (size 1.27 1.27)) (hide yes))))
-(text "W3022" (exclude_from_sim no)
+(text "W3023" (exclude_from_sim no)
               (at 52.07 168.18 0) (effects (font (size 1.27 1.27)) (justify bottom))
 )
@@
               (property "Intersheetrefs" "${INTERSHEET_REFS}" (at 46.99 167.64 0)
                 (effects (font (size 1.27 1.27)) (hide yes))))
-(text "W3023" (exclude_from_sim no)
+(text "W3024" (exclude_from_sim no)
               (at 52.07 163.10 0) (effects (font (size 1.27 1.27)) (justify bottom))
 )
@@
               (property "Intersheetrefs" "${INTERSHEET_REFS}" (at 46.99 162.56 0)
                 (effects (font (size 1.27 1.27)) (hide yes))))
-(text "W3024" (exclude_from_sim no)
+(text "W3025" (exclude_from_sim no)
               (at 52.07 158.02 0) (effects (font (size 1.27 1.27)) (justify bottom))
 ) (wire (pts (xy 373.38 170.18) (xy 383.54 170.18))
@@
               (property "Intersheetrefs" "${INTERSHEET_REFS}" (at 383.54 172.72 0)
                 (effects (font (size 1.27 1.27)) (hide yes))))
-(text "W3025" (exclude_from_sim no)
+(text "W3026" (exclude_from_sim no)
               (at 378.46 168.18 0) (effects (font (size 1.27 1.27)) (justify bottom))
 )
@@
               (property "Intersheetrefs" "${INTERSHEET_REFS}" (at 383.54 167.64 0)
                 (effects (font (size 1.27 1.27)) (hide yes))))
-(text "W3026" (exclude_from_sim no)
+(text "W3027" (exclude_from_sim no)
               (at 378.46 163.10 0) (effects (font (size 1.27 1.27)) (justify bottom))
 )
@@
               (property "Intersheetrefs" "${INTERSHEET_REFS}" (at 383.54 162.56 0)
                 (effects (font (size 1.27 1.27)) (hide yes))))
-(text "W3027" (exclude_from_sim no)
+(text "W3028" (exclude_from_sim no)
               (at 378.46 158.02 0) (effects (font (size 1.27 1.27)) (justify bottom))
 ) (wire (pts (xy 57.15 209.55) (xy 46.99 209.55))
@@
               (property "Intersheetrefs" "${INTERSHEET_REFS}" (at 46.99 212.09 0)
                 (effects (font (size 1.27 1.27)) (hide yes))))
-(text "W3028" (exclude_from_sim no)
+(text "W3029" (exclude_from_sim no)
               (at 52.07 207.55 0) (effects (font (size 1.27 1.27)) (justify bottom))
 )
@@
               (property "Intersheetrefs" "${INTERSHEET_REFS}" (at 46.99 207.01 0)
                 (effects (font (size 1.27 1.27)) (hide yes))))
-(text "W3029" (exclude_from_sim no)
+(text "W3030" (exclude_from_sim no)
               (at 52.07 202.47 0) (effects (font (size 1.27 1.27)) (justify bottom))
 )
@@
               (property "Intersheetrefs" "${INTERSHEET_REFS}" (at 46.99 201.93 0)
                 (effects (font (size 1.27 1.27)) (hide yes))))
-(text "W3030" (exclude_from_sim no)
+(text "W3031" (exclude_from_sim no)
               (at 52.07 197.39 0) (effects (font (size 1.27 1.27)) (justify bottom))
 ) (wire (pts (xy 373.38 209.55) (xy 383.54 209.55))
@@
               (property "Intersheetrefs" "${INTERSHEET_REFS}" (at 383.54 212.09 0)
                 (effects (font (size 1.27 1.27)) (hide yes))))
-(text "W3031" (exclude_from_sim no)
+(text "W3032" (exclude_from_sim no)
               (at 378.46 207.55 0) (effects (font (size 1.27 1.27)) (justify bottom))
 )
@@
               (property "Intersheetrefs" "${INTERSHEET_REFS}" (at 383.54 201.93 0)
                 (effects (font (size 1.27 1.27)) (hide yes))))
-(text "W3032" (exclude_from_sim no)
+(text "W3033" (exclude_from_sim no)
               (at 378.46 197.39 0) (effects (font (size 1.27 1.27)) (justify bottom))
 ) (wire (pts (xy 57.15 240.03) (xy 46.99 240.03))
@@
               (property "Intersheetrefs" "${INTERSHEET_REFS}" (at 46.99 242.57 0)
                 (effects (font (size 1.27 1.27)) (hide yes))))
-(text "W3033" (exclude_from_sim no)
+(text "W3034" (exclude_from_sim no)
               (at 52.07 238.03 0) (effects (font (size 1.27 1.27)) (justify bottom))
 )
@@
               (property "Intersheetrefs" "${INTERSHEET_REFS}" (at 46.99 232.41 0)
                 (effects (font (size 1.27 1.27)) (hide yes))))
-(text "W3034" (exclude_from_sim no)
+(text "W3035" (exclude_from_sim no)
               (at 52.07 227.87 0) (effects (font (size 1.27 1.27)) (justify bottom))
 ) (wire (pts (xy 373.38 240.03) (xy 383.54 240.03))
@@
               (property "Intersheetrefs" "${INTERSHEET_REFS}" (at 383.54 242.57 0)
                 (effects (font (size 1.27 1.27)) (hide yes))))
-(text "W3035" (exclude_from_sim no)
+(text "W3036" (exclude_from_sim no)
               (at 378.46 238.03 0) (effects (font (size 1.27 1.27)) (justify bottom))
 )
@@
               (property "Intersheetrefs" "${INTERSHEET_REFS}" (at 383.54 232.41 0)
                 (effects (font (size 1.27 1.27)) (hide yes))))
-(text "W3036" (exclude_from_sim no)
+(text "W3037" (exclude_from_sim no)
               (at 378.46 227.87 0) (effects (font (size 1.27 1.27)) (justify bottom))
 ) (text "NOTE 1: Conversational compute emits expiring high-level actions only; it never writes" (exclude_from_sim no) (at 17.78 260.00 0)

Commit message: Add HR-30 motion controller candidate
Connections:
- net UART_TTL-RDIST_DIR: now also MCU_IO_TTL_RDIST.60 (PE9 AF7 RTS/DE); no longer MCU_IO_TTL_RDIST.63 (PE9 AF7 RTS/DE)
- net UART_TTL-RDIST_TX: now also MCU_IO_TTL_RDIST.59 (PE8 AF7 HALF-DUPLEX IO); no longer MCU_IO_TTL_RDIST.62 (PE8 AF7 HALF-DUPLEX IO)
Changed lines of the file:
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@@
       (property "Evidence" "ST DS12110 Rev 11 LQFP144 pinout and alternate-function tables checked 2026-08-14." (at 115.57 234.95 0) (effects (font (size 1.50 1.50)) (hide yes)))
       (property "Display" "MCU1 UART7 PHYSICAL PIN UNIT - TTL-RDIST" (at 59.69 221.45 0) (effects (font (size 1.50 1.50)) (justify left bottom)))
-      (pin "62")
-      (pin "61")
-      (pin "63")
+      (pin "59")
+      (pin "58")
+      (pin "60")
       (instances (project "hr30-whole-body-electrical-p0.1" (path "/6dbc6f1c-d05b-56f0-8b51-042e5f8599ba/fd78e1fa-d6cc-51ca-87cc-a50b66f00db9" (reference "MCU_IO_TTL_RDIST") (unit 1)))))
 (symbol

Commit message: Integrate HR-30 three-rail auxiliary power
Connections:
- new net AUX_0V_STAR: CPU1.LOG-RET (AUXILIARY RETURN)
- new net COMPUTE_5V1: CPU1.LOG-5V (COMPUTE 5.1 V INPUT)
Other:
- note added: "W3038"
- note added: "W3039"
