File: hr30/whole-body-p0.1/electrical/kicad/hr30-whole-body-electrical-p0.1/04_motion_controller_carrier_connectors.kicad_sch (KiCad schematic)
At the start: 3 parts

Commit message: Add HR-30 motion controller candidate
Connections:
- net CTRL_3V3: now also JMCU_A.3 (CONTROL 3.3 V), JMCU_B.3 (CONTROL 3.3 V); no longer JMCU_A.2 (CONTROL 3.3 V), JMCU_B.2 (CONTROL 3.3 V)
- net CTRL_5V: now also JMCU_A.2 (CONTROL 5 V), JMCU_B.2 (CONTROL 5 V); no longer JMCU_A.1 (CONTROL 5 V), JMCU_B.1 (CONTROL 5 V)
- net CTRL_GND: now also JMCU_A.1 (CONTROL GROUND), JMCU_B.1 (CONTROL GROUND); no longer JMCU_A.3 (CONTROL GROUND), JMCU_B.3 (CONTROL GROUND)
Changed lines of the file:
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@@
 ) (wire (pts (xy 60.96 170.18) (xy 50.80 170.18))
               (stroke (width 0) (type default)))
-(global_label "CTRL_5V" (shape bidirectional) (at 50.80 170.18 180)
+(global_label "CTRL_GND" (shape bidirectional) (at 50.80 170.18 180)
               (fields_autoplaced yes) (effects (font (size 1.50 1.50)) (justify right))
               (property "Intersheetrefs" "${INTERSHEET_REFS}" (at 50.80 172.72 0)
@@
 (wire (pts (xy 60.96 165.10) (xy 50.80 165.10))
               (stroke (width 0) (type default)))
-(global_label "CTRL_3V3" (shape bidirectional) (at 50.80 165.10 180)
+(global_label "CTRL_5V" (shape bidirectional) (at 50.80 165.10 180)
               (fields_autoplaced yes) (effects (font (size 1.50 1.50)) (justify right))
               (property "Intersheetrefs" "${INTERSHEET_REFS}" (at 50.80 167.64 0)
@@
 (wire (pts (xy 60.96 160.02) (xy 50.80 160.02))
               (stroke (width 0) (type default)))
-(global_label "CTRL_GND" (shape bidirectional) (at 50.80 160.02 180)
+(global_label "CTRL_3V3" (shape bidirectional) (at 50.80 160.02 180)
               (fields_autoplaced yes) (effects (font (size 1.50 1.50)) (justify right))
               (property "Intersheetrefs" "${INTERSHEET_REFS}" (at 50.80 162.56 0)
@@
 ) (wire (pts (xy 251.46 170.18) (xy 241.30 170.18))
               (stroke (width 0) (type default)))
-(global_label "CTRL_5V" (shape bidirectional) (at 241.30 170.18 180)
+(global_label "CTRL_GND" (shape bidirectional) (at 241.30 170.18 180)
               (fields_autoplaced yes) (effects (font (size 1.50 1.50)) (justify right))
               (property "Intersheetrefs" "${INTERSHEET_REFS}" (at 241.30 172.72 0)
@@
 (wire (pts (xy 251.46 165.10) (xy 241.30 165.10))
               (stroke (width 0) (type default)))
-(global_label "CTRL_3V3" (shape bidirectional) (at 241.30 165.10 180)
+(global_label "CTRL_5V" (shape bidirectional) (at 241.30 165.10 180)
               (fields_autoplaced yes) (effects (font (size 1.50 1.50)) (justify right))
               (property "Intersheetrefs" "${INTERSHEET_REFS}" (at 241.30 167.64 0)
@@
 (wire (pts (xy 251.46 160.02) (xy 241.30 160.02))
               (stroke (width 0) (type default)))
-(global_label "CTRL_GND" (shape bidirectional) (at 241.30 160.02 180)
+(global_label "CTRL_3V3" (shape bidirectional) (at 241.30 160.02 180)
               (fields_autoplaced yes) (effects (font (size 1.50 1.50)) (justify right))
               (property "Intersheetrefs" "${INTERSHEET_REFS}" (at 241.30 162.56 0)

Commit message: Integrate HR-30 three-rail auxiliary power
Connections:
- net AUX_0V renamed AUX_0V_STAR
Changed lines of the file:
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@@
 (wire (pts (xy 147.32 62.23) (xy 137.16 62.23))
               (stroke (width 0) (type default)))
-(global_label "AUX_0V" (shape bidirectional) (at 137.16 62.23 180)
+(global_label "AUX_0V_STAR" (shape bidirectional) (at 137.16 62.23 180)
               (fields_autoplaced yes) (effects (font (size 1.50 1.50)) (justify right))
               (property "Intersheetrefs" "${INTERSHEET_REFS}" (at 137.16 64.77 0)
