File: hr30/whole-body-p0.1/electrical/kicad/hr30-whole-body-electrical-p0.1/14_head_ttl_sensors_hmi.kicad_sch (KiCad schematic)
At the start: 13 parts

Commit message: Correct HR-30 whole-body electrical architecture
Parts:
- removed PBR_TTL_HEAD: TTL-HEAD BRANCH PROTECTION / TELEMETRY - SELECTIO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, symbol PBV3:PBR_TTL_HEAD
- added PBR_HEAD_PAN: HEAD_PAN INDIVIDUAL PROTECTION / TELEMETRY - SELE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, symbol PBV3:PBR_HEAD_PAN
- added PBR_HEAD_TILT: HEAD_TILT INDIVIDUAL PROTECTION / TELEMETRY - SEL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, symbol PBV3:PBR_HEAD_TILT
Connections:
- net ACT_0V_CONTROLLED: now also PBR_HEAD_PAN.LOG-RET-IN (SOURCE RETURN), PBR_HEAD_TILT.LOG-RET-IN (SOURCE RETURN)
- net TTL-HEAD_RET: now also PBR_HEAD_PAN.LOG-RET-OUT (ACTUATOR / DATA REFERENCE), PBR_HEAD_TILT.LOG-RET-OUT (ACTUATOR / DATA REFERENCE)
- net TTL-HEAD_VDD renamed HEAD_PAN_VDD
- net HEAD_PAN_VDD: now also PBR_HEAD_PAN.LOG-OUT (PROTECTED ACTUATOR VDD); no longer AX_HEAD_TILT.2 (VDD)
- new net HEAD_TILT_VDD: AX_HEAD_TILT.2 (VDD), PBR_HEAD_TILT.LOG-OUT (PROTECTED ACTUATOR VDD)
- new net TTL_HEAD_SAFE_9V: PBR_HEAD_PAN.LOG-IN (INTERRUPTED SOURCE), PBR_HEAD_TILT.LOG-IN (INTERRUPTED SOURCE)
- no-connect marks 1 -> 2
Other:
- note added: "Connected TTL-HEAD data-only segment and one separately protected power feed per actuator."
- note added: "IDs, baud rate, cable, EMC, thermal and fault behavior remain unvalidated."
- note added: "NOTE 1: The listed axes share only data and reference. Each pin-2 VDD has a distinct"
- note added: "NOTE 3: A custom/de-pinned data-only harness or breakout is SELECTION REQUIRED. Termination,"
- note added: "W14045"
- note added: "W14046"
- note added: "W14047"
- note added: "W14048"
- note added: "protected feed; no standard VDD-carrying daisy cable may parallel those feeds."
- note removed: "Connected TTL-HEAD data segment and separately protected actuator-power branch."
- note removed: "NOTE 1: The segment shares data and branch power only among the listed axes; it does not"
- note removed: "NOTE 3: Termination, bias, actuator IDs, baud rate, cable length, waveform, latency, EMC,"
- note removed: "join any other protected branch VDD."
- note removed: "thermal and fault behavior remain unvalidated."
- moved on the sheet: AX_HEAD_PAN, AX_HEAD_TILT, PORT_TTL_HEAD

Commit message: Integrate HR-30 three-rail auxiliary power
Parts:
- HPWR1: value PROTECTED HEAD AUXILIARY DISTRIBUTION - DESIGN REQUIRED -> PROTECTED HEAD HMI DISTRIBUTION - DESIGN REQUIRED; Display PROTECTED HEAD AUXILIARY DISTRIBUTION - DESIGN REQUIRED -> PROTECTED HEAD HMI DISTRIBUTION - DESIGN REQUIRED
Connections:
- net AUX_0V renamed AUX_0V_STAR
- net AUX_5V_SAFE renamed HMI_5V0
Changed lines of the file:
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@@
 ) (wire (pts (xy 26.67 237.49) (xy 16.51 237.49))
               (stroke (width 0) (type default)))
-(global_label "AUX_5V_SAFE" (shape bidirectional) (at 16.51 237.49 180)
+(global_label "HMI_5V0" (shape bidirectional) (at 16.51 237.49 180)
               (fields_autoplaced yes) (effects (font (size 1.50 1.50)) (justify right))
               (property "Intersheetrefs" "${INTERSHEET_REFS}" (at 16.51 240.03 0)
@@
 (wire (pts (xy 26.67 232.41) (xy 16.51 232.41))
               (stroke (width 0) (type default)))
-(global_label "AUX_0V" (shape bidirectional) (at 16.51 232.41 180)
+(global_label "AUX_0V_STAR" (shape bidirectional) (at 16.51 232.41 180)
               (fields_autoplaced yes) (effects (font (size 1.50 1.50)) (justify right))
               (property "Intersheetrefs" "${INTERSHEET_REFS}" (at 16.51 234.95 0)
@@
       (exclude_from_sim no) (in_bom yes) (on_board yes) (dnp no)
       (property "Reference" "HPWR1" (at 29.21 218.25 0) (effects (font (size 1.50 1.50)) (justify left bottom)))
-      (property "Value" "PROTECTED HEAD AUXILIARY DISTRIBUTION - DESIGN REQUIRED" (at 69.85 234.95 0) (effects (font (size 1.50 1.50)) (hide yes)))
+      (property "Value" "PROTECTED HEAD HMI DISTRIBUTION - DESIGN REQUIRED" (at 69.85 234.95 0) (effects (font (size 1.50 1.50)) (hide yes)))
       (property "Footprint" "" (at 69.85 234.95 0) (effects (font (size 1.50 1.50)) (hide yes)))
       (property "Datasheet" "" (at 69.85 234.95 0) (effects (font (size 1.50 1.50)) (hide yes)))
-      (property "Description" "Branch protection, filtering, connector and current allocation remain open." (at 69.85 234.95 0) (effects (font (size 1.50 1.50)) (hide yes)))
+      (property "Description" "Branch protection, filtering, connector and current allocation remain open. The present coarse HMI peak equals the 30 W converter rating, so measured-load closure or redesign is mandatory." (at 69.85 234.95 0) (effects (font (size 1.50 1.50)) (hide yes)))
       (property "Status" "SELECTION REQUIRED - LOGICAL CONNECTIVITY ONLY" (at 69.85 250.65 0) (effects (font (size 1.50 1.50)) (justify bottom)))
       (property "Evidence" "" (at 69.85 234.95 0) (effects (font (size 1.50 1.50)) (hide yes)))
-      (property "Display" "PROTECTED HEAD AUXILIARY DISTRIBUTION - DESIGN REQUIRED" (at 29.21 221.45 0) (effects (font (size 1.50 1.50)) (justify left bottom)))
+      (property "Display" "PROTECTED HEAD HMI DISTRIBUTION - DESIGN REQUIRED" (at 29.21 221.45 0) (effects (font (size 1.50 1.50)) (justify left bottom)))
       (pin "LOG-IN")
       (pin "LOG-RET-IN")
