File: hr30/whole-body-p0.1/electrical/kicad/hr30-whole-body-electrical-p0.1/17_right_foot_load_sensing.kicad_sch (KiCad schematic)
At the start: 5 parts

Commit message: Integrate HR-30 three-rail auxiliary power
Connections:
- net AUX_0V renamed AUX_0V_STAR
Changed lines of the file:
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@@
 (wire (pts (xy 146.05 297.18) (xy 135.89 297.18))
               (stroke (width 0) (type default)))
-(global_label "AUX_0V" (shape bidirectional) (at 135.89 297.18 180)
+(global_label "AUX_0V_STAR" (shape bidirectional) (at 135.89 297.18 180)
               (fields_autoplaced yes) (effects (font (size 1.50 1.50)) (justify right))
               (property "Intersheetrefs" "${INTERSHEET_REFS}" (at 135.89 299.72 0)
