File: hr30/whole-body-p0.1/electrical/kicad/hr30-whole-body-electrical-p0.1/15_pelvis_aux_imu.kicad_sch (KiCad schematic)
At the start: 3 parts

Commit message: Correct HR-30 whole-body electrical architecture
Parts:
- AUXD1: value 14.8 V TO 5.1 V AUXILIARY CONVERTER - SELECTION REQUIRED -> CONTROLLED 12 V TO 5.1 V AUXILIARY CONVERTER - SELECTION REQUIRED; Display 14.8 V TO 5.1 V AUXILIARY CONVERTER - SELECTION REQUIRED -> CONTROLLED 12 V TO 5.1 V AUXILIARY CONVERTER - SELECTION RE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
Connections:
- net ACT_14V8_SAFE renamed ACT_MAIN_SAFE_12V
Changed lines of the file:
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@@
       (stroke (width 0.50) (type solid)) (fill (type none))) (wire (pts (xy 73.66 118.11) (xy 63.50 118.11))
               (stroke (width 0) (type default)))
-(global_label "ACT_14V8_SAFE" (shape bidirectional) (at 63.50 118.11 180)
+(global_label "ACT_MAIN_SAFE_12V" (shape bidirectional) (at 63.50 118.11 180)
               (fields_autoplaced yes) (effects (font (size 1.50 1.50)) (justify right))
               (property "Intersheetrefs" "${INTERSHEET_REFS}" (at 63.50 120.65 0)
@@
       (exclude_from_sim no) (in_bom yes) (on_board yes) (dnp no)
       (property "Reference" "AUXD1" (at 76.20 98.87 0) (effects (font (size 1.50 1.50)) (justify left bottom)))
-      (property "Value" "14.8 V TO 5.1 V AUXILIARY CONVERTER - SELECTION REQUIRED" (at 124.46 115.57 0) (effects (font (size 1.50 1.50)) (hide yes)))
+      (property "Value" "CONTROLLED 12 V TO 5.1 V AUXILIARY CONVERTER - SELECTION REQUIRED" (at 124.46 115.57 0) (effects (font (size 1.50 1.50)) (hide yes)))
       (property "Footprint" "" (at 124.46 115.57 0) (effects (font (size 1.50 1.50)) (hide yes)))
       (property "Datasheet" "" (at 124.46 115.57 0) (effects (font (size 1.50 1.50)) (hide yes)))
@@
       (property "Status" "SELECTION REQUIRED - LOGICAL CONNECTIVITY ONLY" (at 124.46 131.27 0) (effects (font (size 1.50 1.50)) (justify bottom)))
       (property "Evidence" "" (at 124.46 115.57 0) (effects (font (size 1.50 1.50)) (hide yes)))
-      (property "Display" "14.8 V TO 5.1 V AUXILIARY CONVERTER - SELECTION REQUIRED" (at 76.20 102.07 0) (effects (font (size 1.50 1.50)) (justify left bottom)))
+      (property "Display" "CONTROLLED 12 V TO 5.1 V AUXILIARY CONVERTER - SELECTION REQUIRED" (at 76.20 102.07 0) (effects (font (size 1.50 1.50)) (justify left bottom)))
       (pin "LOG-IN")
       (pin "LOG-RET-IN")

Commit message: Integrate HR-30 three-rail auxiliary power
Parts:
- removed AUXD1: CONTROLLED 12 V TO 5.1 V AUXILIARY CONVERTER - SE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, symbol PBV3:AUXD1
- added AUXCOM1: RECOM REC30E-2405SZ COMPUTE-RAIL CANDIDATE, symbol PBV3:AUXCOM1
- added AUXCTL1: RECOM REC30E-2405SZ CONTROL-RAIL CANDIDATE, symbol PBV3:AUXCTL1
- added AUXHMI1: RECOM REC30E-2405SZ HMI-RAIL CANDIDATE, symbol PBV3:AUXHMI1
- added AUXSTAR1: SINGLE PROPOSED AUXILIARY RETURN STAR / PE BOND B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, symbol PBV3:AUXSTAR1
Connections:
- net ACT_0V_CONTROLLED: now also AUXCOM1.LOG-RET-IN (CONTROLLED RETURN), AUXCTL1.LOG-RET-IN (CONTROLLED RETURN), AUXHMI1.LOG-RET-IN (CONTROLLED RETURN)
- net ACT_MAIN_SAFE_12V: now also AUXCOM1.LOG-IN (CONTROLLED 12 V INPUT), AUXCTL1.LOG-IN (CONTROLLED 12 V INPUT), AUXHMI1.LOG-IN (CONTROLLED 12 V INPUT)
- net AUX_5V_SAFE: now also AUXCTL1.LOG-OUT (CONTROL 5 V)
- net AUX_0V renamed AUX_0V_STAR
- net AUX_0V_STAR: now also AUXCOM1.LOG-RET-OUT (ISOLATED SECONDARY RETURN), AUXCTL1.LOG-RET-OUT (ISOLATED SECONDARY RETURN), AUXHMI1.LOG-RET-OUT (ISOLATED SECONDARY RETURN), AUXSTAR1.LOG-RET (COMMON SECONDARY RETURN)
- new net COMPUTE_5V1: AUXCOM1.LOG-OUT (COMPUTE 5.1 V)
- new net FRAME_PE_BOUNDARY: AUXSTAR1.LOG-PE (SOLE PROPOSED PE BOND)
- new net HMI_5V0: AUXHMI1.LOG-OUT (HMI 5 V)
- no-connect marks 1 -> 3
Other:
- note added: "15 Three-rail auxiliary conversion and pelvis inertial sensing"
- note added: "Three independent REC30E-2405SZ candidates supply compute, HMI and deterministic control; protection and validation remain open."
- note added: "W15013"
- note added: "W15014"
- note added: "W15015"
- note added: "W15016"
- note added: "W15017"
- note added: "W15018"
- note added: "W15019"
- note added: "W15020"
- note added: "W15021"
- note added: "W15022"
- note removed: "15 Auxiliary conversion and pelvis inertial sensing"
- note removed: "Logical 5 V auxiliary rail and pelvis IMU boundary."
- moved on the sheet: IMU1

Commit message: Increase HR-30 HMI power margin
Parts:
- AUXHMI1: value RECOM REC30E-2405SZ HMI-RAIL CANDIDATE -> TRACO POWER TEN 40-1211E HMI-RAIL CANDIDATE; Display RECOM REC30E-2405SZ HMI-RAIL CANDIDATE -> TRACO POWER TEN 40-1211E HMI-RAIL CANDIDATE
Other:
- note added: "Two REC30E-2405SZ candidates supply compute/control and one TEN 40-1211E supplies HMI; protection and validation remain open."
- note removed: "Three independent REC30E-2405SZ candidates supply compute, HMI and deterministic control; protection and validation remain open."
Changed lines of the file:
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@@
   (text "PRELIMINARY - NOT APPROVED FOR CONNECTION, FABRICATION, MOTION OR ENERGIZATION" (exclude_from_sim no) (at 17.78 10.16 0)
       (effects (font (size 2.54 2.54)) (justify left bottom))) (text "15  Three-rail auxiliary conversion and pelvis inertial sensing" (exclude_from_sim no) (at 17.78 19.05 0)
-      (effects (font (size 2.20 2.20)) (justify left bottom))) (text "Three independent REC30E-2405SZ candidates supply compute, HMI and deterministic control; protection and validation remain open." (exclude_from_sim no) (at 17.78 26.67 0)
+      (effects (font (size 2.20 2.20)) (justify left bottom))) (text "Two REC30E-2405SZ candidates supply compute/control and one TEN 40-1211E supplies HMI; protection and validation remain open." (exclude_from_sim no) (at 17.78 26.67 0)
       (effects (font (size 1.80 1.80)) (justify left bottom))) (rectangle (start 12.70 31.75) (end 406.40 281.94)
       (stroke (width 0.50) (type solid)) (fill (type none))) (wire (pts (xy 30.48 110.49) (xy 20.32 110.49))
@@
       (exclude_from_sim no) (in_bom yes) (on_board yes) (dnp no)
       (property "Reference" "AUXHMI1" (at 162.56 88.71 0) (effects (font (size 1.50 1.50)) (justify left bottom)))
-      (property "Value" "RECOM REC30E-2405SZ HMI-RAIL CANDIDATE" (at 214.63 105.41 0) (effects (font (size 1.50 1.50)) (hide yes)))
+      (property "Value" "TRACO POWER TEN 40-1211E HMI-RAIL CANDIDATE" (at 214.63 105.41 0) (effects (font (size 1.50 1.50)) (hide yes)))
       (property "Footprint" "" (at 214.63 105.41 0) (effects (font (size 1.50 1.50)) (hide yes)))
       (property "Datasheet" "" (at 214.63 105.41 0) (effects (font (size 1.50 1.50)) (hide yes)))
-      (property "Description" "The current coarse HMI peak is 30 W, leaving zero published headroom. Measured-load closure or redesign is mandatory; protection and validation remain open." (at 214.63 105.41 0) (effects (font (size 1.50 1.50)) (hide yes)))
+      (property "Description" "TEN 40E datasheet Rev. August 7, 2024: 9-18 V input, 5 V/8 A, 40 W. The 30 W coarse HMI peak has 10 W planning headroom; protection, physical load, transient, thermal, EMC and received-part FAI remain open." (at 214.63 105.41 0) (effects (font (size 1.50 1.50)) (hide yes)))
       (property "Status" "SELECTION REQUIRED - LOGICAL CONNECTIVITY ONLY" (at 214.63 121.11 0) (effects (font (size 1.50 1.50)) (justify bottom)))
       (property "Evidence" "" (at 214.63 105.41 0) (effects (font (size 1.50 1.50)) (hide yes)))
-      (property "Display" "RECOM REC30E-2405SZ HMI-RAIL CANDIDATE" (at 162.56 91.91 0) (effects (font (size 1.50 1.50)) (justify left bottom)))
+      (property "Display" "TRACO POWER TEN 40-1211E HMI-RAIL CANDIDATE" (at 162.56 91.91 0) (effects (font (size 1.50 1.50)) (justify left bottom)))
       (pin "LOG-IN")
       (pin "LOG-RET-IN")
