File: hr30/whole-body-p0.1/electrical/actuator-branch-pdu-p0.1/01_pdu_boundaries.kicad_sch (KiCad schematic)
At the start: 8 parts, among them J1 12 V CONTROLLED INPUT, J101 CHANNEL 1 OUTPUT, J102 CHANNEL 2 OUTPUT, J103 CHANNEL 3 OUTPUT, J104 CHANNEL 4 OUTPUT, J105 CHANNEL 5 OUTPUT, J106 CHANNEL 6 OUTPUT, J2 6x DISABLE_OD + 6x PG

Commit message: Route HR-30 actuator branch PDU
Parts:
- removed J2: 6x DISABLE_OD + 6x PG, Connector_JST:JST_GH_BM14B-GHS-TBT_1x14-1MP_P1.25mm_Vertical, symbol PBV3:J2
- added J201: CHANNEL 1 CONTROL, Connector_JST:JST_GH_BM03B-GHS-TBT_1x03-1MP_P1.25mm_Vertical, symbol PBV3:J201
- added J202: CHANNEL 2 CONTROL, Connector_JST:JST_GH_BM03B-GHS-TBT_1x03-1MP_P1.25mm_Vertical, symbol PBV3:J202
- added J203: CHANNEL 3 CONTROL, Connector_JST:JST_GH_BM03B-GHS-TBT_1x03-1MP_P1.25mm_Vertical, symbol PBV3:J203
- added J204: CHANNEL 4 CONTROL, Connector_JST:JST_GH_BM03B-GHS-TBT_1x03-1MP_P1.25mm_Vertical, symbol PBV3:J204
- added J205: CHANNEL 5 CONTROL, Connector_JST:JST_GH_BM03B-GHS-TBT_1x03-1MP_P1.25mm_Vertical, symbol PBV3:J205
- added J206: CHANNEL 6 CONTROL, Connector_JST:JST_GH_BM03B-GHS-TBT_1x03-1MP_P1.25mm_Vertical, symbol PBV3:J206
Connections:
- net CH1_EN: now also J201.2
- net CH1_PG: now also J201.3
- net CH2_EN: now also J202.2
- net CH2_PG: now also J202.3
- net CH3_EN: now also J203.2
- net CH3_PG: now also J203.3
- net CH4_EN: now also J204.2
- net CH4_PG: now also J204.3
- net CH5_EN: now also J205.2
- net CH5_PG: now also J205.3
- net CH6_EN: now also J206.2
- net CH6_PG: now also J206.3
- net PDU_0V: now also J201.1, J202.1, J203.1, J204.1, J205.1, J206.1
Other:
- note added: "NOTE 1: Each J20x GND/DISABLE_OD/PG boundary is ordinary control and diagnostics only; it"
- note added: "W1029"
- note added: "W1030"
- note added: "W1031"
- note added: "W1032"
- note added: "has zero safety credit."
- note removed: "NOTE 1: J2 DISABLE_OD/PG is ordinary control and diagnostics only; it has zero safety"
- note removed: "credit."
- moved on the sheet: J101, J102, J103, J104, J105, J106
