File: hr30/whole-body-p0.1/electrical/axis-commissioning-station-p0.1/01_current_limited_source.kicad_sch (KiCad schematic)
At the start: 2 parts, among them P1 POMONA 4933-2 / 4933-0 SHEATH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

Commit message: Select manufacturer-assembled HR-30 bench leads
Parts:
- P1: value POMONA 4933-2 / 4933-0 SHEATHED PLUG PAIR -> MUELLER BU-0061-M-39-2 / -39-0 LEAD PAIR; Display POMONA 4933-2 / 4933-0 SHEATHED PLUG PAIR -> MUELLER BU-0061-M-39-2 / -39-0 LEAD PAIR; Evidence live official product family; accessed 2026-08-15 -> DS-BU-0061-M-@; live official data sheet accessed 2026-08-15
Changed lines of the file:
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@@
       (exclude_from_sim no) (in_bom yes) (on_board yes) (dnp no)
       (property "Reference" "P1" (at 250.19 83.63 0) (effects (font (size 1.50 1.50)) (justify left bottom)))
-      (property "Value" "POMONA 4933-2 / 4933-0 SHEATHED PLUG PAIR" (at 304.80 100.33 0) (effects (font (size 1.50 1.50)) (hide yes)))
+      (property "Value" "MUELLER BU-0061-M-39-2 / -39-0 LEAD PAIR" (at 304.80 100.33 0) (effects (font (size 1.50 1.50)) (hide yes)))
       (property "Footprint" "" (at 304.80 100.33 0) (effects (font (size 1.50 1.50)) (hide yes)))
-      (property "Datasheet" "https://www.pomonaelectronics.com/products/banana-plugs-jacks-and-hardware/banana-plugs-and-jacks" (at 304.80 100.33 0) (effects (font (size 1.50 1.50)) (hide yes)))
-      (property "Description" "One metre bench lead candidate. No stacking, adapters or exposed clip ends. Polarity and insulation require 100% inspection." (at 304.80 100.33 0) (effects (font (size 1.50 1.50)) (hide yes)))
+      (property "Datasheet" "https://www.muellerelectric.com/product_files/21/DS-BU-0061-M-%40.pdf" (at 304.80 100.33 0) (effects (font (size 1.50 1.50)) (hide yes)))
+      (property "Description" "Manufacturer-assembled 39 inch shrouded-banana leads with 18 AWG silicone cable and tin-dipped free ends. The dipped portions are sacrificial and must not enter the Mini-Fit crimp. Received wire OD/material, fresh-cut preparation, polarity and insulation require 100% inspection." (at 304.80 100.33 0) (effects (font (size 1.50 1.50)) (hide yes)))
       (property "Status" "CANDIDATE / VALIDATION OPEN" (at 304.80 116.03 0) (effects (font (size 1.50 1.50)) (justify bottom)))
-      (property "Evidence" "live official product family; accessed 2026-08-15" (at 304.80 100.33 0) (effects (font (size 1.50 1.50)) (hide yes)))
-      (property "Display" "POMONA 4933-2 / 4933-0 SHEATHED PLUG PAIR" (at 250.19 86.83 0) (effects (font (size 1.50 1.50)) (justify left bottom)))
+      (property "Evidence" "DS-BU-0061-M-@; live official data sheet accessed 2026-08-15" (at 304.80 100.33 0) (effects (font (size 1.50 1.50)) (hide yes)))
+      (property "Display" "MUELLER BU-0061-M-39-2 / -39-0 LEAD PAIR" (at 250.19 86.83 0) (effects (font (size 1.50 1.50)) (justify left bottom)))
       (pin "RED")
       (pin "BLACK")
