File: hr30/whole-body-p0.1/electrical/axis-commissioning-station-p0.1/02_power_hub_and_usb.kicad_sch (KiCad schematic)
At the start: 3 parts, among them J1 MOLEX 39-01-2020 / 39-00-0038, U1 ROBOTIS U2D2 902-0132-000

Commit message: Select manufacturer-assembled HR-30 bench leads
Parts:
- J1: Evidence Mini-Fit Jr application-tooling specification accessed 2026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 -> 638190901 Rev D; 2025-03-31; accessed 2026-08-15
Changed lines of the file:
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@@
       (property "Value" "MOLEX 39-01-2020 / 39-00-0038" (at 90.17 100.33 0) (effects (font (size 1.50 1.50)) (hide yes)))
       (property "Footprint" "" (at 90.17 100.33 0) (effects (font (size 1.50 1.50)) (hide yes)))
-      (property "Datasheet" "https://www.molex.com/content/dam/molex/molex-dot-com/products/automated/en-us/applicationtoolingspecificationpdf/638/63860/ATS-638601000-001.pdf" (at 90.17 100.33 0) (effects (font (size 1.50 1.50)) (hide yes)))
-      (property "Description" "20 AWG Alpha 3073 red/black lead into the PHB Mini-Fit Jr input. Contact crimp height, pull test and received polarity remain validation work." (at 90.17 100.33 0) (effects (font (size 1.50 1.50)) (hide yes)))
+      (property "Datasheet" "https://www.molex.com/content/dam/molex/molex-dot-com/products/automated/en-us/applicationtoolingspecificationpdf/638/63819/638190901-000.pdf" (at 90.17 100.33 0) (effects (font (size 1.50 1.50)) (hide yes)))
+      (property "Description" "18 AWG Mueller BU-0061-M red/black leads into the PHB Mini-Fit Jr input after complete removal of the tin-dipped free-end segment. Received cable OD/material, contact crimp height, pull test and polarity remain validation work." (at 90.17 100.33 0) (effects (font (size 1.50 1.50)) (hide yes)))
       (property "Status" "CANDIDATE / VALIDATION OPEN" (at 90.17 116.03 0) (effects (font (size 1.50 1.50)) (justify bottom)))
-      (property "Evidence" "Mini-Fit Jr application-tooling specification accessed 2026-08-15" (at 90.17 100.33 0) (effects (font (size 1.50 1.50)) (hide yes)))
+      (property "Evidence" "638190901 Rev D; 2025-03-31; accessed 2026-08-15" (at 90.17 100.33 0) (effects (font (size 1.50 1.50)) (hide yes)))
       (property "Display" "MOLEX 39-01-2020 / 39-00-0038" (at 40.64 86.83 0) (effects (font (size 1.50 1.50)) (justify left bottom)))
       (pin "1")
