File: hr30/whole-body-p0.1/electrical/tether-power-core-p0.1/03_redundant_dc_interruption.kicad_sch (KiCad schematic)
At the start: 3 parts, among them K1 SENSATA GIGAVAC GV121CAC, K2 SENSATA GIGAVAC GV121CAC

Commit message: Complete HR-30 safety and clean-build package
Parts:
- K1: value SENSATA GIGAVAC GV121CAC -> SCHNEIDER TESYS DECA LC1D40ABD; Display SENSATA GIGAVAC GV121CAC -> SCHNEIDER TESYS DECA LC1D40ABD; Evidence GV12 series Rev 28-Apr-2022 -> MKTED210011EN v17.1, 2026-07-10, A5/120-A5/123; product pag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; Status EXACT ORDER-CODE CANDIDATE - NOT AN IEC MIRROR-CONTACT CLAIM -> EXACT ORDER-CODE / MIRROR CONTACT VERIFIED - APPLICATION VA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
- K2: value SENSATA GIGAVAC GV121CAC -> SCHNEIDER TESYS DECA LC1D40ABD; Display SENSATA GIGAVAC GV121CAC -> SCHNEIDER TESYS DECA LC1D40ABD; Evidence GV12 series Rev 28-Apr-2022 -> MKTED210011EN v17.1, 2026-07-10, A5/120-A5/123; product pag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; Status EXACT ORDER-CODE CANDIDATE - APPLICATION OPEN -> EXACT ORDER-CODE / MIRROR CONTACT VERIFIED - APPLICATION VA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
Connections:
- net EDM_K1_OUT: now also K1.22 (MIRROR NC RETURN), K2.21 (MIRROR NC COMMON); no longer K1.AUX-NC (NC AUX RETURN), K2.AUX-C (NC AUX COMMON)
- net K1_COIL_POS: now also K1.A1 (24 VDC COIL POSITIVE); no longer K1.COIL+ (24 V COIL POSITIVE)
- net K1_OUT: now also K1.6/T3 (MAIN POLE 3 OUTPUT), K2.1/L1 (MAIN POLE 1 INPUT); no longer K1.M2 (MAIN OUTPUT STUD), K2.M1 (MAIN INPUT STUD)
- net K2_COIL_POS: now also K2.A1 (24 VDC COIL POSITIVE); no longer K2.COIL+ (24 V COIL POSITIVE)
- net RAW_12V_POS: now also K1.1/L1 (MAIN POLE 1 INPUT); no longer K1.M1 (MAIN INPUT STUD)
- net RESET_EDM: now also K1.21 (MIRROR NC COMMON), K2.22 (MIRROR NC RETURN); no longer K1.AUX-C (NC AUX COMMON), K2.AUX-NC (NC AUX RETURN)
- net SAFE_0V: now also K1.A2 (COIL RETURN), K2.A2 (COIL RETURN); no longer K1.COIL- (COIL RETURN), K2.COIL- (COIL RETURN)
- net TETHER_POS_SWITCHED: now also K2.6/T3 (MAIN POLE 3 OUTPUT); no longer K2.M2 (MAIN OUTPUT STUD)
- new net K1_POLE2_IN: K1.2/T1 (MAIN POLE 1 OUTPUT), K1.3/L2 (MAIN POLE 2 INPUT)
- new net K1_POLE3_IN: K1.4/T2 (MAIN POLE 2 OUTPUT), K1.5/L3 (MAIN POLE 3 INPUT)
- new net K2_POLE2_IN: K2.2/T1 (MAIN POLE 1 OUTPUT), K2.3/L2 (MAIN POLE 2 INPUT)
- new net K2_POLE3_IN: K2.4/T2 (MAIN POLE 2 OUTPUT), K2.5/L3 (MAIN POLE 3 INPUT)
- no-connect marks 0 -> 4
Other:
- note added: "03 Two series LC1D40ABD contactors and mirror-feedback loop"
- note added: "External-panel three-pole-series DC interruption candidate; no achieved safety-performance claim."
- note added: "NOTE 1: Both high-current contactors are in the external panel, not on the robot. Each"
- note added: "NOTE 2: Schneider identifies built-in 21-22 as an IEC 60947-4-1 mirror contact. This"
- note added: "W3015"
- note added: "W3016"
- note added: "W3017"
- note added: "W3018"
- note added: "W3019"
- note added: "W3020"
- note added: "W3021"
- note added: "W3022"
- note added: "contactor's three main poles are wired in series; K1 and K2 remain independent"
- note added: "machine safety claim is made."
- note added: "series interruption elements."
- note added: "supports the proposed EDM architecture only; no achieved Category, PL, SIL or whole-"
- note removed: "03 Two series GV121CAC contactors and feedback loop"
- note removed: "External-panel DC interruption candidate; no safety-performance claim."
- note removed: "NOTE 1: Both high-current contactors are in the external panel, not on the robot."
- note removed: "NOTE 2: The GV12 auxiliary is manufacturer-described as mechanically linked; this package"
- note removed: "does not call it an IEC mirror contact or claim a safety category."
