File: hr30/whole-body-p0.1/electrical/walking-power-successor-p0.1/01_system_boundaries.kicad_sch (KiCad schematic)
At the start: 14 parts, among them J1 12 V CONTROLLED INPUT, J1C CHANNEL 1 CONTROL/MONITOR, J1O CHANNEL 1 AXIS OUTPUT, J2C CHANNEL 2 CONTROL/MONITOR, J2O CHANNEL 2 AXIS OUTPUT, J3C CHANNEL 3 CONTROL/MONITOR, J3O CHANNEL 3 AXIS OUTPUT, J4C CHANNEL 4 CONTROL/MONITOR, J4O CHANNEL 4 AXIS OUTPUT, J5C CHANNEL 5 CONTROL/MONITOR, J5O CHANNEL 5 AXIS OUTPUT, J6C CHANNEL 6 CONTROL/MONITOR, J6O CHANNEL 6 AXIS OUTPUT

Commit message: Correct HR-30 whole-body power and harness architecture (#48)
Validated whole-body correction; preserves all preliminary and no-energization holds.
Parts:
- J1: value 12 V CONTROLLED INPUT -> CONTROLLED BUS-FEED INPUT; Display 12 V CONTROLLED INPUT -> CONTROLLED BUS-FEED INPUT; Evidence existing five-feed input boundary; exact terminal and produ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 -> one isolated board input per authoritative bus; exact termi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
Connections:
- net BRANCH_1_12V renamed BRANCH_1_VPOS
- net BRANCH_2_12V renamed BRANCH_2_VPOS
- net BRANCH_3_12V renamed BRANCH_3_VPOS
- net BRANCH_4_12V renamed BRANCH_4_VPOS
- net BRANCH_5_12V renamed BRANCH_5_VPOS
- net BRANCH_6_12V renamed BRANCH_6_VPOS
- net PDU_0V renamed FEED_0V
- net PDU_12V_IN renamed FEED_VPOS
Other:
- note added: "01 Eight isolated bus feeds and six-channel board pattern"
- note added: "NOTE 1: Each of eight board instances receives exactly one authoritative bus feed; no"
- note added: "NOTE 2: JBRK is a real downstream interface obligation, not a released resistor/chopper"
- note added: "NOTE 3: Each axis output is an individual power pair; data harnesses remain data-only."
- note added: "NOTE 4: PRELIMINARY - WALKING-POWER ARCHITECTURE CANDIDATE ONLY - NOT APPROVED FOR"
- note added: "One board pattern is instantiated once per authoritative actuator bus; 25 channels populated and 23 DNP."
- note added: "left/right or 9 V domains are tied together."
- note removed: "01 Five-feed and six-channel board boundaries"
- note removed: "NOTE 1: JBRK is a real downstream interface obligation, not a released resistor/chopper"
- note removed: "NOTE 2: Each axis output is an individual power pair; data harnesses remain data-only."
- note removed: "NOTE 3: PRELIMINARY - WALKING-POWER ARCHITECTURE CANDIDATE ONLY - NOT APPROVED FOR"
- note removed: "One board pattern is instantiated five times; 25 channels populated and five DNP."
