File: hr30/whole-body-p0.1/electrical/walking-power-successor-p0.1/03_paired_channel_2.kicad_sch (KiCad schematic)
At the start: 10 parts, among them U2F TPS259482L FORWARD OCP, U2R TPS259482L REVERSE OCP

Commit message: Correct HR-30 whole-body power and harness architecture (#48)
Validated whole-body correction; preserves all preliminary and no-energization holds.
Connections:
- net BRANCH_2_12V renamed BRANCH_2_VPOS
- net PDU_0V renamed FEED_0V
- net PDU_12V_IN renamed FEED_VPOS
Other:
- note added: "NOTE 4: Eight isolated bus-domain brake/dump circuits are still required for contactor-open"
- note added: "energy."
- note removed: "NOTE 4: Five downstream brake/dump circuits are still required for contactor-open energy."
Changed lines of the file:
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@@
 (wire (pts (xy 7.62 46.99) (xy -2.54 46.99))
               (stroke (width 0) (type default)))
-(global_label "PDU_12V_IN" (shape bidirectional) (at -2.54 46.99 180)
+(global_label "FEED_VPOS" (shape bidirectional) (at -2.54 46.99 180)
               (fields_autoplaced yes) (effects (font (size 1.50 1.50)) (justify right))
               (property "Intersheetrefs" "${INTERSHEET_REFS}" (at -2.54 49.53 0)
@@
 (wire (pts (xy 101.60 41.91) (xy 111.76 41.91))
               (stroke (width 0) (type default)))
-(global_label "PDU_0V" (shape bidirectional) (at 111.76 41.91 0)
+(global_label "FEED_0V" (shape bidirectional) (at 111.76 41.91 0)
               (fields_autoplaced yes) (effects (font (size 1.50 1.50)) (justify left))
               (property "Intersheetrefs" "${INTERSHEET_REFS}" (at 111.76 44.45 0)
@@
 (wire (pts (xy 101.60 31.75) (xy 111.76 31.75))
               (stroke (width 0) (type default)))
-(global_label "PDU_12V_IN" (shape bidirectional) (at 111.76 31.75 0)
+(global_label "FEED_VPOS" (shape bidirectional) (at 111.76 31.75 0)
               (fields_autoplaced yes) (effects (font (size 1.50 1.50)) (justify left))
               (property "Intersheetrefs" "${INTERSHEET_REFS}" (at 111.76 34.29 0)
@@
 (wire (pts (xy 152.40 46.99) (xy 142.24 46.99))
               (stroke (width 0) (type default)))
-(global_label "BRANCH_2_12V" (shape bidirectional) (at 142.24 46.99 180)
+(global_label "BRANCH_2_VPOS" (shape bidirectional) (at 142.24 46.99 180)
               (fields_autoplaced yes) (effects (font (size 1.50 1.50)) (justify right))
               (property "Intersheetrefs" "${INTERSHEET_REFS}" (at 142.24 49.53 0)
@@
 (wire (pts (xy 246.38 41.91) (xy 256.54 41.91))
               (stroke (width 0) (type default)))
-(global_label "PDU_0V" (shape bidirectional) (at 256.54 41.91 0)
+(global_label "FEED_0V" (shape bidirectional) (at 256.54 41.91 0)
               (fields_autoplaced yes) (effects (font (size 1.50 1.50)) (justify left))
               (property "Intersheetrefs" "${INTERSHEET_REFS}" (at 256.54 44.45 0)
@@
 (wire (pts (xy 246.38 31.75) (xy 256.54 31.75))
               (stroke (width 0) (type default)))
-(global_label "BRANCH_2_12V" (shape bidirectional) (at 256.54 31.75 0)
+(global_label "BRANCH_2_VPOS" (shape bidirectional) (at 256.54 31.75 0)
               (fields_autoplaced yes) (effects (font (size 1.50 1.50)) (justify left))
               (property "Intersheetrefs" "${INTERSHEET_REFS}" (at 256.54 34.29 0)
@@
 (wire (pts (xy 391.16 44.45) (xy 401.32 44.45))
               (stroke (width 0) (type default)))
-(global_label "PDU_0V" (shape bidirectional) (at 401.32 44.45 0)
+(global_label "FEED_0V" (shape bidirectional) (at 401.32 44.45 0)
               (fields_autoplaced yes) (effects (font (size 1.50 1.50)) (justify left))
               (property "Intersheetrefs" "${INTERSHEET_REFS}" (at 401.32 46.99 0)
@@
 (wire (pts (xy 101.60 111.76) (xy 111.76 111.76))
               (stroke (width 0) (type default)))
-(global_label "PDU_0V" (shape bidirectional) (at 111.76 111.76 0)
+(global_label "FEED_0V" (shape bidirectional) (at 111.76 111.76 0)
               (fields_autoplaced yes) (effects (font (size 1.50 1.50)) (justify left))
               (property "Intersheetrefs" "${INTERSHEET_REFS}" (at 111.76 114.30 0)
@@
 (wire (pts (xy 246.38 111.76) (xy 256.54 111.76))
               (stroke (width 0) (type default)))
-(global_label "PDU_0V" (shape bidirectional) (at 256.54 111.76 0)
+(global_label "FEED_0V" (shape bidirectional) (at 256.54 111.76 0)
               (fields_autoplaced yes) (effects (font (size 1.50 1.50)) (justify left))
               (property "Intersheetrefs" "${INTERSHEET_REFS}" (at 256.54 114.30 0)
@@
 (wire (pts (xy 391.16 111.76) (xy 401.32 111.76))
               (stroke (width 0) (type default)))
-(global_label "PDU_0V" (shape bidirectional) (at 401.32 111.76 0)
+(global_label "FEED_0V" (shape bidirectional) (at 401.32 111.76 0)
               (fields_autoplaced yes) (effects (font (size 1.50 1.50)) (justify left))
               (property "Intersheetrefs" "${INTERSHEET_REFS}" (at 401.32 114.30 0)
@@
 (wire (pts (xy 101.60 179.07) (xy 111.76 179.07))
               (stroke (width 0) (type default)))
-(global_label "PDU_0V" (shape bidirectional) (at 111.76 179.07 0)
+(global_label "FEED_0V" (shape bidirectional) (at 111.76 179.07 0)
               (fields_autoplaced yes) (effects (font (size 1.50 1.50)) (justify left))
               (property "Intersheetrefs" "${INTERSHEET_REFS}" (at 111.76 181.61 0)
@@
 (wire (pts (xy 246.38 179.07) (xy 256.54 179.07))
               (stroke (width 0) (type default)))
-(global_label "PDU_0V" (shape bidirectional) (at 256.54 179.07 0)
+(global_label "FEED_0V" (shape bidirectional) (at 256.54 179.07 0)
               (fields_autoplaced yes) (effects (font (size 1.50 1.50)) (justify left))
               (property "Intersheetrefs" "${INTERSHEET_REFS}" (at 256.54 181.61 0)
@@
 ) (wire (pts (xy 297.18 179.07) (xy 287.02 179.07))
               (stroke (width 0) (type default)))
-(global_label "PDU_12V_IN" (shape bidirectional) (at 287.02 179.07 180)
+(global_label "FEED_VPOS" (shape bidirectional) (at 287.02 179.07 180)
               (fields_autoplaced yes) (effects (font (size 1.50 1.50)) (justify right))
               (property "Intersheetrefs" "${INTERSHEET_REFS}" (at 287.02 181.61 0)
@@
 (wire (pts (xy 391.16 179.07) (xy 401.32 179.07))
               (stroke (width 0) (type default)))
-(global_label "PDU_0V" (shape bidirectional) (at 401.32 179.07 0)
+(global_label "FEED_0V" (shape bidirectional) (at 401.32 179.07 0)
               (fields_autoplaced yes) (effects (font (size 1.50 1.50)) (justify left))
               (property "Intersheetrefs" "${INTERSHEET_REFS}" (at 401.32 181.61 0)
@@
 ) (wire (pts (xy 7.62 246.38) (xy -2.54 246.38))
               (stroke (width 0) (type default)))
-(global_label "BRANCH_2_12V" (shape bidirectional) (at -2.54 246.38 180)
+(global_label "BRANCH_2_VPOS" (shape bidirectional) (at -2.54 246.38 180)
               (fields_autoplaced yes) (effects (font (size 1.50 1.50)) (justify right))
               (property "Intersheetrefs" "${INTERSHEET_REFS}" (at -2.54 248.92 0)
@@
 (wire (pts (xy 101.60 246.38) (xy 111.76 246.38))
               (stroke (width 0) (type default)))
-(global_label "PDU_0V" (shape bidirectional) (at 111.76 246.38 0)
+(global_label "FEED_0V" (shape bidirectional) (at 111.76 246.38 0)
               (fields_autoplaced yes) (effects (font (size 1.50 1.50)) (justify left))
               (property "Intersheetrefs" "${INTERSHEET_REFS}" (at 111.76 248.92 0)
@@
       (effects (font (size 1.50 1.50)) (justify left bottom))) (text "NOTE 2: Regeneration: UxR provides IN-to-OUT overcurrent protection." (exclude_from_sim no) (at 17.78 265.50 0)
       (effects (font (size 1.50 1.50)) (justify left bottom))) (text "NOTE 3: A single TPS25948 is insufficient because reverse-direction OCP is not provided." (exclude_from_sim no) (at 17.78 271.00 0)
-      (effects (font (size 1.50 1.50)) (justify left bottom))) (text "NOTE 4: Five downstream brake/dump circuits are still required for contactor-open energy." (exclude_from_sim no) (at 17.78 276.50 0)
-      (effects (font (size 1.50 1.50)) (justify left bottom))) (text "NOTE 5: PRELIMINARY - WALKING-POWER ARCHITECTURE CANDIDATE ONLY - NOT APPROVED FOR" (exclude_from_sim no) (at 17.78 282.00 0)
-      (effects (font (size 1.50 1.50)) (justify left bottom))) (text "        PROCUREMENT, FABRICATION, CONNECTION, POWERED TESTING, MOTION OR ENERGIZATION" (exclude_from_sim no) (at 17.78 287.50 0)
+      (effects (font (size 1.50 1.50)) (justify left bottom))) (text "NOTE 4: Eight isolated bus-domain brake/dump circuits are still required for contactor-open" (exclude_from_sim no) (at 17.78 276.50 0)
+      (effects (font (size 1.50 1.50)) (justify left bottom))) (text "        energy." (exclude_from_sim no) (at 17.78 282.00 0)
+      (effects (font (size 1.50 1.50)) (justify left bottom))) (text "NOTE 5: PRELIMINARY - WALKING-POWER ARCHITECTURE CANDIDATE ONLY - NOT APPROVED FOR" (exclude_from_sim no) (at 17.78 287.50 0)
+      (effects (font (size 1.50 1.50)) (justify left bottom))) (text "        PROCUREMENT, FABRICATION, CONNECTION, POWERED TESTING, MOTION OR ENERGIZATION" (exclude_from_sim no) (at 17.78 293.00 0)
       (effects (font (size 1.50 1.50)) (justify left bottom)))
   (symbol

Commit message: Add routed HR-30 walking-power PCB candidate
Parts:
- added R2OF: 0R OVLO FORWARD PULLDOWN CANDIDATE, Resistor_SMD:R_0603_1608Metric, symbol PBV3:R2OF
- added R2OR: 0R OVLO REVERSE PULLDOWN CANDIDATE, Resistor_SMD:R_0603_1608Metric, symbol PBV3:R2OR
- U2F, U2R: footprint (none) -> ProjectButton_WPS:TI_YWP0012A_PowerWCSP_2.441x1.728mm; Evidence TPS259482LYWPR candidate; native footprint deliberately bla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 -> TPS259482LYWPR candidate on exact TI YWP0012A example land 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
Connections:
- net FEED_0V: now also R2OF.2, R2OR.2
- net CH2_OV_R: now reaches U2R.2
- net CH2_OV_R: now also R2OR.1
- net CH2_OV_F: now reaches U2F.2
- net CH2_OV_F: now also R2OF.1
- no-connect marks 4 -> 2
Other:
- note added: "W3037"
- note added: "W3038"
- note added: "W3039"
- note added: "W3040"
- note added: "W3041"
- note added: "W3042"
- moved on the sheet: C2F, C2I, C2O, C2R
