Commit message: Lighten HR-30 joint carrier topology

File: release/hr30/whole-body-p0.1/hr30.urdf (robot description, URDF)
Before this commit: robot hr30_whole_body_p01, 26 links, 25 joints
Links:
- link L_forearm: mass 0.127975 -> 0.125225
- link L_hand: mass 0.059216 -> 0.055657
- link L_shin: mass 0.784854 -> 0.745112
- link L_shoulder_pitch_link: mass 0.298024 -> 0.280768
- link L_thigh: mass 1.713300 -> 1.642432
- link L_upper_arm: mass 0.489145 -> 0.465854
- link R_forearm: mass 0.127975 -> 0.125225
- link R_hand: mass 0.059216 -> 0.055657
- link R_shin: mass 0.784854 -> 0.745112
- link R_shoulder_pitch_link: mass 0.298024 -> 0.280768
- link R_thigh: mass 1.713300 -> 1.642432
- link R_upper_arm: mass 0.489145 -> 0.465854
- link base_link: mass 1.702403 -> 1.686946
- link head: mass 0.433766 -> 0.431016
- link neck_pan_link: mass 0.123901 -> 0.121151

Commit message: Complete HR-30 whole-body transmission architecture

File: release/hr30/whole-body-p0.1/hr30.urdf (robot description, URDF)
Before this commit: robot hr30_whole_body_p01, 26 links, 25 joints
Links:
- link L_shoulder_pitch_link: mass 0.280768 -> 0.283380
- link L_upper_arm: mass 0.465854 -> 0.468466
- link R_shoulder_pitch_link: mass 0.280768 -> 0.283380
- link R_upper_arm: mass 0.465854 -> 0.468466

Commit message: Lightweight HR-30 whole-body candidate

File: release/hr30/whole-body-p0.1/hr30.urdf (robot description, URDF)
Before this commit: robot hr30_whole_body_p01, 26 links, 25 joints
Links:
- link L_foot: mass 0.211981 -> 0.167444
- link L_forearm: mass 0.120221 -> 0.113606
- link L_shin: mass 0.705487 -> 0.697911
- link L_thigh: mass 1.638884 -> 1.630169
- link L_upper_arm: mass 0.453947 -> 0.446793
- link R_foot: mass 0.211981 -> 0.167444
- link R_forearm: mass 0.120221 -> 0.113606
- link R_shin: mass 0.705487 -> 0.697911
- link R_thigh: mass 1.638884 -> 1.630169
- link R_upper_arm: mass 0.453947 -> 0.446793
- link base_link: mass 1.592722 -> 1.550063
- link head: mass 0.439477 -> 0.418231
- link torso: mass 2.560361 -> 2.499749

File: release/hr30/whole-body-p0.1/hr30_tether.urdf (robot description, URDF)
Before this commit: robot hr30_whole_body_p01, 26 links, 25 joints
Links:
- link L_foot: mass 0.211981 -> 0.167444
- link L_forearm: mass 0.120221 -> 0.113606
- link L_shin: mass 0.705487 -> 0.697911
- link L_thigh: mass 1.638884 -> 1.630169
- link L_upper_arm: mass 0.453947 -> 0.446793
- link R_foot: mass 0.211981 -> 0.167444
- link R_forearm: mass 0.120221 -> 0.113606
- link R_shin: mass 0.705487 -> 0.697911
- link R_thigh: mass 1.638884 -> 1.630169
- link R_upper_arm: mass 0.453947 -> 0.446793
- link base_link: mass 1.592722 -> 1.550063
- link head: mass 0.439477 -> 0.418231
- link torso: mass 1.094801 -> 1.034189
