Commit message: Reconcile HR-30 whole-body mass model

File: hr30/whole-body-p0.1/hr30.urdf (robot description, URDF)
Before this commit: robot hr30_whole_body_p01, 26 links, 25 joints
Links:
- link L_forearm: mass 0.220000 -> 0.245747
- link L_shin: mass 0.470000 -> 1.375365
- link L_shoulder_pitch_link: mass 0.100000 -> 0.346898
- link L_thigh: mass 0.660000 -> 2.468826
- link L_upper_arm: mass 0.270000 -> 0.785245
- link R_forearm: mass 0.220000 -> 0.245747
- link R_shin: mass 0.470000 -> 1.375365
- link R_shoulder_pitch_link: mass 0.100000 -> 0.346898
- link R_thigh: mass 0.660000 -> 2.468826
- link R_upper_arm: mass 0.270000 -> 0.785245
- link neck_pan_link: mass 0.100000 -> 0.140911

Commit message: Lighten HR-30 whole-body architecture

File: hr30/whole-body-p0.1/hr30.urdf (robot description, URDF)
Before this commit: robot hr30_whole_body_p01, 26 links, 25 joints
Links:
- link L_forearm: mass 0.245747 -> 0.220000
- link L_shin: mass 1.375365 -> 0.884419
- link L_shoulder_pitch_link: mass 0.346898 -> 0.261770
- link L_thigh: mass 2.468826 -> 1.569667
- link L_upper_arm: mass 0.785245 -> 0.574138
- link R_forearm: mass 0.245747 -> 0.220000
- link R_shin: mass 1.375365 -> 0.884419
- link R_shoulder_pitch_link: mass 0.346898 -> 0.261770
- link R_thigh: mass 2.468826 -> 1.569667
- link R_upper_arm: mass 0.785245 -> 0.574138
- link neck_pan_link: mass 0.140911 -> 0.116516

Commit message: Install HR-30 whole-body equipment layout

File: hr30/whole-body-p0.1/hr30.urdf (robot description, URDF)
Before this commit: robot hr30_whole_body_p01, 26 links, 25 joints
Links:
- link L_ankle_pitch_link: mass 0.130000 -> 0.000000
- link L_foot: mass 0.605000 -> 0.243626
- link L_forearm: mass 0.220000 -> 0.198596
- link L_gripper: mass 0.030000 -> 0.000000
- link L_hand: mass 0.180000 -> 0.055246
- link L_hip_roll_link: mass 0.080000 -> 0.000000
- link L_hip_yaw_link: mass 0.080000 -> 0.000000
- link L_shin: mass 0.884419 -> 0.955173
- link L_shoulder_pitch_link: mass 0.261770 -> 0.282712
- link L_thigh: mass 1.569667 -> 1.770841
- link L_upper_arm: mass 0.574138 -> 0.663269
- link R_ankle_pitch_link: mass 0.130000 -> 0.000000
- link R_foot: mass 0.605000 -> 0.243626
- link R_forearm: mass 0.220000 -> 0.198596
- link R_gripper: mass 0.030000 -> 0.000000
- link R_hand: mass 0.180000 -> 0.055246
- link R_hip_roll_link: mass 0.080000 -> 0.000000
- link R_hip_yaw_link: mass 0.080000 -> 0.000000
- link R_shin: mass 0.884419 -> 0.955173
- link R_shoulder_pitch_link: mass 0.261770 -> 0.282712
- link R_thigh: mass 1.569667 -> 1.770841
- link R_upper_arm: mass 0.574138 -> 0.663269
- link base_link: mass 1.650000 -> 1.792017
- link head: mass 0.400000 -> 0.454523
- link neck_pan_link: mass 0.116516 -> 0.125838
- link torso: mass 1.830000 -> 0.861933

Commit message: Add HR-30 whole-body joint load architecture

File: hr30/whole-body-p0.1/hr30.urdf (robot description, URDF)
Before this commit: robot hr30_whole_body_p01, 26 links, 25 joints
Links:
- link L_forearm: mass 0.198596 -> 0.196659
- link L_hand: mass 0.055246 -> 0.057587
- link L_shin: mass 0.955173 -> 0.916987
- link L_shoulder_pitch_link: mass 0.282712 -> 0.272121
- link L_thigh: mass 1.770841 -> 1.711317
- link L_upper_arm: mass 0.663269 -> 0.557743
- link R_forearm: mass 0.198596 -> 0.196659
- link R_hand: mass 0.055246 -> 0.057587
- link R_shin: mass 0.955173 -> 0.916987
- link R_shoulder_pitch_link: mass 0.282712 -> 0.272121
- link R_thigh: mass 1.770841 -> 1.711317
- link R_upper_arm: mass 0.663269 -> 0.557743
- link base_link: mass 1.792017 -> 1.753100
- link head: mass 0.454523 -> 0.452586
- link neck_pan_link: mass 0.125838 -> 0.123901

Commit message: Complete HR-30 whole-body actuation and mass architecture

File: hr30/whole-body-p0.1/hr30.urdf (robot description, URDF)
Before this commit: robot hr30_whole_body_p01, 26 links, 25 joints
Links:
- link L_foot: mass 0.243626 -> 0.239897
- link L_forearm: mass 0.196659 -> 0.127975
- link L_hand: mass 0.057587 -> 0.057028
- link L_shin: mass 0.916987 -> 0.706736
- link L_thigh: mass 1.711317 -> 1.592396
- link L_upper_arm: mass 0.557743 -> 0.462631
- link R_foot: mass 0.243626 -> 0.239897
- link R_forearm: mass 0.196659 -> 0.127975
- link R_hand: mass 0.057587 -> 0.057028
- link R_shin: mass 0.916987 -> 0.706736
- link R_thigh: mass 1.711317 -> 1.592396
- link R_upper_arm: mass 0.557743 -> 0.462631
- link base_link: mass 1.753100 -> 1.701164
- link head: mass 0.452586 -> 0.430808
- link torso: mass 0.861933 -> 0.819217

Commit message: Model HR-30 onboard walking energy

File: hr30/whole-body-p0.1/hr30.urdf (robot description, URDF)
Before this commit: robot hr30_whole_body_p01, 26 links, 25 joints
Links:
- link torso: mass 0.819217 -> 2.284777

Commit message: Correct HR-30 arm datums and close nominal pose collisions

File: hr30/whole-body-p0.1/hr30.urdf (robot description, URDF)
Before this commit: robot hr30_whole_body_p01, 26 links, 25 joints
Joints:
- joint L_ELBOW_PITCH: origin xyz=0.020000 0.000000 -0.150000 rpy=0 0 0 -> xyz=0.030000 0.000000 -0.150000 rpy=0 0 0
- joint L_GRIPPER: axis 1 0 0 -> 1.0 0 0
- joint L_WRIST_ROTATION: origin xyz=0.000000 0.000000 -0.145000 rpy=0 0 0 -> xyz=0.005000 0.000000 -0.145000 rpy=0 0 0
- joint R_ELBOW_PITCH: origin xyz=-0.020000 0.000000 -0.150000 rpy=0 0 0 -> xyz=-0.030000 0.000000 -0.150000 rpy=0 0 0
- joint R_GRIPPER: axis 1 0 0 -> -1.0 0 0
- joint R_WRIST_ROTATION: origin xyz=0.000000 0.000000 -0.145000 rpy=0 0 0 -> xyz=-0.005000 0.000000 -0.145000 rpy=0 0 0

Commit message: Add located HR-30 joint fasteners

File: hr30/whole-body-p0.1/hr30.urdf (robot description, URDF)
Before this commit: robot hr30_whole_body_p01, 26 links, 25 joints
Links:
- link L_hand: mass 0.057028 -> 0.059216
- link L_shin: mass 0.706736 -> 0.784854
- link L_shoulder_pitch_link: mass 0.272121 -> 0.298024
- link L_thigh: mass 1.592396 -> 1.713300
- link L_upper_arm: mass 0.462631 -> 0.489145
- link R_hand: mass 0.057028 -> 0.059216
- link R_shin: mass 0.706736 -> 0.784854
- link R_shoulder_pitch_link: mass 0.272121 -> 0.298024
- link R_thigh: mass 1.592396 -> 1.713300
- link R_upper_arm: mass 0.462631 -> 0.489145
- link base_link: mass 1.701164 -> 1.702403
- link head: mass 0.430808 -> 0.433766

Commit message: Integrate detailed hands into HR-30 whole-body build

File: hr30/whole-body-p0.1/hr30.urdf (robot description, URDF)
Before this commit: robot hr30_whole_body_p01, 26 links, 25 joints
Links:
- link L_hand: mass 0.055657 -> 0.180321
- link R_hand: mass 0.055657 -> 0.180321

Commit message: Install product-specific drivetrains in HR-30 body

File: hr30/whole-body-p0.1/hr30.urdf (robot description, URDF)
Before this commit: robot hr30_whole_body_p01, 26 links, 25 joints
Links:
- link L_hand: mass 0.180321 -> 0.179531
- link L_shin: mass 0.745112 -> 0.739993
- link L_thigh: mass 1.642432 -> 1.635577; geometry collision box size=0.074000 0.076000 0.160000; visual box size=0.074000 0.076000 0.160000
- link R_hand: mass 0.180321 -> 0.179531
- link R_shin: mass 0.745112 -> 0.739993
- link R_thigh: mass 1.642432 -> 1.635577; geometry collision box size=0.074000 0.076000 0.160000; visual box size=0.074000 0.076000 0.160000
- link base_link: mass 1.686946 -> 1.690125
Joints:
- joint L_ANKLE_PITCH: origin xyz=0.000000 0.000000 -0.165000 rpy=0 0 0 -> xyz=0.000000 0.000000 -0.155000 rpy=0 0 0
- joint L_ANKLE_ROLL: origin xyz=0.000000 0.000000 -0.008000 rpy=0 0 0 -> xyz=0.000000 0.000000 -0.020000 rpy=0 0 0
- joint L_HIP_PITCH: origin xyz=0.000000 0.000000 -0.008000 rpy=0 0 0 -> xyz=0.000000 0.000000 -0.020000 rpy=0 0 0
- joint L_HIP_ROLL: origin xyz=0.000000 0.000000 -0.009000 rpy=0 0 0 -> xyz=0.000000 0.000000 -0.020000 rpy=0 0 0
- joint L_HIP_YAW: origin xyz=0.062500 0.000000 0.007000 rpy=0 0 0 -> xyz=0.062500 0.000000 0.020000 rpy=0 0 0
- joint L_KNEE_PITCH: origin xyz=0.000000 0.000000 -0.170000 rpy=0 0 0 -> xyz=0.000000 0.000000 -0.160000 rpy=0 0 0
- joint R_ANKLE_PITCH: origin xyz=0.000000 0.000000 -0.165000 rpy=0 0 0 -> xyz=0.000000 0.000000 -0.155000 rpy=0 0 0
- joint R_ANKLE_ROLL: origin xyz=0.000000 0.000000 -0.008000 rpy=0 0 0 -> xyz=0.000000 0.000000 -0.020000 rpy=0 0 0
- joint R_HIP_PITCH: origin xyz=0.000000 0.000000 -0.008000 rpy=0 0 0 -> xyz=0.000000 0.000000 -0.020000 rpy=0 0 0
- joint R_HIP_ROLL: origin xyz=0.000000 0.000000 -0.009000 rpy=0 0 0 -> xyz=0.000000 0.000000 -0.020000 rpy=0 0 0
- joint R_HIP_YAW: origin xyz=-0.062500 0.000000 0.007000 rpy=0 0 0 -> xyz=-0.062500 0.000000 0.020000 rpy=0 0 0
- joint R_KNEE_PITCH: origin xyz=0.000000 0.000000 -0.170000 rpy=0 0 0 -> xyz=0.000000 0.000000 -0.160000 rpy=0 0 0

Commit message: Increase HR-30 hip-to-torso service clearance

File: hr30/whole-body-p0.1/hr30.urdf (robot description, URDF)
Before this commit: robot hr30_whole_body_p01, 26 links, 25 joints
Links:
- link torso: mass 2.351799 -> 2.340610; geometry collision box size=0.190000 0.110000 0.145000; visual box size=0.190000 0.110000 0.145000

Commit message: Build HR-30 tether power core

File: hr30/whole-body-p0.1/hr30.urdf (robot description, URDF)
Before this commit: robot hr30_whole_body_p01, 26 links, 25 joints
Links:
- link base_link: mass 1.538925 -> 1.511925

Commit message: Close HR-30 current-constrained whole-body candidate

File: hr30/whole-body-p0.1/hr30.urdf (robot description, URDF)
Before this commit: robot hr30_whole_body_p01, 26 links, 25 joints
Links:
- link L_thigh: mass 1.680577 -> 1.677714
- link R_thigh: mass 1.680577 -> 1.677714

File: hr30/whole-body-p0.1/hr30_tether.urdf (robot description, URDF)
Before this commit: robot hr30_whole_body_p01, 26 links, 25 joints
Links:
- link L_thigh: mass 1.680577 -> 1.677714
- link R_thigh: mass 1.680577 -> 1.677714

Commit message: Close HR-30 10 kg planning envelope

File: hr30/whole-body-p0.1/hr30.urdf (robot description, URDF)
Before this commit: robot hr30_whole_body_p01, 26 links, 25 joints
Links:
- link L_foot: mass 0.239897 -> 0.211981
- link L_forearm: mass 0.125225 -> 0.120261
- link L_shin: mass 0.739993 -> 0.705487
- link L_thigh: mass 1.677714 -> 1.638884
- link L_upper_arm: mass 0.460814 -> 0.455342
- link R_foot: mass 0.239897 -> 0.211981
- link R_forearm: mass 0.125225 -> 0.120261
- link R_shin: mass 0.739993 -> 0.705487
- link R_thigh: mass 1.677714 -> 1.638884
- link R_upper_arm: mass 0.460814 -> 0.455342
- link base_link: mass 1.511925 -> 1.495522
- link head: mass 0.431016 -> 0.409453
- link torso: mass 2.437810 -> 2.356726

File: hr30/whole-body-p0.1/hr30_tether.urdf (robot description, URDF)
Before this commit: robot hr30_whole_body_p01, 26 links, 25 joints
Links:
- link L_foot: mass 0.239897 -> 0.211981
- link L_forearm: mass 0.125225 -> 0.120261
- link L_shin: mass 0.739993 -> 0.705487
- link L_thigh: mass 1.677714 -> 1.638884
- link L_upper_arm: mass 0.460814 -> 0.455342
- link R_foot: mass 0.239897 -> 0.211981
- link R_forearm: mass 0.125225 -> 0.120261
- link R_shin: mass 0.739993 -> 0.705487
- link R_thigh: mass 1.677714 -> 1.638884
- link R_upper_arm: mass 0.460814 -> 0.455342
- link base_link: mass 1.511925 -> 1.495522
- link head: mass 0.431016 -> 0.409453
- link torso: mass 0.972250 -> 0.891166

Commit message: Add synchronized HR-30 head HMI harness

File: hr30/whole-body-p0.1/hr30.urdf (robot description, URDF)
Before this commit: robot hr30_whole_body_p01, 26 links, 25 joints
Links:
- link head: mass 0.409453 -> 0.439477

File: hr30/whole-body-p0.1/hr30_tether.urdf (robot description, URDF)
Before this commit: robot hr30_whole_body_p01, 26 links, 25 joints
Links:
- link head: mass 0.409453 -> 0.439477

Commit message: Add HR-30 whole-body dynamics validation

File: hr30/whole-body-p0.1/hr30.urdf (robot description, URDF)
Before this commit: robot hr30_whole_body_p01, 26 links, 25 joints
Links:
- link L_ankle_pitch_link: mass 0.000000 -> 0.258987
- link L_foot: mass 0.167444 -> 0.448853
- link L_forearm: mass 0.113606 -> 0.201786
- link L_gripper: mass 0.000000 -> 0.040804
- link L_hand: mass 0.169931 -> 0.172070
- link L_hip_roll_link: mass 0.000000 -> 0.343564
- link L_hip_yaw_link: mass 0.000000 -> 0.249282
- link L_shin: mass 0.697911 -> 0.524223
- link L_thigh: mass 1.630169 -> 0.691460
- link L_upper_arm: mass 0.446793 -> 0.310504
- link R_ankle_pitch_link: mass 0.000000 -> 0.258987
- link R_foot: mass 0.167444 -> 0.448853
- link R_forearm: mass 0.113606 -> 0.201786
- link R_gripper: mass 0.000000 -> 0.040804
- link R_hand: mass 0.169931 -> 0.172070
- link R_hip_roll_link: mass 0.000000 -> 0.343564
- link R_hip_yaw_link: mass 0.000000 -> 0.249282
- link R_shin: mass 0.697911 -> 0.524223
- link R_thigh: mass 1.630169 -> 0.691460
- link R_upper_arm: mass 0.446793 -> 0.310504

File: hr30/whole-body-p0.1/hr30_tether.urdf (robot description, URDF)
Before this commit: robot hr30_whole_body_p01, 26 links, 25 joints
Links:
- link L_ankle_pitch_link: mass 0.000000 -> 0.258987
- link L_foot: mass 0.167444 -> 0.448853
- link L_forearm: mass 0.113606 -> 0.201786
- link L_gripper: mass 0.000000 -> 0.040804
- link L_hand: mass 0.169931 -> 0.172070
- link L_hip_roll_link: mass 0.000000 -> 0.343564
- link L_hip_yaw_link: mass 0.000000 -> 0.249282
- link L_shin: mass 0.697911 -> 0.524223
- link L_thigh: mass 1.630169 -> 0.691460
- link L_upper_arm: mass 0.446793 -> 0.310504
- link R_ankle_pitch_link: mass 0.000000 -> 0.258987
- link R_foot: mass 0.167444 -> 0.448853
- link R_forearm: mass 0.113606 -> 0.201786
- link R_gripper: mass 0.000000 -> 0.040804
- link R_hand: mass 0.169931 -> 0.172070
- link R_hip_roll_link: mass 0.000000 -> 0.343564
- link R_hip_yaw_link: mass 0.000000 -> 0.249282
- link R_shin: mass 0.697911 -> 0.524223
- link R_thigh: mass 1.630169 -> 0.691460
- link R_upper_arm: mass 0.446793 -> 0.310504
