File: hr30/whole-body-p0.1/electrical/carriers-p0.1/06_rs_waist.kicad_sch (KiCad schematic)
At the start: 12 parts, among them J105 RS-WAIST data-only field, U105 ISOW1432DFMR RS-WAIST

Commit message: Integrate HR-30 PA field connector harnesses
Parts:
- J105: footprint Connector_JST:JST_GH_BM03B-GHS-TBT_1x03-1MP_P1.25mm_Vertical -> HR30_PA:JST_PA_B03B-PASK-1; Evidence No actuator VDD contact -> JST PA 2.0 mm secure-lock through-hole header; PAP-03V-S/SP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
Changed lines of the file:
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@@
       (property "Reference" "J105" (at 160.02 31.56 0) (effects (font (size 1.50 1.50)) (justify left bottom)))
       (property "Value" "RS-WAIST data-only field" (at 199.39 48.26 0) (effects (font (size 1.50 1.50)) (hide yes)))
-      (property "Footprint" "Connector_JST:JST_GH_BM03B-GHS-TBT_1x03-1MP_P1.25mm_Vertical" (at 199.39 48.26 0) (effects (font (size 1.50 1.50)) (hide yes)))
-      (property "Datasheet" "https://www.jst-mfg.com/product/pdf/eng/eGH.pdf" (at 199.39 48.26 0) (effects (font (size 1.50 1.50)) (hide yes)))
-      (property "Description" "No actuator VDD contact" (at 199.39 48.26 0) (effects (font (size 1.50 1.50)) (hide yes)))
+      (property "Footprint" "HR30_PA:JST_PA_B03B-PASK-1" (at 199.39 48.26 0) (effects (font (size 1.50 1.50)) (hide yes)))
+      (property "Datasheet" "https://www.jst-mfg.com/product/pdf/eng/ePA-F.pdf" (at 199.39 48.26 0) (effects (font (size 1.50 1.50)) (hide yes)))
+      (property "Description" "JST PA 2.0 mm secure-lock through-hole header; PAP-03V-S/SPHD-001T-P0.5 harness candidate; no actuator VDD contact" (at 199.39 48.26 0) (effects (font (size 1.50 1.50)) (hide yes)))
       (property "Status" "EXACT COMPONENT AND FOOTPRINT CANDIDATE; APPLICATION VALIDATION OPEN" (at 199.39 63.96 0) (effects (font (size 1.50 1.50)) (justify bottom)))
-      (property "Evidence" "No actuator VDD contact" (at 199.39 48.26 0) (effects (font (size 1.50 1.50)) (hide yes)))
+      (property "Evidence" "JST PA 2.0 mm secure-lock through-hole header; PAP-03V-S/SPHD-001T-P0.5 harness candidate; no actuator VDD contact" (at 199.39 48.26 0) (effects (font (size 1.50 1.50)) (hide yes)))
       (property "Display" "RS-WAIST data-only field" (at 160.02 34.76 0) (effects (font (size 1.50 1.50)) (justify left bottom)))
       (pin "1")
