File: hr30/whole-body-p0.1/electrical/carriers-p0.1/07_ttl_ldist.kicad_sch (KiCad schematic)
At the start: 8 parts, among them J201 TTL-LDIST data-only field, U201 SN74LVC1T45DCKR TTL-LDIST

Commit message: Integrate HR-30 PA field connector harnesses
Parts:
- J201: footprint Connector_JST:JST_GH_BM02B-GHS-TBT_1x02-1MP_P1.25mm_Vertical -> HR30_PA:JST_PA_B02B-PASK-1; Evidence No actuator VDD contact -> JST PA 2.0 mm secure-lock through-hole header; PAP-02V-S/SP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
Changed lines of the file:
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@@
       (property "Reference" "J201" (at 160.02 31.56 0) (effects (font (size 1.50 1.50)) (justify left bottom)))
       (property "Value" "TTL-LDIST data-only field" (at 199.39 48.26 0) (effects (font (size 1.50 1.50)) (hide yes)))
-      (property "Footprint" "Connector_JST:JST_GH_BM02B-GHS-TBT_1x02-1MP_P1.25mm_Vertical" (at 199.39 48.26 0) (effects (font (size 1.50 1.50)) (hide yes)))
-      (property "Datasheet" "https://www.jst-mfg.com/product/pdf/eng/eGH.pdf" (at 199.39 48.26 0) (effects (font (size 1.50 1.50)) (hide yes)))
-      (property "Description" "No actuator VDD contact" (at 199.39 48.26 0) (effects (font (size 1.50 1.50)) (hide yes)))
+      (property "Footprint" "HR30_PA:JST_PA_B02B-PASK-1" (at 199.39 48.26 0) (effects (font (size 1.50 1.50)) (hide yes)))
+      (property "Datasheet" "https://www.jst-mfg.com/product/pdf/eng/ePA-F.pdf" (at 199.39 48.26 0) (effects (font (size 1.50 1.50)) (hide yes)))
+      (property "Description" "JST PA 2.0 mm secure-lock through-hole header; PAP-02V-S/SPHD-002T-P0.5 harness candidate; no actuator VDD contact" (at 199.39 48.26 0) (effects (font (size 1.50 1.50)) (hide yes)))
       (property "Status" "EXACT COMPONENT AND FOOTPRINT CANDIDATE; APPLICATION VALIDATION OPEN" (at 199.39 63.96 0) (effects (font (size 1.50 1.50)) (justify bottom)))
-      (property "Evidence" "No actuator VDD contact" (at 199.39 48.26 0) (effects (font (size 1.50 1.50)) (hide yes)))
+      (property "Evidence" "JST PA 2.0 mm secure-lock through-hole header; PAP-02V-S/SPHD-002T-P0.5 harness candidate; no actuator VDD contact" (at 199.39 48.26 0) (effects (font (size 1.50 1.50)) (hide yes)))
       (property "Display" "TTL-LDIST data-only field" (at 160.02 34.76 0) (effects (font (size 1.50 1.50)) (justify left bottom)))
       (pin "1")
