File: hr30/whole-body-p0.1/electrical/motion-controller-p0.1/board/hr30-motion-controller-p0.1.kicad_pcb (KiCad board)
At the start: 6 copper layers, 82 x 42 mm, 40 parts, among them J1 Protected auxiliary 5 V input, U1 STM32H743ZIT6 deterministic m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, U2 TPS62132 3.3 V / 3 A buck

Commit message: Integrate HR-30 PA field connector harnesses
Routing:
- net AUX_5V_SAFE: track 13.7 -> 16.6 mm
