Commit message: Reconcile HR-30 whole-body mass and harness

File: hr30/whole-body-p0.1/hip-transmission-p0.1/hr30_tether_hip4_candidate.urdf (robot description, URDF)
Before this commit: robot hr30_whole_body_p01, 26 links, 25 joints
Links:
- link L_foot: mass 0.448853 -> 0.436839
- link L_forearm: mass 0.201786 -> 0.195138
- link L_shin: mass 0.524223 -> 0.509954
- link L_thigh: mass 0.691460 -> 0.675468
- link L_upper_arm: mass 0.310504 -> 0.303473
- link R_foot: mass 0.448853 -> 0.436839
- link R_forearm: mass 0.201786 -> 0.195138
- link R_shin: mass 0.524223 -> 0.509954
- link R_thigh: mass 0.691460 -> 0.675468
- link R_upper_arm: mass 0.310504 -> 0.303473
- link torso: mass 1.034189 -> 0.987371

File: hr30/whole-body-p0.1/hr30.urdf (robot description, URDF)
Before this commit: robot hr30_whole_body_p01, 26 links, 25 joints
Links:
- link L_foot: mass 0.448853 -> 0.436839
- link L_forearm: mass 0.201786 -> 0.195138
- link L_shin: mass 0.524223 -> 0.509954
- link L_thigh: mass 0.691460 -> 0.675468
- link L_upper_arm: mass 0.310504 -> 0.303473
- link R_foot: mass 0.448853 -> 0.436839
- link R_forearm: mass 0.201786 -> 0.195138
- link R_shin: mass 0.524223 -> 0.509954
- link R_thigh: mass 0.691460 -> 0.675468
- link R_upper_arm: mass 0.310504 -> 0.303473
- link torso: mass 2.499749 -> 2.452931

File: hr30/whole-body-p0.1/hr30_tether.urdf (robot description, URDF)
Before this commit: robot hr30_whole_body_p01, 26 links, 25 joints
Links:
- link L_foot: mass 0.448853 -> 0.436839
- link L_forearm: mass 0.201786 -> 0.195138
- link L_shin: mass 0.524223 -> 0.509954
- link L_thigh: mass 0.691460 -> 0.675468
- link L_upper_arm: mass 0.310504 -> 0.303473
- link R_foot: mass 0.448853 -> 0.436839
- link R_forearm: mass 0.201786 -> 0.195138
- link R_shin: mass 0.524223 -> 0.509954
- link R_thigh: mass 0.691460 -> 0.675468
- link R_upper_arm: mass 0.310504 -> 0.303473
- link torso: mass 1.034189 -> 0.987371

File: hr30/whole-body-p0.1/lightweight-hip-successor-p0.1/hr30_tether_light4_candidate.urdf (robot description, URDF)
Before this commit: robot hr30_whole_body_p01, 26 links, 25 joints
Links:
- link L_foot: mass 0.448853 -> 0.436839
- link L_forearm: mass 0.201786 -> 0.195138
- link L_shin: mass 0.524223 -> 0.509954
- link L_thigh: mass 0.691460 -> 0.675468
- link L_upper_arm: mass 0.310504 -> 0.303473
- link R_foot: mass 0.448853 -> 0.436839
- link R_forearm: mass 0.201786 -> 0.195138
- link R_shin: mass 0.524223 -> 0.509954
- link R_thigh: mass 0.691460 -> 0.675468
- link R_upper_arm: mass 0.310504 -> 0.303473
- link torso: mass 1.034189 -> 0.987371
