File: hr30/whole-body-p0.1/electrical/measurement-boundary-panel-p0.1/01_channels_1_4.kicad_sch (KiCad schematic)
At the start: 24 parts, among them J1I ACT_MAIN_SOURCE_12V floating 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, J1O to ACT_MAIN_SOURCE_12V DAQ in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, J2I ACT_MAIN_SAFE_12V floating in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, J2O to ACT_MAIN_SAFE_12V DAQ input, J3I TTL_SELECTED_SAFE_9V floating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, J3O to TTL_SELECTED_SAFE_9V DAQ i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, J4I CTRL_SAFE_5V floating input, J4O to CTRL_SAFE_5V DAQ input

Commit message: Add HR-30 first-energization measurement harness
Parts:
- J3I: value TTL_SELECTED_SAFE_9V floating input -> TTL_LDIST_SAFE_9V floating input; Display TTL_SELECTED_SAFE_9V floating input -> TTL_LDIST_SAFE_9V floating input
- J3O: value to TTL_SELECTED_SAFE_9V DAQ input -> to TTL_LDIST_SAFE_9V DAQ input; Display to TTL_SELECTED_SAFE_9V DAQ input -> to TTL_LDIST_SAFE_9V DAQ input
- J4I: value CTRL_SAFE_5V floating input -> CTRL_5V floating input; Display CTRL_SAFE_5V floating input -> CTRL_5V floating input
- J4O: value to CTRL_SAFE_5V DAQ input -> to CTRL_5V DAQ input; Display to CTRL_SAFE_5V DAQ input -> to CTRL_5V DAQ input
