File: hr30/whole-body-p0.1/electrical/measurement-boundary-panel-p0.1/02_channels_5_8.kicad_sch (KiCad schematic)
At the start: 24 parts, among them J5I ESTOP_CH_A_24V floating input, J5O to ESTOP_CH_A_24V DAQ input, J6I WATCHDOG_PERMIT_24V floating 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, J6O to WATCHDOG_PERMIT_24V DAQ in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, J7I K1_DIAGNOSTIC_24V floating in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, J7O to K1_DIAGNOSTIC_24V DAQ input, J8I K2_DIAGNOSTIC_24V floating in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, J8O to K2_DIAGNOSTIC_24V DAQ input

Commit message: Add HR-30 first-energization measurement harness
Parts:
- J6I: value WATCHDOG_PERMIT_24V floating input -> HARDWIRED_PERMIT_24V floating input; Display WATCHDOG_PERMIT_24V floating input -> HARDWIRED_PERMIT_24V floating input
- J6O: value to WATCHDOG_PERMIT_24V DAQ input -> to HARDWIRED_PERMIT_24V DAQ input; Display to WATCHDOG_PERMIT_24V DAQ input -> to HARDWIRED_PERMIT_24V DAQ input
- J7I: value K1_DIAGNOSTIC_24V floating input -> K1_COIL_24V floating input; Display K1_DIAGNOSTIC_24V floating input -> K1_COIL_24V floating input
- J7O: value to K1_DIAGNOSTIC_24V DAQ input -> to K1_COIL_24V DAQ input; Display to K1_DIAGNOSTIC_24V DAQ input -> to K1_COIL_24V DAQ input
- J8I: value K2_DIAGNOSTIC_24V floating input -> K2_COIL_24V floating input; Display K2_DIAGNOSTIC_24V floating input -> K2_COIL_24V floating input
- J8O: value to K2_DIAGNOSTIC_24V DAQ input -> to K2_COIL_24V DAQ input; Display to K2_DIAGNOSTIC_24V DAQ input -> to K2_COIL_24V DAQ input
