File: hr30/whole-body-p0.1/electrical/auxiliary-power-module-p0.1/01_compute_rail.kicad_sch (KiCad schematic)
At the start: 5 parts, among them U1 REC30E-2405SZ COMPUTE isolate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

Commit message: Increase HR-30 HMI power margin
Parts:
- U1: Evidence REV 1/2024; 9-36 V input, 5 V 6 A output, 89% typical effic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 -> REV 1/2024; 9-36 V input, 5 V/6 A output, 89% typical effic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
Changed lines of the file:
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@@
       (property "Footprint" "HR30_AUX:REC30E-Z" (at 54.61 152.40 0) (effects (font (size 1.50 1.50)) (hide yes)))
       (property "Datasheet" "https://recom-power.com/pdf/Econoline/REC30E-Z.pdf" (at 54.61 152.40 0) (effects (font (size 1.50 1.50)) (hide yes)))
-      (property "Description" "REV 1/2024; 9-36 V input, 5 V 6 A output, 89% typical efficiency, 2 kVDC/1 min isolation; pin 5 trim deliberately unconnected" (at 54.61 152.40 0) (effects (font (size 1.50 1.50)) (hide yes)))
+      (property "Description" "REV 1/2024; 9-36 V input, 5 V/6 A output, 89% typical efficiency, 2 kVDC/1 min isolation; pin 5 trim deliberately unconnected" (at 54.61 152.40 0) (effects (font (size 1.50 1.50)) (hide yes)))
       (property "Status" "CANDIDATE / SELECTION REQUIRED" (at 54.61 168.10 0) (effects (font (size 1.50 1.50)) (justify bottom)))
-      (property "Evidence" "REV 1/2024; 9-36 V input, 5 V 6 A output, 89% typical efficiency, 2 kVDC/1 min isolation; pin 5 trim deliberately unconnected" (at 54.61 152.40 0) (effects (font (size 1.50 1.50)) (hide yes)))
+      (property "Evidence" "REV 1/2024; 9-36 V input, 5 V/6 A output, 89% typical efficiency, 2 kVDC/1 min isolation; pin 5 trim deliberately unconnected" (at 54.61 152.40 0) (effects (font (size 1.50 1.50)) (hide yes)))
       (property "Display" "REC30E-2405SZ COMPUTE isolated converter" (at 7.62 138.90 0) (effects (font (size 1.50 1.50)) (justify left bottom)))
       (pin "1")
